File: SoilMoistureSensor/Sim/sim1/sim1.kicad_sch (KiCad schematic)
At the start: 32 parts, among them U1 74AUC1G86, U10 74AUC1G66, U11 74AUC1G66, U12 74AUC1G66, U2 74AUC1G86, U3 74AUC1G86, U4 74AUC1G86, U5 74AUC1G08, U6 74AUC1G08, U7 OPA356xxDBV, U8 OPA356xxDBV, U9 74AUC1G66

Commit message: wip
Parts:
- C3, C4: value 640p -> 10p
- C5, C6: value 1n -> 100p
- R5, R7: value 1k -> 10k
Changed lines of the file:
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@@
       (effects (font (size 1.27 1.27)) (justify left))
     )
-    (property "Value" "640p" (id 1) (at 130.81 143.5099 0)
+    (property "Value" "10p" (id 1) (at 130.81 143.5099 0)
       (effects (font (size 1.27 1.27)) (justify left))
     )
@@
       (effects (font (size 1.27 1.27)) (justify left))
     )
-    (property "Value" "1n" (id 1) (at 151.1299 45.72 0)
+    (property "Value" "100p" (id 1) (at 151.1299 45.72 0)
       (effects (font (size 1.27 1.27)) (justify left))
     )
@@
       (effects (font (size 1.27 1.27)) (justify right))
     )
-    (property "Value" "1k" (id 1) (at 160.02 105.4099 0)
+    (property "Value" "10k" (id 1) (at 160.02 105.4099 0)
       (effects (font (size 1.27 1.27)) (justify right))
     )
@@
       (effects (font (size 1.27 1.27)) (justify right))
     )
-    (property "Value" "1k" (id 1) (at 160.02 59.6899 0)
+    (property "Value" "10k" (id 1) (at 160.02 59.6899 0)
       (effects (font (size 1.27 1.27)) (justify right))
     )
@@
       (effects (font (size 1.27 1.27)) (justify left))
     )
-    (property "Value" "1n" (id 1) (at 149.8599 93.98 0)
+    (property "Value" "100p" (id 1) (at 149.8599 93.98 0)
       (effects (font (size 1.27 1.27)) (justify left))
     )
@@
       (effects (font (size 1.27 1.27)) (justify left))
     )
-    (property "Value" "640p" (id 1) (at 142.24 143.5099 0)
+    (property "Value" "10p" (id 1) (at 142.24 143.5099 0)
       (effects (font (size 1.27 1.27)) (justify left))
     )
@@
     )
     (path "/20f1a5b6-a0c0-4191-b380-40a92bac1750"
-      (reference "C3") (unit 1) (value "640p") (footprint "")
+      (reference "C3") (unit 1) (value "10p") (footprint "")
     )
     (path "/fd95ad9f-2731-4a7d-a50f-63a04c501383"
-      (reference "C4") (unit 1) (value "640p") (footprint "")
+      (reference "C4") (unit 1) (value "10p") (footprint "")
     )
     (path "/dc06e083-559e-48fc-b28e-cbb8a27e61e9"
-      (reference "C5") (unit 1) (value "1n") (footprint "")
+      (reference "C5") (unit 1) (value "100p") (footprint "")
     )
     (path "/7aac5cb9-47a9-4183-bae5-661ca330207d"
-      (reference "C6") (unit 1) (value "1n") (footprint "")
+      (reference "C6") (unit 1) (value "100p") (footprint "")
     )
     (path "/c22cca3d-8784-4c3c-990f-b6c9443b22f8"
@@
     )
     (path "/9b7b4ae1-5927-4ae1-b372-06ad64ba3673"
-      (reference "R5") (unit 1) (value "1k") (footprint "")
+      (reference "R5") (unit 1) (value "10k") (footprint "")
     )
     (path "/5b9e649c-2282-4f1c-a519-ede702a18acb"
@@
     )
     (path "/bdd69951-27a8-48b2-beef-ac79c545d712"
-      (reference "R7") (unit 1) (value "1k") (footprint "")
+      (reference "R7") (unit 1) (value "10k") (footprint "")
     )
     (path "/8310945c-8e79-4f54-9866-4b4eb7d1e2ac"

Commit message: - wip
Parts:
- removed C8: 100n, symbol Device:C
- removed C9: 400n, symbol Device:C
- removed R4: 40k, symbol Device:R
- removed R6: 10k, symbol Device:R
- added R10, R9: 1k, symbol Device:R
- added R12, R13, R16, R17: 10k, symbol Device:R
- added R14, R15, R18, R19: 20k, symbol Device:R
- added U13, U14, U15: MCP6001-OT, Package_TO_SOT_SMD:SOT-23-5, symbol Amplifier_Operational:MCP6001-OT
- added V3: VDC, symbol Simulation_SPICE:VDC
- C1: Spice_Model (none) -> 1n; Spice_Netlist_Enabled (none) -> Y; Spice_Primitive (none) -> C
- C3, C4: Spice_Model (none) -> 10p IC=1.25; Spice_Netlist_Enabled (none) -> Y; Spice_Primitive (none) -> C
- R1, R2: value 2k2 -> 1k
- V1: Spice_Model pulse(0 2.5 0 3.3n 3.3n 4.5125n 15.625n) -> pulse(0 2.5 0 1n 1n 4n 10n)
Connections:
- net +2V5: now also U13.5 (V+), U14.5 (V+), U15.5 (V+)
- net 0: now also R14.1, R16.1, R17.1, U13.2 (V-), U14.2 (V-), U15.2 (V-), V3.2
- net 0.5VREF: now also V3.1
- net at R11.1, U11.2: no longer U9.2
- net at R8.1, U12.2: no longer U10.2
- net Cout+: no longer names the net of C7.1, R11.2
- net Cout+: now also R9.2, U15.3 (+)
- net Cout-: no longer names the net of C1.1, R8.2
- net Cout-: now also R10.2, U14.3 (+)
- new net: R13.1, R15.2, U13.4 (-)
- new net: R13.2, R18.2, U14.1
- new net: R9.1, U9.2
- new net: R12.2, R14.2, U13.3 (+)
- new net: R16.2, R18.1, U14.4 (-)
- new net: R10.1, U10.2
- new net: R12.1, R19.2, U15.1
- new net: R17.2, R19.1, U15.4 (-)
- new net Cout: R15.1, U13.1
Other:
- moved on the sheet: C1, C2, C3, C4, C5, C6, C7, R1, R11, R2, R3, R5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

Commit message: wip
Parts:
- removed R14, R15, R18, R19: 20k, symbol Device:R
- removed R17: 10k, symbol Device:R
- removed U13, U14, U15: MCP6001-OT, Package_TO_SOT_SMD:SOT-23-5, symbol Amplifier_Operational:MCP6001-OT
- added R4: 20k, symbol Device:R
- added R6: 10k, symbol Device:R
- added U13, U14: TLV9001IDCK, Package_TO_SOT_SMD:SOT-353_SC-70-5, symbol Amplifier_Operational:TLV9001IDCK
- C1, C7: value 1n -> 10n
- R13: value 10k -> 20k
Connections:
- net +2V5: now also U13.5 (V+), U14.5 (V+)
- net 0: now also R13.1, U13.2 (V-), U14.2 (V-); no longer R16.1
- net Cout: now also R4.2, U13.4
- net at R13.2: now also R12.1, R16.1, U14.3 (-)
- net at C7.1, R11.2, R9.2: now also U13.1 (+)
- net at R12.2: now also R6.1, U14.4
- net at R16.2: now also R4.1, R6.2, U13.3 (-)
- net at C1.1, R10.2, R8.2: now also U14.1 (+)
Other:
- note added: ".TRAN 1n 20u uic"
- note added: "Test Capacitors"
- moved on the sheet: R16

Commit message: wip
Other:
- moved on the sheet: V3
Changed lines of the file:
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@@
     (stroke (width 0) (type default) (color 0 0 0 0))
   )
-  (wire (pts (xy 67.31 173.99) (xy 67.31 176.53))
+  (wire (pts (xy 67.31 176.53) (xy 67.31 179.07))
     (stroke (width 0) (type default) (color 0 0 0 0))
   )
@@
     (effects (font (size 1.27 1.27)) (justify left bottom))
   )
-  (label "0.5VREF" (at 67.31 163.83 0)
+  (label "0.5VREF" (at 67.31 166.37 0)
     (effects (font (size 1.27 1.27)) (justify left bottom))
   )
@@
     )
   )
-  (symbol (lib_id "pspice:0") (at 67.31 176.53 0) (unit 1)
-    (in_bom yes) (on_board yes)
-    (property "Reference" "#GND021" (id 0) (at 67.31 179.07 0)
-      (effects (font (size 1.27 1.27)) hide)
-    )
-    (property "Value" "0" (id 1) (at 69.85 177.8 0))
-    (property "Footprint" "" (id 2) (at 67.31 176.53 0)
-      (effects (font (size 1.27 1.27)) hide)
-    )
-    (property "Datasheet" "~" (id 3) (at 67.31 176.53 0)
+  (symbol (lib_id "pspice:0") (at 67.31 179.07 0) (unit 1)
+    (in_bom yes) (on_board yes)
+    (property "Reference" "#GND021" (id 0) (at 67.31 181.61 0)
+      (effects (font (size 1.27 1.27)) hide)
+    )
+    (property "Value" "0" (id 1) (at 69.85 180.34 0))
+    (property "Footprint" "" (id 2) (at 67.31 179.07 0)
+      (effects (font (size 1.27 1.27)) hide)
+    )
+    (property "Datasheet" "~" (id 3) (at 67.31 179.07 0)
       (effects (font (size 1.27 1.27)) hide)
     )
@@
     (pin "1")
   )
-  (symbol (lib_id "Simulation_SPICE:VDC") (at 67.31 168.91 0) (unit 1)
+  (symbol (lib_id "Simulation_SPICE:VDC") (at 67.31 171.45 0) (unit 1)
     (in_bom yes) (on_board yes) (fields_autoplaced)
-    (property "Reference" "V3" (id 0) (at 71.12 166.1801 0)
+    (property "Reference" "V3" (id 0) (at 71.12 168.7201 0)
       (effects (font (size 1.27 1.27)) (justify left))
     )
-    (property "Value" "VDC" (id 1) (at 71.12 168.7201 0)
+    (property "Value" "VDC" (id 1) (at 71.12 171.2601 0)
       (effects (font (size 1.27 1.27)) (justify left))
     )
-    (property "Footprint" "" (id 2) (at 67.31 168.91 0)
-      (effects (font (size 1.27 1.27)) hide)
-    )
-    (property "Datasheet" "~" (id 3) (at 67.31 168.91 0)
-      (effects (font (size 1.27 1.27)) hide)
-    )
-    (property "Spice_Netlist_Enabled" "Y" (id 4) (at 67.31 168.91 0)
+    (property "Footprint" "" (id 2) (at 67.31 171.45 0)
+      (effects (font (size 1.27 1.27)) hide)
+    )
+    (property "Datasheet" "~" (id 3) (at 67.31 171.45 0)
+      (effects (font (size 1.27 1.27)) hide)
+    )
+    (property "Spice_Netlist_Enabled" "Y" (id 4) (at 67.31 171.45 0)
       (effects (font (size 1.27 1.27)) (justify left) hide)
     )
-    (property "Spice_Primitive" "V" (id 5) (at 67.31 168.91 0)
+    (property "Spice_Primitive" "V" (id 5) (at 67.31 171.45 0)
       (effects (font (size 1.27 1.27)) (justify left) hide)
     )
-    (property "Spice_Model" "dc(0.5)" (id 6) (at 71.12 171.2601 0)
+    (property "Spice_Model" "dc(0.5)" (id 6) (at 71.12 173.8001 0)
       (effects (font (size 1.27 1.27)) (justify left))
     )
