File: DualLevelSensor/DualLevelSensor.kicad_sch (KiCad schematic)
At the start: 91 parts, among them J1 USB_B_Micro, J2 Conn_01x03, K1 capPad, K13 capPad, K14 capPad, K15 capPad, K16 capPad, K17 capPad, K18 capPad, K19 capPad, K2 capPad, K20 capPad, K21 capPad, K22 capPad, SW1 SW_MEC_5E, U1 W25Q16JVUXIQ, U2 RP2040, U3 AP63357Q, Y1 12Mhz

Commit message: dual level sensor routed
Parts:
- removed C22: 22µ, Capacitor_SMD:C_1206_3216Metric, symbol Device:C
- removed SW1: SW_MEC_5E, symbol Switch:SW_MEC_5E
- added J5: Conn_01x02, Connector_PinSocket_2.54mm:PinSocket_1x02_P2.54mm_Vertical, symbol Connector_Generic:Conn_01x02
- C1, C11, C14, C2, C4, C5, C7, C8: footprint (none) -> Capacitor_SMD:C_0603_1608Metric
- C10, C12, C13, C15, C16, C17, C19, C21, C23, C3, C9: footprint Capacitor_SMD:C_0201_0603Metric -> Capacitor_SMD:C_0603_1608Metric
- J2: footprint (none) -> Connector_PinHeader_2.54mm:PinHeader_1x03_P2.54mm_Vertical
- J3, J4: renamed from J?; footprint (none) -> Connector_Molex:Molex_KK-254_AE-6410-03A_1x03_P2.54mm_Vertical
- K1, K13, K14, K15, K16, K17, K18, K19, K2, K20, K21, K22: footprint (none) -> Bergi:dummyPad
- K10, K11, K12, K3, K4, K5, K6, K7, K8, K9: renamed from K?; footprint (none) -> Bergi:dummyPad
- R1, R10, R11, R12, R13, R14, R15, R16, R17, R18, R19, R2, R20, R21, R22, R23, R24, R25, R26, R27, R28, R29, R3, R30, R31, R32, R4, R5, R6, R7, R8, R9: footprint (none) -> Resistor_SMD:R_0603_1608Metric
- R33, R34: renamed from R?; footprint (none) -> Resistor_SMD:R_0603_1608Metric
Connections:
- net -aktShield: now also U2.35 (GPIO23); no longer U2.16 (GPIO13)
- net -sens1: now also U2.16 (GPIO13); no longer U2.17 (GPIO14)
- net -sens10: now also U2.34 (GPIO22); no longer U2.35 (GPIO23)
- net -sens2: now also U2.17 (GPIO14); no longer U2.18 (GPIO15)
- net -sens3: now also U2.18 (GPIO15); no longer U2.27 (GPIO16)
- net -sens4: now also U2.27 (GPIO16); no longer U2.28 (GPIO17)
- net -sens5: now also U2.28 (GPIO17); no longer U2.29 (GPIO18)
- net -sens6: now also U2.29 (GPIO18); no longer U2.30 (GPIO19)
- net -sens7: now also U2.30 (GPIO19); no longer U2.31 (GPIO20)
- net -sens8: now also U2.31 (GPIO20); no longer U2.32 (GPIO21)
- net -sens9: now also U2.32 (GPIO21); no longer U2.34 (GPIO22)
- net GND: now also J5.2 (Pin_2)
- net at R4.2: now also J5.1 (Pin_1)

Commit message: wip
Parts:
- C13, C17: value 100nF -> 1µF
Changed lines of the file:
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@@
       (effects (font (size 1.27 1.27)) (justify left))
     )
-    (property "Value" "100nF" (id 1) (at 220.98 115.57 0)
+    (property "Value" "1µF" (id 1) (at 220.98 115.57 0)
       (effects (font (size 1.27 1.27)) (justify left))
     )
@@
       (effects (font (size 1.27 1.27)) (justify left))
     )
-    (property "Value" "100nF" (id 1) (at 237.49 90.17 0)
+    (property "Value" "1µF" (id 1) (at 237.49 90.17 0)
       (effects (font (size 1.27 1.27)) (justify left))
     )
@@
     )
     (path "/89eff69f-6271-4e79-94af-7c15b44d0ef0"
-      (reference "C13") (unit 1) (value "100nF") (footprint "Capacitor_SMD:C_0603_1608Metric")
+      (reference "C13") (unit 1) (value "1µF") (footprint "Capacitor_SMD:C_0603_1608Metric")
     )
     (path "/604e75b9-6c5e-4ae1-8f98-6c6b586c6f59"
@@
     )
     (path "/8b7347cc-133e-45f8-b286-23264fb7b5ca"
-      (reference "C17") (unit 1) (value "100nF") (footprint "Capacitor_SMD:C_0603_1608Metric")
+      (reference "C17") (unit 1) (value "1µF") (footprint "Capacitor_SMD:C_0603_1608Metric")
     )
     (path "/f609e956-3b1d-49c0-8d35-2704941e274b"

Commit message: wip
Parts:
- added R35, R36: 10R, Resistor_SMD:R_0603_1608Metric, symbol Device:R
Connections:
- net VBUS: now also R35.1, R36.1; no longer D1.2 (A)
- new net: D1.2 (A), R35.2, R36.2
Other:
- moved on the sheet: D1
Changed lines of the file:
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@@
   (junction (at 256.54 33.02) (diameter 0) (color 0 0 0 0)
   )
+  (junction (at 30.48 67.31) (diameter 0) (color 0 0 0 0)
+  )
   (junction (at 167.64 113.03) (diameter 0) (color 0 0 0 0)
   )
+  (junction (at 30.48 60.96) (diameter 0) (color 0 0 0 0)
+  )
   (junction (at 152.4 97.79) (diameter 0) (color 0 0 0 0)
   )
@@
   (junction (at 80.01 57.15) (diameter 0) (color 0 0 0 0)
   )
-  (junction (at 31.75 67.31) (diameter 0) (color 0 0 0 0)
-  )
   (junction (at 165.1 57.15) (diameter 0) (color 0 0 0 0)
   )
@@
   (junction (at 139.7 57.15) (diameter 0) (color 0 0 0 0)
   )
+  (junction (at 38.1 60.96) (diameter 0) (color 0 0 0 0)
+  )
   (junction (at 137.16 57.15) (diameter 0) (color 0 0 0 0)
   )
@@
     (stroke (width 0) (type default) (color 0 0 0 0))
   )
+  (wire (pts (xy 38.1 60.96) (xy 38.1 67.31))
+    (stroke (width 0) (type default) (color 0 0 0 0))
+  )
   (wire (pts (xy 139.7 64.77) (xy 139.7 87.63))
     (stroke (width 0) (type default) (color 0 0 0 0))
@@
     (stroke (width 0) (type default) (color 0 0 0 0))
   )
-  (wire (pts (xy 43.18 67.31) (xy 45.72 67.31))
+  (wire (pts (xy 45.72 60.96) (xy 48.26 60.96))
     (stroke (width 0) (type default) (color 0 0 0 0))
   )
@@
     (stroke (width 0) (type default) (color 0 0 0 0))
   )
-  (wire (pts (xy 30.48 67.31) (xy 31.75 67.31))
+  (wire (pts (xy 30.48 67.31) (xy 30.48 60.96))
     (stroke (width 0) (type default) (color 0 0 0 0))
   )
@@
     (stroke (width 0) (type default) (color 0 0 0 0))
   )
-  (wire (pts (xy 31.75 67.31) (xy 35.56 67.31))
-    (stroke (width 0) (type default) (color 0 0 0 0))
-  )
   (wire (pts (xy 218.44 50.8) (xy 218.44 44.45))
     (stroke (width 0) (type default) (color 0 0 0 0))
@@
     (pin "1")
   )
+  (symbol (lib_id "Device:R") (at 34.29 60.96 90) (unit 1)
+    (in_bom yes) (on_board yes)
+    (property "Reference" "R35" (id 0) (at 33.02 58.42 90))
+    (property "Value" "10R" (id 1) (at 34.29 60.96 90))
+    (property "Footprint" "Resistor_SMD:R_0603_1608Metric" (id 2) (at 34.29 62.738 90)
+      (effects (font (size 1.27 1.27)) hide)
+    )
+    (property "Datasheet" "~" (id 3) (at 34.29 60.96 0)
+      (effects (font (size 1.27 1.27)) hide)
+    )
+    (pin "1")
+    (pin "2")
+  )
   (symbol (lib_id "Device:C") (at 237.49 113.03 0) (unit 1)
     (in_bom yes) (on_board yes)
@@
     (pin "1")
   )
+  (symbol (lib_id "Device:R") (at 34.29 67.31 90) (unit 1)
+    (in_bom yes) (on_board yes)
+    (property "Reference" "R36" (id 0) (at 33.02 64.77 90))
+    (property "Value" "10R" (id 1) (at 34.29 67.31 90))
+    (property "Footprint" "Resistor_SMD:R_0603_1608Metric" (id 2) (at 34.29 69.088 90)
+      (effects (font (size 1.27 1.27)) hide)
+    )
+    (property "Datasheet" "~" (id 3) (at 34.29 67.31 0)
+      (effects (font (size 1.27 1.27)) hide)
+    )
+    (pin "1")
+    (pin "2")
+  )
   (symbol (lib_id "Device:C") (at 212.09 29.21 180) (unit 1)
     (in_bom yes) (on_board yes)
@@
     (pin "2")
   )
-  (symbol (lib_id "Device:D_Filled") (at 39.37 67.31 180) (unit 1)
+  (symbol (lib_id "Device:D_Filled") (at 41.91 60.96 180) (unit 1)
     (in_bom yes) (on_board yes) (fields_autoplaced)
-    (property "Reference" "D1" (id 0) (at 39.37 60.96 0))
-    (property "Value" "BAT54W" (id 1) (at 39.37 63.5 0))
-    (property "Footprint" "Diode_SMD:D_SOD-323" (id 2) (at 39.37 67.31 0)
+    (property "Reference" "D1" (id 0) (at 41.91 54.61 0))
+    (property "Value" "BAT54W" (id 1) (at 41.91 57.15 0))
+    (property "Footprint" "Diode_SMD:D_SOD-323" (id 2) (at 41.91 60.96 0)
       (effects (font (size 1.27 1.27)) hide)
     )
-    (property "Datasheet" "~" (id 3) (at 39.37 67.31 0)
+    (property "Datasheet" "~" (id 3) (at 41.91 60.96 0)
       (effects (font (size 1.27 1.27)) hide)
     )
@@
     (pin "2")
   )
-  (symbol (lib_id "power:+24V") (at 45.72 67.31 0) (unit 1)
+  (symbol (lib_id "power:+24V") (at 48.26 60.96 0) (unit 1)
     (in_bom yes) (on_board yes) (fields_autoplaced)
-    (property "Reference" "#PWR010" (id 0) (at 45.72 71.12 0)
+    (property "Reference" "#PWR010" (id 0) (at 48.26 64.77 0)
       (effects (font (size 1.27 1.27)) hide)
     )
-    (property "Value" "+24V" (id 1) (at 45.72 62.23 0))
-    (property "Footprint" "" (id 2) (at 45.72 67.31 0)
+    (property "Value" "+24V" (id 1) (at 48.26 55.88 0))
+    (property "Footprint" "" (id 2) (at 48.26 60.96 0)
       (effects (font (size 1.27 1.27)) hide)
     )
-    (property "Datasheet" "" (id 3) (at 45.72 67.31 0)
+    (property "Datasheet" "" (id 3) (at 48.26 60.96 0)
       (effects (font (size 1.27 1.27)) hide)
     )
@@
     (pin "1")
   )
-  (symbol (lib_id "power:VBUS") (at 31.75 67.31 0) (unit 1)
+  (symbol (lib_id "power:VBUS") (at 30.48 60.96 0) (unit 1)
     (in_bom yes) (on_board yes) (fields_autoplaced)
-    (property "Reference" "#PWR05" (id 0) (at 31.75 71.12 0)
+    (property "Reference" "#PWR05" (id 0) (at 30.48 64.77 0)
       (effects (font (size 1.27 1.27)) hide)
     )
-    (property "Value" "VBUS" (id 1) (at 31.75 62.23 0))
-    (property "Footprint" "" (id 2) (at 31.75 67.31 0)
+    (property "Value" "VBUS" (id 1) (at 30.48 55.88 0))
+    (property "Footprint" "" (id 2) (at 30.48 60.96 0)
       (effects (font (size 1.27 1.27)) hide)
     )
-    (property "Datasheet" "" (id 3) (at 31.75 67.31 0)
+    (property "Datasheet" "" (id 3) (at 30.48 60.96 0)
       (effects (font (size 1.27 1.27)) hide)
     )
@@
   )
   (symbol (lib_id "Bergi:AP63357Q") (at 196.85 34.29 0) (unit 1)
-    (in_bom yes) (on_board yes) (fields_autoplaced)
+    (in_bom yes) (on_board yes)
     (property "Reference" "U3" (id 0) (at 196.85 21.59 0))
     (property "Value" "AP63357Q" (id 1) (at 196.85 24.13 0))
@@
       (reference "R34") (unit 1) (value "1k") (footprint "Resistor_SMD:R_0603_1608Metric")
     )
+    (path "/0399bf47-770b-4c30-8650-a3df6edc8cf3"
+      (reference "R35") (unit 1) (value "10R") (footprint "Resistor_SMD:R_0603_1608Metric")
+    )
+    (path "/33416c7e-4c02-4369-9042-682a4a026c19"
+      (reference "R36") (unit 1) (value "10R") (footprint "Resistor_SMD:R_0603_1608Metric")
+    )
     (path "/dc148993-ceb9-4294-a55a-f51f3401b421"

Commit message: wip
Parts:
- added L2: 1µ, Inductor_SMD:L_0805_2012Metric, symbol Device:L_Ferrite
Connections:
- net +24V: now also L2.2; no longer C6.2, U3.1 (VIN), U3.2 (EN)
- new net: C6.2, L2.1, U3.1 (VIN), U3.2 (EN)
Changed lines of the file:
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@@
   (junction (at 132.08 80.01) (diameter 0) (color 0 0 0 0)
   )
-  (junction (at 176.53 31.75) (diameter 0) (color 0 0 0 0)
-  )
   (junction (at 186.69 31.75) (diameter 0) (color 0 0 0 0)
   )
@@
   (junction (at 237.49 40.64) (diameter 0) (color 0 0 0 0)
   )
+  (junction (at 176.53 31.75) (diameter 0) (color 0 0 0 0)
+  )
   (junction (at 139.7 57.15) (diameter 0) (color 0 0 0 0)
   )
@@
     (stroke (width 0) (type default) (color 0 0 0 0))
   )
-  (wire (pts (xy 176.53 29.21) (xy 176.53 31.75))
-    (stroke (width 0) (type default) (color 0 0 0 0))
-  )
   (wire (pts (xy 38.1 171.45) (xy 38.1 177.8))
     (stroke (width 0) (type default) (color 0 0 0 0))
@@
     (stroke (width 0) (type default) (color 0 0 0 0))
   )
+  (wire (pts (xy 163.83 31.75) (xy 165.1 31.75))
+    (stroke (width 0) (type default) (color 0 0 0 0))
+  )
   (wire (pts (xy 139.7 87.63) (xy 180.34 87.63))
     (stroke (width 0) (type default) (color 0 0 0 0))
@@
     (stroke (width 0) (type default) (color 0 0 0 0))
   )
+  (wire (pts (xy 172.72 31.75) (xy 176.53 31.75))
+    (stroke (width 0) (type default) (color 0 0 0 0))
+  )
   (wire (pts (xy 121.92 44.45) (xy 142.24 44.45))
     (stroke (width 0) (type default) (color 0 0 0 0))
@@
     (pin "2")
   )
+  (symbol (lib_id "Device:L_Ferrite") (at 168.91 31.75 270) (unit 1)
+    (in_bom yes) (on_board yes) (fields_autoplaced)
+    (property "Reference" "L2" (id 0) (at 168.91 26.67 90))
+    (property "Value" "1µ" (id 1) (at 168.91 29.21 90))
+    (property "Footprint" "Inductor_SMD:L_0805_2012Metric" (id 2) (at 168.91 31.75 0)
+      (effects (font (size 1.27 1.27)) hide)
+    )
+    (property "Datasheet" "~" (id 3) (at 168.91 31.75 0)
+      (effects (font (size 1.27 1.27)) hide)
+    )
+    (pin "1")
+    (pin "2")
+  )
   (symbol (lib_id "Device:L") (at 222.25 33.02 90) (unit 1)
     (in_bom yes) (on_board yes)
@@
     (pin "2")
   )
+  (symbol (lib_id "power:+24V") (at 163.83 31.75 0) (unit 1)
+    (in_bom yes) (on_board yes) (fields_autoplaced)
+    (property "Reference" "#PWR024" (id 0) (at 163.83 35.56 0)
+      (effects (font (size 1.27 1.27)) hide)
+    )
+    (property "Value" "+24V" (id 1) (at 163.83 26.67 0))
+    (property "Footprint" "" (id 2) (at 163.83 31.75 0)
+      (effects (font (size 1.27 1.27)) hide)
+    )
+    (property "Datasheet" "" (id 3) (at 163.83 31.75 0)
+      (effects (font (size 1.27 1.27)) hide)
+    )
+    (pin "1")
+  )
   (symbol (lib_id "Device:C") (at 38.1 184.15 0) (unit 1)
     (in_bom yes) (on_board yes) (fields_autoplaced)
@@
     (pin "1")
   )
-  (symbol (lib_id "power:+24V") (at 176.53 29.21 0) (unit 1)
-    (in_bom yes) (on_board yes) (fields_autoplaced)
-    (property "Reference" "#PWR024" (id 0) (at 176.53 33.02 0)
-      (effects (font (size 1.27 1.27)) hide)
-    )
-    (property "Value" "+24V" (id 1) (at 176.53 24.13 0))
-    (property "Footprint" "" (id 2) (at 176.53 29.21 0)
-      (effects (font (size 1.27 1.27)) hide)
-    )
-    (property "Datasheet" "" (id 3) (at 176.53 29.21 0)
-      (effects (font (size 1.27 1.27)) hide)
-    )
-    (pin "1")
-  )
   (symbol (lib_id "Device:C") (at 251.46 87.63 0) (unit 1)
     (in_bom yes) (on_board yes)
@@
       (reference "#PWR023") (unit 1) (value "GND") (footprint "")
     )
-    (path "/bbeea750-fdbd-4dd6-92f4-55b6384f34ab"
+    (path "/766e65c3-bef8-41f5-90d0-36521263f4d3"
       (reference "#PWR024") (unit 1) (value "+24V") (footprint "")
     )
@@
       (reference "L1") (unit 1) (value "4.7u") (footprint "Inductor_SMD:L_1008_2520Metric")
     )
+    (path "/21efa11b-39d3-4f53-ba2c-acb613f9de54"
+      (reference "L2") (unit 1) (value "1µ") (footprint "Inductor_SMD:L_0805_2012Metric")
+    )
     (path "/e24d31a3-fcfc-40dd-92eb-52ff5fe4874c"
