File: DualLevelSensor/DualLevelSensor.kicad_sch (KiCad schematic)
At the start: 95 parts, among them J1 USB_B_Micro, J2 Conn_01x03, J3 Conn_01x03, J4 Conn_01x03, J5 Conn_01x02, K1 capPad, K10 capPad, K11 capPad, K12 capPad, K13 capPad, K14 capPad, K15 capPad, K16 capPad, K17 capPad, K18 capPad, K19 capPad, K2 capPad, K20 capPad, K21 capPad, K22 capPad, K3 capPad, K4 capPad, K5 capPad, K6 capPad, K7 capPad, K8 capPad, K9 capPad, U1 W25Q16JVUXIQ, U2 RP2040, U3 AP63357Q, Y1 12Mhz

Commit message: wip
Parts:
- C1, C2: value 12p -> 15p
Changed lines of the file:
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@@
       (effects (font (size 1.27 1.27)) (justify left))
     )
-    (property "Value" "12p" (id 1) (at 17.78 186.69 0)
+    (property "Value" "15p" (id 1) (at 17.78 186.69 0)
       (effects (font (size 1.27 1.27)) (justify left))
     )
@@
   )
   (symbol (lib_id "Device:C") (at 38.1 184.15 0) (unit 1)
-    (in_bom yes) (on_board yes) (fields_autoplaced)
-    (property "Reference" "C2" (id 0) (at 41.91 182.8799 0)
-      (effects (font (size 1.27 1.27)) (justify left))
-    )
-    (property "Value" "12p" (id 1) (at 41.91 185.4199 0)
+    (in_bom yes) (on_board yes)
+    (property "Reference" "C2" (id 0) (at 40.64 182.88 0)
+      (effects (font (size 1.27 1.27)) (justify left))
+    )
+    (property "Value" "15p" (id 1) (at 40.64 185.42 0)
       (effects (font (size 1.27 1.27)) (justify left))
     )
@@
     )
     (path "/75676d7a-1271-4373-bb3f-f93fce0f46d5"
-      (reference "C1") (unit 1) (value "12p") (footprint "Capacitor_SMD:C_0603_1608Metric")
+      (reference "C1") (unit 1) (value "15p") (footprint "Capacitor_SMD:C_0603_1608Metric")
     )
     (path "/776eb652-ebea-46bf-8d29-7e83d0799b9c"
-      (reference "C2") (unit 1) (value "12p") (footprint "Capacitor_SMD:C_0603_1608Metric")
+      (reference "C2") (unit 1) (value "15p") (footprint "Capacitor_SMD:C_0603_1608Metric")
     )
     (path "/a31d64cc-acc4-4691-aca7-f8cc3165559d"
