File: SoilMoistureSensor/Pcb/soilMoistureSensor.kicad_sch (KiCad schematic)
At the start: 44 parts

Commit message: - wip
Parts:
- removed D?: Green, LED_SMD:LED_0603_1608Metric, symbol Device:LED_Filled
- removed R?: 10k, Resistor_SMD:R_0603_1608Metric, symbol Device:R
- removed R?: 470R, Resistor_SMD:R_0603_1608Metric, symbol Device:R
- removed R?: 5.6k, Resistor_SMD:R_0603_1608Metric, symbol Device:R
- added C?: 1µF, Capacitor_SMD:C_0603_1608Metric, symbol Device:C
- added D?: Green, LED_SMD:LED_0603_1608Metric, symbol Device:LED_Filled
- added L?: 600R, symbol Device:L_Ferrite
- added R?: 470R, Resistor_SMD:R_0603_1608Metric, symbol Device:R
- added R?: 5.6k, Resistor_SMD:R_0603_1608Metric, symbol Device:R
- added R?: 10k, Resistor_SMD:R_0603_1608Metric, symbol Device:R
Connections:
- net +3V3: now also L?.2; no longer U?.43 (ADC_AVDD)
- net GND: now also C?.2, D?.1 (K), R?.2
- net UART0: now also U?.6 (GPIO4), U?.7 (GPIO5); no longer U?.40 (GPIO28_ADC2), U?.41 (GPIO29_ADC3)
- net UART1: now also U?.2 (GPIO0), U?.3 (GPIO1); no longer U?.36 (GPIO24), U?.37 (GPIO25)
- net VBUS: now also R?.1
- net EN_Sens: now reaches U?.11 (GPIO8)
- net at U?.13 (GPIO10): now also R?.1
- net at U?.14 (GPIO11): now also R?.1, R?.2
- net Sens_Clk: now reaches U?.32 (GPIO21)
- net Csens: now reaches U?.38 (GPIO26_ADC0)
- net GAIN: now reaches U?.9 (GPIO7)
- new net: C?.1, L?.1, U?.43 (ADC_AVDD)
- new net: D?.2 (A), R?.2
Other:
- sheet capSens ports: added EN_Sens, GAIN; removed none

Commit message: wip
Parts:
- gave numbers to parts that had none: 46
Connections:
- net GAIN: no longer names the net of U2.9 (GPIO7)
Other:
- sheet capSens ports: added GAIN_NCS, GAIN_U/ND; removed GAIN

Commit message: wip
Connections:
- net EN_Sens: now also U2.13 (GPIO10); no longer U2.11 (GPIO8)
- net at R5.1: now also U2.16 (GPIO13); no longer U2.13 (GPIO10)
- net GAIN_NCS: now reaches U2.12 (GPIO9)
- net at R6.2, R7.1: now also U2.17 (GPIO14); no longer U2.14 (GPIO11)
- new net GAIN_U/ND: U2.11 (GPIO8)

Commit message: wip
Parts:
- added R?: 10k, Resistor_SMD:R_0603_1608Metric, symbol Device:R
- added R?: 4.3k, Resistor_SMD:R_0603_1608Metric, symbol Device:R
- L1: footprint (none) -> Inductor_SMD:L_0603_1608Metric
Connections:
- net GND: now also R?.2
- net Sens_Clk: now also R?.1, R?.2; no longer U2.32 (GPIO21)
- new net: R?.1, U2.32 (GPIO21)
Other:
- moved on the sheet: D2, R5, R6, R7

Commit message: wip
Parts:
- gave numbers to parts that had none: 2
Changed lines of the file:
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@@
   (symbol (lib_id "power:GND") (at 115.57 134.62 0) (unit 1)
     (in_bom yes) (on_board yes)
-    (property "Reference" "#PWR?" (id 0) (at 115.57 140.97 0)
+    (property "Reference" "#PWR0116" (id 0) (at 115.57 140.97 0)
       (effects (font (size 1.27 1.27)) hide)
     )
@@
   (symbol (lib_id "Device:R") (at 115.57 130.81 0) (unit 1)
     (in_bom yes) (on_board yes)
-    (property "Reference" "R?" (id 0) (at 113.03 130.81 90)
+    (property "Reference" "R30" (id 0) (at 113.03 130.81 90)
       (effects (font (size 1.27 1.27)) (justify right))
     )
@@
   (symbol (lib_id "Device:R") (at 115.57 123.19 0) (unit 1)
     (in_bom yes) (on_board yes)
-    (property "Reference" "R?" (id 0) (at 113.03 123.19 90)
+    (property "Reference" "R29" (id 0) (at 113.03 123.19 90)
       (effects (font (size 1.27 1.27)) (justify right))
     )
@@
     )
     (path "/032f2f6d-38fb-4cfd-b1e2-8ce4fd3468ff"
-      (reference "#PWR?") (unit 1) (value "GND") (footprint "")
+      (reference "#PWR0116") (unit 1) (value "GND") (footprint "")
     )
     (path "/bc1c1471-bf88-411b-af46-c3b0c9f2824d"
@@
       (reference "R28") (unit 1) (value "20k") (footprint "Resistor_SMD:R_0603_1608Metric")
     )
+    (path "/e54d112e-51e3-4af7-babc-96386e4bdecc"
+      (reference "R29") (unit 1) (value "4.3k") (footprint "Resistor_SMD:R_0603_1608Metric")
+    )
     (path "/50ee3373-70e7-44df-a412-82d31b286840"
-      (reference "R?") (unit 1) (value "10k") (footprint "Resistor_SMD:R_0603_1608Metric")
-    )
-    (path "/e54d112e-51e3-4af7-babc-96386e4bdecc"
-      (reference "R?") (unit 1) (value "4.3k") (footprint "Resistor_SMD:R_0603_1608Metric")
+      (reference "R30") (unit 1) (value "10k") (footprint "Resistor_SMD:R_0603_1608Metric")
     )
     (path "/596a3a1e-6f3a-4b5d-9915-c32063e13f7e"

Commit message: wip
Parts:
- added R31, R32: 20R, Resistor_SMD:R_0603_1608Metric, symbol Device:R
Connections:
- net VBUS: now also R31.2, R32.2; no longer D1.2 (A)
- new net: D1.2 (A), R31.1, R32.1
Other:
- moved on the sheet: D1
Changed lines of the file:
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@@
 (kicad_sch (version 20211123) (generator eeschema)
   (paper "A4")
-  (junction (at 34.29 68.58) (diameter 0) (color 0 0 0 0)
-  )
   (junction (at 43.18 48.26) (diameter 0) (color 0 0 0 0)
   )
@@
   (junction (at 40.64 179.07) (diameter 0) (color 0 0 0 0)
   )
+  (junction (at 33.02 63.5) (diameter 0) (color 0 0 0 0)
+  )
   (junction (at 214.63 34.29) (diameter 0) (color 0 0 0 0)
   )
@@
   (junction (at 212.09 45.72) (diameter 0) (color 0 0 0 0)
   )
+  (junction (at 40.64 63.5) (diameter 0) (color 0 0 0 0)
+  )
   (junction (at 115.57 127) (diameter 0) (color 0 0 0 0)
   )
@@
   (junction (at 189.23 33.02) (diameter 0) (color 0 0 0 0)
   )
+  (junction (at 33.02 68.58) (diameter 0) (color 0 0 0 0)
+  )
   (junction (at 82.55 55.88) (diameter 0) (color 0 0 0 0)
   )
@@
     (stroke (width 0) (type default) (color 0 0 0 0))
   )
-  (wire (pts (xy 34.29 68.58) (xy 38.1 68.58))
-    (stroke (width 0) (type default) (color 0 0 0 0))
-  )
   (wire (pts (xy 36.83 179.07) (xy 40.64 179.07))
     (stroke (width 0) (type default) (color 0 0 0 0))
@@
     (stroke (width 0) (type default) (color 0 0 0 0))
   )
-  (wire (pts (xy 33.02 68.58) (xy 34.29 68.58))
+  (wire (pts (xy 33.02 68.58) (xy 33.02 63.5))
     (stroke (width 0) (type default) (color 0 0 0 0))
   )
@@
     (stroke (width 0) (type default) (color 0 0 0 0))
   )
-  (wire (pts (xy 45.72 68.58) (xy 48.26 68.58))
+  (wire (pts (xy 48.26 63.5) (xy 52.07 63.5))
     (stroke (width 0) (type default) (color 0 0 0 0))
   )
@@
   )
   (wire (pts (xy 106.68 30.48) (xy 106.68 33.02))
+    (stroke (width 0) (type default) (color 0 0 0 0))
+  )
+  (wire (pts (xy 40.64 63.5) (xy 40.64 68.58))
     (stroke (width 0) (type default) (color 0 0 0 0))
   )
@@
     (pin "2")
   )
-  (symbol (lib_id "Device:D_Filled") (at 41.91 68.58 180) (unit 1)
-    (in_bom yes) (on_board yes) (fields_autoplaced)
-    (property "Reference" "D1" (id 0) (at 41.91 62.23 0))
-    (property "Value" "BAT54W" (id 1) (at 41.91 64.77 0))
-    (property "Footprint" "Diode_SMD:D_SOD-323" (id 2) (at 41.91 68.58 0)
-      (effects (font (size 1.27 1.27)) hide)
-    )
-    (property "Datasheet" "~" (id 3) (at 41.91 68.58 0)
+  (symbol (lib_id "Device:D_Filled") (at 44.45 63.5 180) (unit 1)
+    (in_bom yes) (on_board yes) (fields_autoplaced)
+    (property "Reference" "D1" (id 0) (at 44.45 57.15 0))
+    (property "Value" "BAT54W" (id 1) (at 44.45 59.69 0))
+    (property "Footprint" "Diode_SMD:D_SOD-323" (id 2) (at 44.45 63.5 0)
+      (effects (font (size 1.27 1.27)) hide)
+    )
+    (property "Datasheet" "~" (id 3) (at 44.45 63.5 0)
       (effects (font (size 1.27 1.27)) hide)
     )
@@
     (pin "2")
   )
-  (symbol (lib_id "power:VBUS") (at 34.29 68.58 0) (unit 1)
-    (in_bom yes) (on_board yes) (fields_autoplaced)
-    (property "Reference" "#PWR05" (id 0) (at 34.29 72.39 0)
-      (effects (font (size 1.27 1.27)) hide)
-    )
-    (property "Value" "VBUS" (id 1) (at 34.29 63.5 0))
-    (property "Footprint" "" (id 2) (at 34.29 68.58 0)
-      (effects (font (size 1.27 1.27)) hide)
-    )
-    (property "Datasheet" "" (id 3) (at 34.29 68.58 0)
+  (symbol (lib_id "power:VBUS") (at 33.02 63.5 0) (unit 1)
+    (in_bom yes) (on_board yes) (fields_autoplaced)
+    (property "Reference" "#PWR05" (id 0) (at 33.02 67.31 0)
+      (effects (font (size 1.27 1.27)) hide)
+    )
+    (property "Value" "VBUS" (id 1) (at 33.02 58.42 0))
+    (property "Footprint" "" (id 2) (at 33.02 63.5 0)
+      (effects (font (size 1.27 1.27)) hide)
+    )
+    (property "Datasheet" "" (id 3) (at 33.02 63.5 0)
       (effects (font (size 1.27 1.27)) hide)
     )
@@
     )
     (pin "1")
+  )
+  (symbol (lib_id "Device:R") (at 36.83 63.5 270) (unit 1)
+    (in_bom yes) (on_board yes)
+    (property "Reference" "R31" (id 0) (at 36.83 60.96 90)
+      (effects (font (size 1.27 1.27)) (justify right))
+    )
+    (property "Value" "20R" (id 1) (at 38.1 63.5 90)
+      (effects (font (size 1.27 1.27)) (justify right))
+    )
+    (property "Footprint" "Resistor_SMD:R_0603_1608Metric" (id 2) (at 36.83 61.722 90)
+      (effects (font (size 1.27 1.27)) hide)
+    )
+    (property "Datasheet" "~" (id 3) (at 36.83 63.5 0)
+      (effects (font (size 1.27 1.27)) hide)
+    )
+    (pin "1")
+    (pin "2")
   )
   (symbol (lib_id "Device:C") (at 237.49 88.9 0) (unit 1)
@@
     (pin "9")
   )
+  (symbol (lib_id "Device:R") (at 36.83 68.58 270) (unit 1)
+    (in_bom yes) (on_board yes)
+    (property "Reference" "R32" (id 0) (at 36.83 66.04 90)
+      (effects (font (size 1.27 1.27)) (justify right))
+    )
+    (property "Value" "20R" (id 1) (at 38.1 68.58 90)
+      (effects (font (size 1.27 1.27)) (justify right))
+    )
+    (property "Footprint" "Resistor_SMD:R_0603_1608Metric" (id 2) (at 36.83 66.802 90)
+      (effects (font (size 1.27 1.27)) hide)
+    )
+    (property "Datasheet" "~" (id 3) (at 36.83 68.58 0)
+      (effects (font (size 1.27 1.27)) hide)
+    )
+    (pin "1")
+    (pin "2")
+  )
   (symbol (lib_id "power:GND") (at 251.46 49.53 0) (unit 1)
     (in_bom yes) (on_board yes) (fields_autoplaced)
@@
     (pin "1")
   )
-  (symbol (lib_id "power:+24V") (at 48.26 68.58 0) (unit 1)
-    (in_bom yes) (on_board yes) (fields_autoplaced)
-    (property "Reference" "#PWR010" (id 0) (at 48.26 72.39 0)
-      (effects (font (size 1.27 1.27)) hide)
-    )
-    (property "Value" "+24V" (id 1) (at 48.26 63.5 0))
-    (property "Footprint" "" (id 2) (at 48.26 68.58 0)
-      (effects (font (size 1.27 1.27)) hide)
-    )
-    (property "Datasheet" "" (id 3) (at 48.26 68.58 0)
+  (symbol (lib_id "power:+24V") (at 52.07 63.5 0) (unit 1)
+    (in_bom yes) (on_board yes) (fields_autoplaced)
+    (property "Reference" "#PWR010" (id 0) (at 52.07 67.31 0)
+      (effects (font (size 1.27 1.27)) hide)
+    )
+    (property "Value" "+24V" (id 1) (at 52.07 58.42 0))
+    (property "Footprint" "" (id 2) (at 52.07 63.5 0)
+      (effects (font (size 1.27 1.27)) hide)
+    )
+    (property "Datasheet" "" (id 3) (at 52.07 63.5 0)
       (effects (font (size 1.27 1.27)) hide)
     )
@@
     )
     (path "/12dbac44-96c1-4a7b-b3a4-dfcfee935f2c/4d12ae1c-90f2-4528-b173-1620fd6e7082"
-      (reference "J8") (unit 1) (value "Conn_01x01") (footprint "TestPoint:TestPoint_Pad_D2.0mm")
+      (reference "J8") (unit 1) (value "Conn_01x01") (footprint "TestPoint:TestPoint_Pad_D1.5mm")
     )
     (path "/12dbac44-96c1-4a7b-b3a4-dfcfee935f2c/0dd2ded8-82a6-416a-b3fd-7e4c0d675722"
-      (reference "J9") (unit 1) (value "Conn_01x01") (footprint "TestPoint:TestPoint_Pad_D2.0mm")
+      (reference "J9") (unit 1) (value "Conn_01x01") (footprint "TestPoint:TestPoint_Pad_D1.5mm")
     )
     (path "/0e2f331e-8c31-47e8-a8ee-5c7070b98ce6"
@@
       (reference "R30") (unit 1) (value "10k") (footprint "Resistor_SMD:R_0603_1608Metric")
     )
+    (path "/522d73ad-0a13-4dba-b4bd-3180e8c1e21f"
+      (reference "R31") (unit 1) (value "20R") (footprint "Resistor_SMD:R_0603_1608Metric")
+    )
+    (path "/5acf3507-79d8-4b9a-873c-83967be97f38"
+      (reference "R32") (unit 1) (value "20R") (footprint "Resistor_SMD:R_0603_1608Metric")
+    )
     (path "/596a3a1e-6f3a-4b5d-9915-c32063e13f7e"

Commit message: wip
Connections:
- net EN_Sens: now also U2.37 (GPIO25); no longer U2.13 (GPIO10)
- net GAIN_NCS: now also U2.28 (GPIO17); no longer U2.12 (GPIO9)
- net GAIN_U/ND: now also U2.27 (GPIO16); no longer U2.11 (GPIO8)
- net at R6.2, R7.1: now also U2.4 (GPIO2); no longer U2.17 (GPIO14)
Other:
- moved on the sheet: R29, R30, R6, R7

Commit message: wip
Parts:
- added L4: 1µ, Inductor_SMD:L_0805_2012Metric, symbol Device:L_Ferrite
Connections:
- net +24V: now also L4.2; no longer C5.2, U3.1 (VIN), U3.2 (EN)
- new net: C5.2, L4.1, U3.1 (VIN), U3.2 (EN)
Changed lines of the file:
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@@
-    (stroke (width 0) (type default) (color 0 0 0 0))
-  )
-  (wire (pts (xy 179.07 30.48) (xy 179.07 33.02))
     (stroke (width 0) (type default) (color 0 0 0 0))
   )
@@
     (stroke (width 0) (type default) (color 0 0 0 0))
   )
+  (wire (pts (xy 175.26 33.02) (xy 179.07 33.02))
+    (stroke (width 0) (type default) (color 0 0 0 0))
+  )
   (wire (pts (xy 220.98 52.07) (xy 220.98 45.72))
     (stroke (width 0) (type default) (color 0 0 0 0))
@@
   )
   (wire (pts (xy 52.07 77.47) (xy 52.07 76.2))
+    (stroke (width 0) (type default) (color 0 0 0 0))
+  )
+  (wire (pts (xy 166.37 33.02) (xy 167.64 33.02))
     (stroke (width 0) (type default) (color 0 0 0 0))
   )
@@
     )
     (pin "1")
+  )
+  (symbol (lib_id "Device:L_Ferrite") (at 171.45 33.02 270) (unit 1)
+    (in_bom yes) (on_board yes) (fields_autoplaced)
+    (property "Reference" "L4" (id 0) (at 171.45 27.94 90))
+    (property "Value" "1µ" (id 1) (at 171.45 30.48 90))
+    (property "Footprint" "Inductor_SMD:L_0805_2012Metric" (id 2) (at 171.45 33.02 0)
+      (effects (font (size 1.27 1.27)) hide)
+    )
+    (property "Datasheet" "~" (id 3) (at 171.45 33.02 0)
+      (effects (font (size 1.27 1.27)) hide)
+    )
+    (pin "1")
+    (pin "2")
   )
   (symbol (lib_id "Device:C") (at 228.6 88.9 0) (unit 1)
@@
     (pin "2")
   )
+  (symbol (lib_id "power:+24V") (at 166.37 33.02 0) (unit 1)
+    (in_bom yes) (on_board yes) (fields_autoplaced)
+    (property "Reference" "#PWR028" (id 0) (at 166.37 36.83 0)
+      (effects (font (size 1.27 1.27)) hide)
+    )
+    (property "Value" "+24V" (id 1) (at 166.37 27.94 0))
+    (property "Footprint" "" (id 2) (at 166.37 33.02 0)
+      (effects (font (size 1.27 1.27)) hide)
+    )
+    (property "Datasheet" "" (id 3) (at 166.37 33.02 0)
+      (effects (font (size 1.27 1.27)) hide)
+    )
+    (pin "1")
+  )
   (symbol (lib_id "Device:C") (at 25.4 185.42 0) (unit 1)
     (in_bom yes) (on_board yes)
@@
     (pin "2")
     (pin "3")
-  )
-  (symbol (lib_id "power:+24V") (at 179.07 30.48 0) (unit 1)
-    (in_bom yes) (on_board yes) (fields_autoplaced)
-    (property "Reference" "#PWR028" (id 0) (at 179.07 34.29 0)
-      (effects (font (size 1.27 1.27)) hide)
-    )
-    (property "Value" "+24V" (id 1) (at 179.07 25.4 0))
-    (property "Footprint" "" (id 2) (at 179.07 30.48 0)
-      (effects (font (size 1.27 1.27)) hide)
-    )
-    (property "Datasheet" "" (id 3) (at 179.07 30.48 0)
-      (effects (font (size 1.27 1.27)) hide)
-    )
-    (pin "1")
   )
   (symbol (lib_id "power:GND") (at 74.93 36.83 0) (unit 1)
@@
       (reference "#PWR027") (unit 1) (value "+24V") (footprint "")
     )
-    (path "/d1d0a3e9-7f70-4aa1-a68e-7b19254371d0"
+    (path "/ba0f603d-fb98-43f5-a3c6-ec56596bcbd7"
       (reference "#PWR028") (unit 1) (value "+24V") (footprint "")
     )
@@
       (reference "L3") (unit 1) (value "600R") (footprint "Inductor_SMD:L_0603_1608Metric")
     )
+    (path "/138fc1ae-b886-4faa-85e7-f06f356b025d"
+      (reference "L4") (unit 1) (value "1µ") (footprint "Inductor_SMD:L_0805_2012Metric")
+    )
     (path "/a9bd6db7-101e-488d-b0d8-6ad60600008c"
