File: SoilMoistureSensor/Pcb/capSens.kicad_sch (KiCad schematic)
At the start: 47 parts, among them J6 Conn_01x01, J7 Conn_01x01, J8 Conn_01x01, J9 Conn_01x01, U10 74AUC2G66, U11 TLV9002S, U12 MCP4011-xxxxMS, U4 74AUC2G86, U5 MIC5504-2.5YM5, U6 74AUC2G86, U7 74AUC2G08, U8 OPA2356xxDGK, U9 74AUC2G66

Commit message: wip
Parts:
- C24, C28, C29, C31, C32, C35, C36: footprint (none) -> Capacitor_SMD:C_0603_1608Metric
- J6, J7: footprint (none) -> Bergi:dummyPad
- J8, J9: footprint (none) -> TestPoint:TestPoint_Pad_D2.0mm
- L3: footprint (none) -> Inductor_SMD:L_0603_1608Metric
- R13, R14, R15, R16, R17, R18, R19, R20, R21, R22, R23, R24, R25, R26, R27, R28: footprint (none) -> Resistor_SMD:R_0603_1608Metric
- U8: footprint (none) -> Package_SO:MSOP-8_3x3mm_P0.65mm
- renumbered U6 to U4, U4 to U6
Connections:
- net TRI1: now also U7.3, U9.7; no longer U7.7, U9.3
- net TRI2: now also U7.7, U9.3; no longer U7.3, U9.7
- net at U8.1, U8.2 (-): now also U9.2, U9.5; no longer U9.1, U9.5
- net at R20.1: now also U9.6; no longer U9.2
- net at R26.1, R27.2, R28.1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: now also J8.1 (Pin_1)
- net at J9.1 (Pin_1): now also U12.6 (B); no longer U12.3 (A)
- net at U10.5, U8.6 (-), U8.7: now also U10.2; no longer U10.1
- net at R24.1, R25.2, R28.2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: now also U12.3 (A); no longer J8.1 (Pin_1), U12.6 (B)
- net at R14.2, U4.7: now also U7.5; no longer U7.1
- net at R15.2, U4.3: now also U7.2; no longer U7.5
- net at R21.1: now also U9.1; no longer U9.6
- net at R22.1: now also U10.1; no longer U10.2
- new net: U6.3, U7.1, U7.6
Other:
- moved on the sheet: C24, C29, C31, C32, J6, J7, J9, R13, R15, R17, R18, R19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

Commit message: wip
Connections:
- net at U8.1, U8.2 (-): now also U9.1, U9.6; no longer U9.2, U9.5
- net at R20.1: now also U9.5; no longer U9.6
- net at U8.6 (-), U8.7: now also U10.1, U10.6; no longer U10.2, U10.5
- net at R23.1: now also U10.5; no longer U10.6
- net at R21.1: now also U9.2; no longer U9.1
- net at R22.1: now also U10.2; no longer U10.1

Commit message: wip
Parts:
- J8, J9: footprint TestPoint:TestPoint_Pad_D2.0mm -> TestPoint:TestPoint_Pad_D1.5mm
Changed lines of the file:
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@@
       (effects (font (size 1.27 1.27)) (justify left) hide)
     )
-    (property "Footprint" "TestPoint:TestPoint_Pad_D2.0mm" (id 2) (at 245.11 63.5 0)
+    (property "Footprint" "TestPoint:TestPoint_Pad_D1.5mm" (id 2) (at 245.11 63.5 0)
       (effects (font (size 1.27 1.27)) hide)
     )
@@
       (effects (font (size 1.27 1.27)) (justify left) hide)
     )
-    (property "Footprint" "TestPoint:TestPoint_Pad_D2.0mm" (id 2) (at 241.3 100.33 0)
-      (effects (font (size 1.27 1.27)) hide)
-    )
+    (property "Footprint" "TestPoint:TestPoint_Pad_D1.5mm" (id 2) (at 241.3 100.33 0)
+      (effects (font (size 1.27 1.27)) hide)
+    )

Commit message: wip
Parts:
- U12: HTN (none) -> MCP4011T-503E/MS
Changed lines of the file:
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@@
       (effects (font (size 1.27 1.27)) (justify left) hide)
+    )
+    (property "HTN" "MCP4011T-503E/MS" (id 4) (at 255.27 78.74 0)
+      (effects (font (size 1.27 1.27)) hide)
     )
     (pin "1")
