File: sensorNode/sensorNode.kicad_sch (KiCad schematic)
At the start: 50 parts

Commit message: wip
Parts:
- added J? (x2): Conn_01x02, Connector_PinSocket_2.54mm:PinSocket_1x02_P2.54mm_Vertical, symbol Connector_Generic:Conn_01x02
- added R? (x2): 1k, Resistor_SMD:R_0603_1608Metric, symbol Device:R
- L?: value 1µ -> 10µ
Connections:
- net GND: now also J?.2 (Pin_2), J?.2 (Pin_2)
- net DIN1: now reaches U?.14 (GPIO11)
- net DIN1: now also R?.1
- net DIN2: now reaches U?.15 (GPIO12)
- net DIN2: now also R?.1
- net sensorAmp/ecExc+: now reaches U?.17 (GPIO14)
- net sensorAmp/ecExc-: now reaches U?.18 (GPIO15)
- net sensorAmp/PH_R_Exc: now reaches U?.28 (GPIO17)
- net sensorAmp/SDI: now reaches U?.30 (GPIO19)
- net sensorAmp/SDO: now reaches U?.31 (GPIO20)
- net sensorAmp/CS: now reaches U?.32 (GPIO21)
- net sensorAmp/SCK: now reaches U?.34 (GPIO22)
- net sensorAmp/SDA: now reaches U?.36 (GPIO24)
- net sensorAmp/SCL: now reaches U?.37 (GPIO25)
- new net: J?.1 (Pin_1), R?.2 (x2)
Other:
- sheet sensorAmp ports: added CS, PH_R_Exc, SCK, SCL, SDA, SDI, SDO, ecExc+, ecExc-; removed none

Commit message: wip
Parts:
- added H1, H2, H3, H4: MountingHole, MountingHole:MountingHole_3.2mm_M3_DIN965, symbol Mechanical:MountingHole
- L1: renamed from L?; footprint (none) -> Inductor_SMD:L_0603_1608Metric
- gave numbers to parts that had none: 53
Connections:
- net +3V3: no longer L1.2
- new net +3.3VA: L1.2

Commit message: wip
Parts:
- J6, J7: footprint Connector_PinSocket_2.54mm:PinSocket_1x02_P2.54mm_Vertical -> Connector_JST:JST_EH_B2B-EH-A_1x02_P2.50mm_Vertical
Changed lines of the file:
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@@
       (effects (font (size 1.27 1.27)) (justify left))
     )
-    (property "Footprint" "Connector_PinSocket_2.54mm:PinSocket_1x02_P2.54mm_Vertical" (id 2) (at 175.26 100.33 0)
+    (property "Footprint" "Connector_JST:JST_EH_B2B-EH-A_1x02_P2.50mm_Vertical" (id 2) (at 175.26 100.33 0)
       (effects (font (size 1.27 1.27)) hide)
     )
@@
       (effects (font (size 1.27 1.27)) (justify left))
     )
-    (property "Footprint" "Connector_PinSocket_2.54mm:PinSocket_1x02_P2.54mm_Vertical" (id 2) (at 175.26 113.03 0)
+    (property "Footprint" "Connector_JST:JST_EH_B2B-EH-A_1x02_P2.50mm_Vertical" (id 2) (at 175.26 113.03 0)
       (effects (font (size 1.27 1.27)) hide)
     )
@@
       (reference "#PWR0106") (unit 1) (value "GND") (footprint "")
     )
+    (path "/8671f67a-7a0d-4f43-8358-c29ef9469ead/09d05fb7-c215-4b97-959c-aef053489bcf"
+      (reference "#PWR0107") (unit 1) (value "+3.3VA") (footprint "")
+    )
+    (path "/8671f67a-7a0d-4f43-8358-c29ef9469ead/724e0950-55a2-4d6c-9992-c1ea33034899"
+      (reference "#PWR0108") (unit 1) (value "GND") (footprint "")
+    )
     (path "/0692e74b-e302-4a34-90af-db2585783550"
       (reference "C1") (unit 1) (value "12p") (footprint "Capacitor_SMD:C_0603_1608Metric")
@@
       (reference "C40") (unit 1) (value "100nF") (footprint "Capacitor_SMD:C_0603_1608Metric")
     )
+    (path "/8671f67a-7a0d-4f43-8358-c29ef9469ead/0b8a4588-ef44-476d-adee-e382bc10e04a"
+      (reference "C41") (unit 1) (value "100nF") (footprint "Capacitor_SMD:C_0603_1608Metric")
+    )
     (path "/66dc639d-7a71-46bd-817f-6bf6b9796248"
       (reference "D1") (unit 1) (value "BAT54W") (footprint "Diode_SMD:D_SOD-323")
@@
     )
     (path "/6979771c-d22f-452c-b217-491fd4f9d2c2"
-      (reference "J6") (unit 1) (value "Conn_01x02") (footprint "Connector_PinSocket_2.54mm:PinSocket_1x02_P2.54mm_Vertical")
+      (reference "J6") (unit 1) (value "Conn_01x02") (footprint "Connector_JST:JST_EH_B2B-EH-A_1x02_P2.50mm_Vertical")
     )
     (path "/b356c174-35fc-43c2-a045-48c2c655266c"
-      (reference "J7") (unit 1) (value "Conn_01x02") (footprint "Connector_PinSocket_2.54mm:PinSocket_1x02_P2.54mm_Vertical")
+      (reference "J7") (unit 1) (value "Conn_01x02") (footprint "Connector_JST:JST_EH_B2B-EH-A_1x02_P2.50mm_Vertical")
     )
     (path "/8671f67a-7a0d-4f43-8358-c29ef9469ead/1f5174f9-1965-428a-bbfe-1a9fff31937f"

Commit message: wip
Parts:
- removed C4: 1µF, Capacitor_SMD:C_0603_1608Metric, symbol Device:C
- removed L1: 600R, Inductor_SMD:L_0603_1608Metric, symbol Device:L_Ferrite
Connections:
- net +3V3: now also U2.43 (ADC_AVDD)
- net DIN1: now also U2.40 (GPIO28_ADC2); no longer U2.14 (GPIO11)
- net DIN2: now also U2.41 (GPIO29_ADC3); no longer U2.15 (GPIO12)
- net UART0: now also U2.27 (GPIO16), U2.28 (GPIO17); no longer U2.6 (GPIO4), U2.7 (GPIO5)
- net UART1: now also U2.11 (GPIO8), U2.12 (GPIO9); no longer U2.2 (GPIO0), U2.3 (GPIO1)
- net sensorAmp/CS: now also U2.3 (GPIO1); no longer U2.32 (GPIO21)
- net sensorAmp/PH_R_Exc: now also U2.7 (GPIO5); no longer U2.28 (GPIO17)
- net sensorAmp/SCK: now also U2.4 (GPIO2); no longer U2.34 (GPIO22)
- net sensorAmp/SDI: now also U2.5 (GPIO3); no longer U2.30 (GPIO19)
- net sensorAmp/SDO: now also U2.6 (GPIO4); no longer U2.31 (GPIO20)
- net sensorAmp/ecExc+: now also U2.8 (GPIO6); no longer U2.17 (GPIO14)
- net sensorAmp/ecExc-: now also U2.9 (GPIO7); no longer U2.18 (GPIO15)
- net at R8.2, R9.1: now also U2.29 (GPIO18); no longer U2.12 (GPIO9)
- net at R7.1: now also U2.13 (GPIO10); no longer U2.11 (GPIO8)
Other:
- moved on the sheet: D2, R7, R8, R9
