File: sensorNode/sensorNode.kicad_pcb (KiCad board)
At the start: 2 copper layers, 50 x 50 mm, 116 parts, among them J1 USB_B_Micro, J10 Conn_01x04, J11 Conn_01x02, J2 Conn_01x03, J3 Conn_01x02, J4 Conn_01x03, J5 Conn_01x03, J6 Conn_01x02, J7 Conn_01x02, J8 Conn_01x02, J9 Conn_Coaxial, U1 W25Q16JVUXIQ, U2 RP2040, U3 AP63357Q, U4 MCP6001R, U5 TLV9002S, U6 NCS333ASN2T1G, U7 LMP2231AMF, U8 MCP3465R, U9 TMP451, Y1 12Mhz

Commit message: wip
Parts:
- added C41: 100nF, Capacitor_SMD:C_0603_1608Metric, F.Cu at (213.3, 107.2)
- C25, C28, C29, C31, C32, C37, C38, R19, R20, R21, R22, R23, R25, R27, R28, R29, R36, R38, R44, R45, U4, U7, U9: moved to B.Cu
- J6, J7: footprint Connector_PinSocket_2.54mm:PinSocket_1x02_P2.54mm_Vertical -> Connector_JST:JST_EH_B2B-EH-A_1x02_P2.50mm_Vertical
- moved J10 161.6 mm to (243.0, 106.2), turned to 90 degrees
- moved J1 155.2 mm to (242.8, 114.0), turned to 90 degrees
- moved J4 145.5 mm to (237.4, 122.1), turned to 180 degrees
- moved J5 142.0 mm to (229.2, 122.1), turned to 180 degrees
- moved R28 136.7 mm to (223.9, 105.8), turned to -90 degrees
- moved J11 134.7 mm to (234.2, 91.8)
- moved R27 133.6 mm to (214.6, 108.6), turned to -90 degrees
- moved R39 132.8 mm to (215.8, 112.6), turned to 90 degrees
- moved J7 132.2 mm to (234.2, 105.6)
- moved R29 132.2 mm to (221.9, 106.6), turned to 180 degrees
- moved R36 129.7 mm to (220.6, 109.6), turned to 90 degrees
- moved R25 128.6 mm to (212.1, 103.6), turned to 180 degrees
- moved R30 128.5 mm to (221.9, 106.6), turned to 180 degrees
- moved J8 128.5 mm to (211.7, 101.2), turned to 90 degrees
- moved R19 128.2 mm to (214.7, 114.6), turned to 180 degrees
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Connections:
- R39 pad 2: /sensorAmp/ECsens -> /sensorAmp/PHsens
- R40 pad 2: /sensorAmp/PHsens -> /sensorAmp/ECsens

Commit message: wip
Parts:
- removed C4: 1µF, Capacitor_SMD:C_0603_1608Metric
- removed L1: 600R, Inductor_SMD:L_0603_1608Metric
- C1, C10, C12, C13, C14, C16, C18, C19, C2, C20, C21, C22, C3, C5, C6, C7, C8, C9, L2, L3, R1, R10, R11, R2, R3, R34, R4, R41, R42, R5, R6, U1, U3, Y1: moved to B.Cu
- moved J2 146.8 mm to (232.4, 117.5), turned to 90 degrees
- moved R3 142.7 mm to (236.3, 114.3)
- moved R18 139.5 mm to (226.3, 117.0), turned to 180 degrees
- moved C2 138.8 mm to (236.6, 112.3), turned to 90 degrees
- moved D1 137.3 mm to (240.0, 117.3), turned to 90 degrees
- moved D2 136.4 mm to (226.0, 113.3)
- moved R17 132.9 mm to (226.3, 118.2), turned to 180 degrees
- moved U1 131.3 mm to (231.3, 108.6)
- moved R5 131.1 mm to (239.8, 108.8), turned to 90 degrees
- moved R2 130.6 mm to (242.0, 116.9), turned to 90 degrees
- moved R8 130.4 mm to (239.8, 114.4), turned to 90 degrees
- moved R13 130.2 mm to (239.2, 108.0), turned to 90 degrees
- moved R7 127.1 mm to (228.7, 113.3), turned to 180 degrees
- moved R10 126.7 mm to (230.2, 114.9), turned to 180 degrees
- moved C10 126.7 mm to (236.6, 115.7)
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Connections:
- U2 pad 11: Net-(R7-Pad1) -> /UART1
- U2 pad 12: Net-(R8-Pad2) -> /UART1
- U2 pad 13: unconnected-(U2-Pad13) -> Net-(R7-Pad1)
- U2 pad 14: /DIN1 -> unconnected-(U2-Pad14)
- U2 pad 15: /DIN2 -> unconnected-(U2-Pad15)
- U2 pad 17: /sensorAmp/ecExc+ -> unconnected-(U2-Pad17)
- U2 pad 18: /sensorAmp/ecExc- -> unconnected-(U2-Pad18)
- U2 pad 2: /UART1 -> unconnected-(U2-Pad2)
- U2 pad 27: unconnected-(U2-Pad27) -> /UART0
- U2 pad 28: /sensorAmp/PH_R_Exc -> /UART0
- U2 pad 29: unconnected-(U2-Pad29) -> Net-(R8-Pad2)
- U2 pad 3: /UART1 -> /sensorAmp/CS
- U2 pad 30: /sensorAmp/SDI -> unconnected-(U2-Pad30)
- U2 pad 31: /sensorAmp/SDO -> unconnected-(U2-Pad31)
- U2 pad 32: /sensorAmp/CS -> unconnected-(U2-Pad32)
- U2 pad 34: /sensorAmp/SCK -> unconnected-(U2-Pad34)
- U2 pad 4: unconnected-(U2-Pad4) -> /sensorAmp/SCK
- U2 pad 40: unconnected-(U2-Pad40) -> /DIN1
- U2 pad 41: unconnected-(U2-Pad41) -> /DIN2
- U2 pad 43: Net-(C4-Pad1) -> +3V3
- U2 pad 5: unconnected-(U2-Pad5) -> /sensorAmp/SDI
- U2 pad 6: /UART0 -> /sensorAmp/SDO
- U2 pad 7: /UART0 -> /sensorAmp/PH_R_Exc
- U2 pad 8: unconnected-(U2-Pad8) -> /sensorAmp/ecExc+
- U2 pad 9: unconnected-(U2-Pad9) -> /sensorAmp/ecExc-
Routing:
- net GND: track 0.00 -> 117.4 mm, vias 0 -> 43
- net /sensorAmp/Vguard: track 0.00 -> 58.3 mm, vias 0 -> 4
- net +3V3: track 0.00 -> 47.0 mm, vias 0 -> 14
- net +3.3VA: track 0.00 -> 42.2 mm, vias 0 -> 9
- net /sensorAmp/ecExc-: track 0.00 -> 28.3 mm, vias 0 -> 1
- net /sensorAmp/ecExc+: track 0.00 -> 23.8 mm, vias 0 -> 1
- net /sensorAmp/SDO: track 0.00 -> 23.7 mm, vias 0 -> 2
- net /sensorAmp/SDI: track 0.00 -> 23.7 mm, vias 0 -> 2
- net /sensorAmp/CS: track 0.00 -> 23.7 mm, vias 0 -> 2
- net /sensorAmp/SDA: track 0.00 -> 23.6 mm, vias 0 -> 1
- net /sensorAmp/SCL: track 0.00 -> 23.4 mm, vias 0 -> 1
- net /sensorAmp/SCK: track 0.00 -> 22.8 mm, vias 0 -> 2
- net +1V1: track 0.00 -> 15.9 mm, vias 0 -> 3
- net Net-(C30-Pad1): track 0.00 -> 14.3 mm, vias 0 -> 1
- net /sensorAmp/Vref: track 0.00 -> 12.8 mm, vias 0 -> 1
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- added copper zone on B.Cu, net +24V
- added copper zone on In2.Cu, net +3.3VA
- added copper zone on B.Cu, net +3V3
- added copper zone on F.Cu, net +3V3
- added copper zone on In2.Cu, net +3V3
- added copper zone on In1.Cu, net /sensorAmp/Vguard
- added copper zone on B.Cu, net /sensorAmp/Vref
- added copper zone on B.Cu, net GND
- added copper zone on F.Cu, net GND
- added copper zone on In1.Cu, net GND
- added copper zone on B.Cu, net Net-(C12-Pad1)
- added copper zone on B.Cu, net Net-(C26-Pad1)
- added copper zone on F.Cu, net Net-(C26-Pad1)
- added copper zone on B.Cu, net Net-(C6-Pad2)
Other:
- board size 50 x 50 mm -> 35.5 x 35 mm
- copper layers 2 -> 4
- rule pad_to_mask_clearance: 0 -> 0.05

Commit message: prepare for Manufacturing
Other:
- outline, holes or cut-outs redrawn
- board text added: "SensNode V1.0"
Changed lines of the file:
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@@
     (pad_to_mask_clearance 0.05)
     (solder_mask_min_width 0.1)
+    (aux_axis_origin 210 125)
+    (grid_origin 210 125)
     (pcbplotparams
       (layerselection 0x00010fc_ffffffff)
@@
     (fp_line (start 1.15 -1.15) (end 1.15 -0.8) (layer "F.SilkS") (width 0.12))
     (fp_line (start -1.15 1.15) (end -1.15 0.8) (layer "F.SilkS") (width 0.12))
-    (fp_line (start 1.15 1.15) (end 1.15 0.8) (layer "F.SilkS") (width 0.12))
-    (fp_line (start -0.8 1.15) (end -1.15 1.15) (layer "F.SilkS") (width 0.12))
     (fp_line (start -0.8 -1.15) (end -1.35 -1.15) (layer "F.SilkS") (width 0.12))
-    (fp_line (start 0.8 1.15) (end 1.15 1.15) (layer "F.SilkS") (width 0.12))
+    (fp_line (start -0.8 1.15) (end -1.15 1.15) (layer "F.SilkS") (width 0.12))
     (fp_line (start 0.8 -1.15) (end 1.15 -1.15) (layer "F.SilkS") (width 0.12))
+    (fp_line (start 1.15 1.15) (end 1.15 0.8) (layer "F.SilkS") (width 0.12))
+    (fp_line (start 0.8 1.15) (end 1.15 1.15) (layer "F.SilkS") (width 0.12))
     (fp_line (start 1.6 -1.6) (end 1.6 1.6) (layer "F.CrtYd") (width 0.05))
-    (fp_line (start -1.6 1.6) (end -1.6 -1.6) (layer "F.CrtYd") (width 0.05))
     (fp_line (start -1.6 -1.6) (end 1.6 -1.6) (layer "F.CrtYd") (width 0.05))
+    (fp_line (start -1.6 1.6) (end -1.6 -1.6) (layer "F.CrtYd") (width 0.05))
     (fp_line (start 1.6 1.6) (end -1.6 1.6) (layer "F.CrtYd") (width 0.05))
-    (fp_line (start -1 1) (end 1 1) (layer "F.Fab") (width 0.15))
-    (fp_line (start -0.7 -1) (end -1 -0.7) (layer "F.Fab") (width 0.15))
-    (fp_line (start 1 -1) (end -0.7 -1) (layer "F.Fab") (width 0.15))
     (fp_line (start -1 -0.7) (end -1 1) (layer "F.Fab") (width 0.15))
     (fp_line (start 1 1) (end 1 -1) (layer "F.Fab") (width 0.15))
+    (fp_line (start -0.7 -1) (end -1 -0.7) (layer "F.Fab") (width 0.15))
+    (fp_line (start -1 1) (end 1 1) (layer "F.Fab") (width 0.15))
+    (fp_line (start 1 -1) (end -0.7 -1) (layer "F.Fab") (width 0.15))
     (pad "1" smd oval (at -1.075 -0.4 270) (size 0.2 0.7) (layers "F.Cu" "F.Paste" "F.Mask")
       (net 2 "GND") (pinfunction "AGND") (pintype "unspecified"))
@@
       (net 13 "+3.3VA") (pinfunction "AVDD") (pintype "unspecified"))
     (pad "13" smd rect (at 0 0 180) (size 1 1) (layers "F.Cu" "F.Paste" "F.Mask")
-      (net 2 "GND") (pinfunction "EP") (pintype "unspecified") (solder_paste_margin -0.75))
+      (net 2 "GND") (pinfunction "EP") (pintype "unspecified") (solder_paste_margin -0.1))
   )
   (footprint "Inductor_SMD:L_1008_2520Metric" (layer "F.Cu")
@@
     )
   )
-  (gr_line (start 245.5 90) (end 210 90) (layer "Edge.Cuts") (width 0.1))
-  (gr_line (start 210 90) (end 210 125) (layer "Edge.Cuts") (width 0.1))
-  (gr_line (start 210 125) (end 245.5 125) (layer "Edge.Cuts") (width 0.1))
-  (gr_line (start 245.5 125) (end 245.5 90) (layer "Edge.Cuts") (width 0.1))
+  (gr_arc (start 245.5 122) (mid 244.62132 124.12132) (end 242.5 125) (layer "Edge.Cuts") (width 0.1))
+  (gr_arc (start 213 125) (mid 210.87868 124.12132) (end 210 122) (layer "Edge.Cuts") (width 0.1))
+  (gr_line (start 242.5 90) (end 213 90) (layer "Edge.Cuts") (width 0.1))
+  (gr_line (start 210 93) (end 210 122) (layer "Edge.Cuts") (width 0.1))
+  (gr_line (start 213 125) (end 242.5 125) (layer "Edge.Cuts") (width 0.1))
+  (gr_arc (start 242.5 90) (mid 244.62132 90.87868) (end 245.5 93) (layer "Edge.Cuts") (width 0.1))
+  (gr_line (start 245.5 122) (end 245.5 93) (layer "Edge.Cuts") (width 0.1))
+  (gr_arc (start 210 93) (mid 210.87868 90.87868) (end 213 90) (layer "Edge.Cuts") (width 0.1))
+  (gr_text "SensNode\nV1.0" (at 214.5 99 -90) (layer "B.SilkS")
+    (effects (font (size 1 1) (thickness 0.15)) (justify mirror))
+  )
+  (gr_text "SensNode\nV1.0" (at 236 96) (layer "F.SilkS")
+    (effects (font (size 1 1) (thickness 0.15)))
+  )
+  (dimension (type aligned) (layer "Dwgs.User")
+    (pts (xy 242.5 90) (xy 242.5 125))
+    (height -8.14)
+    (gr_text "35,0000 mm" (at 249.49 107.5 90) (layer "Dwgs.User")
+      (effects (font (size 1 1) (thickness 0.15)))
+    )
+    (format (units 3) (units_format 1) (precision 4))
+    (style (thickness 0.15) (arrow_length 1.27) (text_position_mode 0) (extension_height 0.58642) (extension_offset 0.5) keep_text_aligned)
+  )
+  (dimension (type aligned) (layer "Dwgs.User")
+    (pts (xy 245.5 122) (xy 210 122))
+    (height -6.81)
+    (gr_text "35,5000 mm" (at 227.75 127.66) (layer "Dwgs.User")
+      (effects (font (size 1 1) (thickness 0.15)))
+    )
+    (format (units 3) (units_format 1) (precision 4))
+    (style (thickness 0.15) (arrow_length 1.27) (text_position_mode 0) (extension_height 0.58642) (extension_offset 0.5) keep_text_aligned)
+  )
   (segment (start 233.825 114.170674) (end 234.047174 113.9485) (width 0.127) (layer "F.Cu") (net 1))
   (segment (start 233.825 114.8375) (end 233.825 114.170674) (width 0.127) (layer "F.Cu") (net 1))
@@
         (xy 240.2 96.9)
         (xy 245.5 96.9)
-        (xy 245.5 125)
-        (xy 210 125)
+        (xy 245.5 119)
+        (xy 241 119)
+        (xy 239.5 120.5)
+        (xy 239.5 125)
+        (xy 216 125)
+        (xy 216 120.5)
+        (xy 214.5 119)
+        (xy 210 119)
         (xy 210 96.1)
         (xy 216.6 96.1)
