File: sensorNode/sensorAmp.kicad_sch (KiCad schematic)
At the start: 37 parts

Commit message: wip
Parts:
- added C? (x2): 1n, Capacitor_SMD:C_0603_1608Metric, symbol Device:C
- added C? (x6): 100nF, Capacitor_SMD:C_0603_1608Metric, symbol Device:C
- added C?: 1µF, Capacitor_SMD:C_0603_1608Metric, symbol Device:C
- added C?: 22µ, Capacitor_SMD:C_1206_3216Metric, symbol Device:C
- added L?: 4.7u, Inductor_SMD:L_1008_2520Metric, symbol Device:L
- added R?: 100R, symbol Device:R
- added R? (x2): 1k, symbol Device:R
- added R? (x2): 10k, symbol Device:R
- added R?: 0R, symbol Device:R
- added U?: MCP3465R, Bergi:QFN-12_EP_2x2_Pitch0.4mm, symbol Bergi:MCP3465R
- added U?: MCP6001R, Package_TO_SOT_SMD:SOT-23-5, symbol Amplifier_Operational:MCP6001R
Connections:
- net +3.3VA: now also C?.1, C?.1, C?.1, C?.1, C?.2, L?.2, R?.1, R?.1, U?.12 (AVDD), U?.2 (V+)
- net +3V3: now also C?.1, L?.1, U?.11 (DVDD)
- net ECsens: now also R?.2
- net GND: now also C?.1, C?.2, C?.2, C?.2, C?.2, C?.2, C?.2, C?.2, C?.2, C?.2, R?.2, U?.1 (AGND), U?.10 (DGND), U?.13 (EP), U?.2 (REFIN-), U?.5 (V-)
- net PHsens: now also R?.2
- net Vref: now also C?.1, R?.1
- new net: R?.2, U?.1, U?.4 (-)
- new net: C?.1, R?.1, U?.5 (CH0)
- new net: C?.1, R?.2, U?.3 (REFIN+)
- new net: C?.1, R?.1, U?.4 (CH1)
- new net: R?.1, R?.2, U?.3 (+)
- new net CS: U?.6 (CS)
- new net SCK: U?.7 (SCK)
- new net SDI: U?.8 (SDI)
- new net SDO: U?.9 (SDO)
Other:
- note removed: "MCP3465R"

Commit message: wip
Parts:
- added C?: 100nF, Capacitor_SMD:C_0603_1608Metric, symbol Device:C
Connections:
- net GND: now also C?.2
- net ecExc+: no longer R?.2, R?.2
- net at R?.1, R?.2, U?.3 (+): now also C?.1
- net PHRexc renamed PH_R_Exc
- new net ecExc-: R?.2, R?.2
Other:
- moved on the sheet: C?, L?

Commit message: wip
Parts:
- added C24: 22µ, Capacitor_SMD:C_1206_3216Metric, symbol Device:C
- added R17, R18: 1R, Inductor_SMD:L_0603_1608Metric, symbol Device:R
- J10: renamed from J?; footprint (none) -> Connector_JST:JST_EH_B4B-EH-A_1x04_P2.50mm_Vertical
- J11, J8: renamed from J?; footprint (none) -> Connector_JST:JST_EH_B2B-EH-A_1x02_P2.50mm_Vertical
- J9: renamed from J?; footprint (none) -> Connector_Coaxial:BNC_Amphenol_B6252HB-NPP3G-50_Horizontal; HTN (none) -> CONBNC002
- R19, R20, R21, R22, R23, R24, R25, R26, R27, R28, R29, R30, R31, R32, R33, R34, R35, R36, R37, R38, R39, R40, R43: renamed from R?; footprint (none) -> Inductor_SMD:L_0603_1608Metric
- gave numbers to parts that had none: 28
Connections:
- net +3.3VA: now also C24.2
- net GND: now also R17.2, R18.2
- new net: C24.1, R17.1, R18.1
Other:
- moved on the sheet: C23, L4

Commit message: wip
Parts:
- added C41: 100nF, Capacitor_SMD:C_0603_1608Metric, symbol Device:C
Connections:
- net +3.3VA: now also C41.1
- net ECsens: now also R40.2; no longer R39.2
- net GND: now also C41.2
- net PHsens: now also R39.2; no longer R40.2
Changed lines of the file:
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@@
     (effects (font (size 1.27 1.27)) (justify right bottom))
   )
-  (label "ECsens" (at 189.23 128.27 180)
+  (label "ECsens" (at 189.23 130.81 180)
     (effects (font (size 1.27 1.27)) (justify right bottom))
   )
@@
     (effects (font (size 1.27 1.27)) (justify left bottom))
   )
-  (label "PHsens" (at 189.23 130.81 180)
+  (label "PHsens" (at 189.23 128.27 180)
     (effects (font (size 1.27 1.27)) (justify right bottom))
   )
@@
     )
     (property "Datasheet" "" (id 3) (at 162.56 152.4 0)
+      (effects (font (size 1.27 1.27)) hide)
+    )
+    (pin "1")
+  )
+  (symbol (lib_id "power:+3.3VA") (at 160.02 36.83 0) (unit 1)
+    (in_bom yes) (on_board yes) (fields_autoplaced)
+    (property "Reference" "#PWR0107" (id 0) (at 160.02 40.64 0)
+      (effects (font (size 1.27 1.27)) hide)
+    )
+    (property "Value" "+3.3VA" (id 1) (at 160.02 31.75 0))
+    (property "Footprint" "" (id 2) (at 160.02 36.83 0)
+      (effects (font (size 1.27 1.27)) hide)
+    )
+    (property "Datasheet" "" (id 3) (at 160.02 36.83 0)
       (effects (font (size 1.27 1.27)) hide)
     )
@@
     )
     (pin "1")
+  )
+  (symbol (lib_id "Device:C") (at 160.02 40.64 0) (unit 1)
+    (in_bom yes) (on_board yes)
+    (property "Reference" "C41" (id 0) (at 153.67 38.1 0)
+      (effects (font (size 1.27 1.27)) (justify left))
+    )
+    (property "Value" "100nF" (id 1) (at 153.67 43.18 0)
+      (effects (font (size 1.27 1.27)) (justify left))
+    )
+    (property "Footprint" "Capacitor_SMD:C_0603_1608Metric" (id 2) (at 160.9852 44.45 0)
+      (effects (font (size 1.27 1.27)) hide)
+    )
+    (property "Datasheet" "~" (id 3) (at 160.02 40.64 0)
+      (effects (font (size 1.27 1.27)) hide)
+    )
+    (pin "1")
+    (pin "2")
   )
   (symbol (lib_id "Device:C") (at 91.44 57.15 0) (unit 1)
@@
     (pin "7")
   )
+  (symbol (lib_id "power:GND") (at 160.02 44.45 0) (unit 1)
+    (in_bom yes) (on_board yes)
+    (property "Reference" "#PWR0108" (id 0) (at 160.02 50.8 0)
+      (effects (font (size 1.27 1.27)) hide)
+    )
+    (property "Value" "GND" (id 1) (at 160.02 48.26 0))
+    (property "Footprint" "" (id 2) (at 160.02 44.45 0)
+      (effects (font (size 1.27 1.27)) hide)
+    )
+    (property "Datasheet" "" (id 3) (at 160.02 44.45 0)
+      (effects (font (size 1.27 1.27)) hide)
+    )
+    (pin "1")
+  )
   (symbol (lib_id "power:+3V3") (at 203.2 27.94 0) (mirror y) (unit 1)

Commit message: wip
Parts:
- U9: HTN (none) -> TMP451HQDQFRQ1
Other:
- note added: "Adr: 0x49"
- note removed: "Adr: 0x4C"
Changed lines of the file:
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@@
     (stroke (width 0) (type default) (color 0 0 0 0))
   )
-  (text "Adr: 0x4C" (at 231.14 54.61 0)
+  (text "Adr: 0x49" (at 231.14 54.61 0)
     (effects (font (size 1.27 1.27)) (justify left bottom))
   )
@@
       (effects (font (size 1.27 1.27)) hide)
     )
+    (property "HTN" "TMP451HQDQFRQ1" (id 4) (at 227.33 41.91 0)
+      (effects (font (size 1.27 1.27)) hide)
+    )
