File: pumpCon/pumpDrivers.kicad_sch (KiCad schematic)
At the start: 50 parts

Commit message: start placing
Parts:
- J10, J11: renamed from J?; footprint Connector_PinSocket_2.54mm:PinSocket_1x02_P2.54mm_Vertical -> Connector_Molex:Molex_KK-254_AE-6410-02A_1x02_P2.54mm_Vertical
- J12, J13, J14, J15, J16, J17, J18, J19: renamed from J?; footprint (none) -> Connector_JST:JST_EH_B5B-EH-A_1x05_P2.50mm_Vertical
- U10, U15, U16, U9: renamed from U?; footprint (none) -> Package_SO:TSSOP-16_4.4x5mm_P0.65mm
- gave numbers to parts that had none: 36
Connections:
- net at U19.1 (I1): now also U16.3 (QD); no longer U16.15 (QA)
- net at U19.2 (I2): now also U16.2 (QC); no longer U16.1 (QB)
- net at U19.3 (I3): now also U16.1 (QB); no longer U16.2 (QC)
- net at U19.4 (I4): now also U16.15 (QA); no longer U16.3 (QD)
- net at U12.1 (I1): now also U9.7 (QH); no longer U9.4 (QE)
- net at U12.2 (I2): now also U9.6 (QG); no longer U9.5 (QF)
- net at U12.3 (I3): now also U9.5 (QF); no longer U9.6 (QG)
- net at U12.4 (I4): now also U9.4 (QE); no longer U9.7 (QH)
- net at U18.1 (I1): now also U15.7 (QH); no longer U15.4 (QE)
- net at U18.2 (I2): now also U15.6 (QG); no longer U15.5 (QF)
- net at U18.3 (I3): now also U15.5 (QF); no longer U15.6 (QG)
- net at U18.4 (I4): now also U15.4 (QE); no longer U15.7 (QH)
- net at U9.1 (QB): now also U11.3 (I3); no longer U11.2 (I2)
- net at U9.15 (QA): now also U11.4 (I4); no longer U11.1 (I1)
- net at U9.2 (QC): now also U11.2 (I2); no longer U11.3 (I3)
- net at U9.3 (QD): now also U11.1 (I1); no longer U11.4 (I4)
- net at U10.1 (QB): now also U13.3 (I3); no longer U13.2 (I2)
- net at U10.15 (QA): now also U13.4 (I4); no longer U13.1 (I1)
- net at U10.2 (QC): now also U13.2 (I2); no longer U13.3 (I3)
- net at U10.3 (QD): now also U13.1 (I1); no longer U13.4 (I4)
- net at U10.4 (QE): now also U14.4 (I4); no longer U14.1 (I1)
- net at U10.5 (QF): now also U14.3 (I3); no longer U14.2 (I2)
- net at U10.6 (QG): now also U14.2 (I2); no longer U14.3 (I3)
- net at U10.7 (QH): now also U14.1 (I1); no longer U14.4 (I4)
- net at U20.1 (I1): now also U16.7 (QH); no longer U16.4 (QE)
- net at U20.2 (I2): now also U16.6 (QG); no longer U16.5 (QF)
- net at U20.3 (I3): now also U16.5 (QF); no longer U16.6 (QG)
- net at U20.4 (I4): now also U16.4 (QE); no longer U16.7 (QH)
- net at U15.1 (QB): now also U17.3 (I3); no longer U17.2 (I2)
- net at U15.15 (QA): now also U17.4 (I4); no longer U17.1 (I1)
- net at U15.2 (QC): now also U17.2 (I2); no longer U17.3 (I3)
- net at U15.3 (QD): now also U17.1 (I1); no longer U17.4 (I4)

Commit message: wip
Connections:
- net at U19.1 (I1): now also U16.4 (QE); no longer U16.3 (QD)
- net at U19.2 (I2): now also U16.5 (QF); no longer U16.2 (QC)
- net at U19.3 (I3): now also U16.6 (QG); no longer U16.1 (QB)
- net at U19.4 (I4): now also U16.7 (QH); no longer U16.15 (QA)
- net at U12.1 (I1): now also U9.15 (QA); no longer U9.7 (QH)
- net at U12.2 (I2): now also U9.1 (QB); no longer U9.6 (QG)
- net at U12.3 (I3): now also U9.2 (QC); no longer U9.5 (QF)
- net at U12.4 (I4): now also U9.3 (QD); no longer U9.4 (QE)
- net at U18.1 (I1): now also U15.15 (QA); no longer U15.7 (QH)
- net at U18.2 (I2): now also U15.1 (QB); no longer U15.6 (QG)
- net at U18.3 (I3): now also U15.2 (QC); no longer U15.5 (QF)
- net at U18.4 (I4): now also U15.3 (QD); no longer U15.4 (QE)
- net at U11.3 (I3): now also U9.6 (QG); no longer U9.1 (QB)
- net at U11.4 (I4): now also U9.7 (QH); no longer U9.15 (QA)
- net at U11.2 (I2): now also U9.5 (QF); no longer U9.2 (QC)
- net at U11.1 (I1): now also U9.4 (QE); no longer U9.3 (QD)
- net at U10.1 (QB): now also U14.2 (I2); no longer U13.3 (I3)
- net at U10.15 (QA): now also U14.1 (I1); no longer U13.4 (I4)
- net at U10.2 (QC): now also U14.3 (I3); no longer U13.2 (I2)
- net at U10.3 (QD): now also U14.4 (I4); no longer U13.1 (I1)
- net at U10.4 (QE): now also U13.1 (I1); no longer U14.4 (I4)
- net at U10.5 (QF): now also U13.2 (I2); no longer U14.3 (I3)
- net at U10.6 (QG): now also U13.3 (I3); no longer U14.2 (I2)
- net at U10.7 (QH): now also U13.4 (I4); no longer U14.1 (I1)
- net at U20.1 (I1): now also U16.15 (QA); no longer U16.7 (QH)
- net at U20.2 (I2): now also U16.1 (QB); no longer U16.6 (QG)
- net at U20.3 (I3): now also U16.2 (QC); no longer U16.5 (QF)
- net at U20.4 (I4): now also U16.3 (QD); no longer U16.4 (QE)
- net at U17.3 (I3): now also U15.6 (QG); no longer U15.1 (QB)
- net at U17.4 (I4): now also U15.7 (QH); no longer U15.15 (QA)
- net at U17.2 (I2): now also U15.5 (QF); no longer U15.2 (QC)
- net at U17.1 (I1): now also U15.4 (QE); no longer U15.3 (QD)
Other:
- moved on the sheet: C45, C49, C50, J12, J13, J14, J15, J16, J17, J18, J19, U11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

Commit message: wip
Connections:
- net +3.3V is gone; now on net +3V3: U10.10 (~{SRCLR}), U10.16 (VCC), U15.10 (~{SRCLR}), U15.16 (VCC), U16.10 (~{SRCLR}), U16.16 (VCC), U9.10 (~{SRCLR}), U9.16 (VCC)
- net S_D: now also U16.14 (SER); no longer U15.14 (SER)
- net S_D1: now also U15.14 (SER), U16.9 (QH'); no longer U15.9 (QH'), U16.14 (SER)
- net S_D2: now also U10.14 (SER), U15.9 (QH'); no longer U16.9 (QH'), U9.14 (SER)
- net S_D3: now also U10.9 (QH'), U9.14 (SER); no longer U10.14 (SER), U9.9 (QH')

Commit message: wip
Connections:
- net P_EN renamed P_EN0
- net P_EN0: no longer U8.3 (IN1)
- new net P_EN1: U8.3 (IN1)
Changed lines of the file:
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@@
     (effects (font (size 1.27 1.27)) (justify right))
   )
-  (hierarchical_label "P_EN" (shape input) (at 59.69 104.14 180)
+  (hierarchical_label "P_EN0" (shape input) (at 59.69 104.14 180)
     (effects (font (size 1.27 1.27)) (justify right))
   )
-  (hierarchical_label "P_EN" (shape input) (at 60.96 162.56 180)
+  (hierarchical_label "P_EN1" (shape input) (at 60.96 162.56 180)
     (effects (font (size 1.27 1.27)) (justify right))
   )
