File: pumpCon/pumpCon.kicad_sch (KiCad schematic)
At the start: 80 parts

Commit message: start placing
Parts:
- J4, J5: renamed from J?; footprint Connector_Molex:Molex_KK-254_AE-6410-03A_1x03_P2.54mm_Vertical -> Connector_JST:JST_EH_B3B-EH-A_1x03_P2.50mm_Vertical
- L1: renamed from L?; footprint (none) -> Inductor_SMD:L_0603_1608Metric
- gave numbers to parts that had none: 77
Other:
- moved on the sheet: D2, R10, R11, R12, R24, R25

Commit message: -
Parts:
- added C51: 100nF, Capacitor_SMD:C_0603_1608Metric, symbol Device:C
- added C52: 1µF, Capacitor_SMD:C_0603_1608Metric, symbol Device:C
- added H1, H2, H3, H4: MountingHole, MountingHole:MountingHole_3.2mm_M3_DIN965, symbol Mechanical:MountingHole
Connections:
- net +3V3: now also C51.1, C52.1
- net GND: now also C51.2, C52.2
Other:
- moved on the sheet: C7, C9, R17, R18, U3

Commit message: wip
Parts:
- added R32, R33: 1R, Resistor_SMD:R_0603_1608Metric, symbol Device:R
- J6, J7: footprint Connector_PinSocket_2.54mm:PinSocket_1x02_P2.54mm_Vertical -> Connector_JST:JST_EH_B2B-EH-A_1x02_P2.50mm_Vertical
Connections:
- net GND: now also R32.2, R33.2; no longer C13.1
- new net: C13.1, R32.1, R33.1
Other:
- moved on the sheet: C9
Changed lines of the file:
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@@
   (junction (at 203.2 30.48) (diameter 0) (color 0 0 0 0)
   )
+  (junction (at 196.85 41.91) (diameter 0) (color 0 0 0 0)
+  )
   (junction (at 209.55 30.48) (diameter 0) (color 0 0 0 0)
   )
   (junction (at 229.87 31.75) (diameter 0) (color 0 0 0 0)
   )
+  (junction (at 196.85 49.53) (diameter 0) (color 0 0 0 0)
+  )
   (junction (at 250.19 31.75) (diameter 0) (color 0 0 0 0)
   )
@@
     (stroke (width 0) (type default) (color 0 0 0 0))
   )
+  (wire (pts (xy 194.31 41.91) (xy 196.85 41.91))
+    (stroke (width 0) (type default) (color 0 0 0 0))
+  )
   (wire (pts (xy 105.41 124.46) (xy 119.38 124.46))
     (stroke (width 0) (type default) (color 0 0 0 0))
@@
     (stroke (width 0) (type default) (color 0 0 0 0))
   )
-  (wire (pts (xy 196.85 44.45) (xy 196.85 41.91))
+  (wire (pts (xy 194.31 49.53) (xy 196.85 49.53))
     (stroke (width 0) (type default) (color 0 0 0 0))
   )
@@
       (effects (font (size 1.27 1.27)) (justify left))
     )
-    (property "Footprint" "Connector_PinSocket_2.54mm:PinSocket_1x02_P2.54mm_Vertical" (id 2) (at 205.74 91.44 0)
+    (property "Footprint" "Connector_JST:JST_EH_B2B-EH-A_1x02_P2.50mm_Vertical" (id 2) (at 205.74 91.44 0)
       (effects (font (size 1.27 1.27)) hide)
     )
@@
     (pin "1")
   )
-  (symbol (lib_id "power:+24V") (at 185.42 38.1 0) (unit 1)
-    (in_bom yes) (on_board yes) (fields_autoplaced)
-    (property "Reference" "#PWR0123" (id 0) (at 185.42 41.91 0)
+  (symbol (lib_id "power:+24V") (at 180.34 38.1 0) (unit 1)
+    (in_bom yes) (on_board yes)
+    (property "Reference" "#PWR0123" (id 0) (at 180.34 41.91 0)
       (effects (font (size 1.27 1.27)) hide)
     )
-    (property "Value" "+24V" (id 1) (at 185.42 33.02 0))
-    (property "Footprint" "" (id 2) (at 185.42 38.1 0)
+    (property "Value" "+24V" (id 1) (at 180.34 34.29 0))
+    (property "Footprint" "" (id 2) (at 180.34 38.1 0)
       (effects (font (size 1.27 1.27)) hide)
     )
-    (property "Datasheet" "" (id 3) (at 185.42 38.1 0)
+    (property "Datasheet" "" (id 3) (at 180.34 38.1 0)
       (effects (font (size 1.27 1.27)) hide)
     )
@@
       (effects (font (size 1.27 1.27)) (justify left))
     )
-    (property "Footprint" "Connector_PinSocket_2.54mm:PinSocket_1x02_P2.54mm_Vertical" (id 2) (at 199.39 128.27 0)
+    (property "Footprint" "Connector_JST:JST_EH_B2B-EH-A_1x02_P2.50mm_Vertical" (id 2) (at 199.39 128.27 0)
       (effects (font (size 1.27 1.27)) hide)
     )
@@
     (pin "1")
   )
-  (symbol (lib_id "Device:C") (at 185.42 41.91 180) (unit 1)
+  (symbol (lib_id "Device:C") (at 180.34 41.91 180) (unit 1)
     (in_bom yes) (on_board yes)
-    (property "Reference" "C9" (id 0) (at 186.69 39.37 0)
+    (property "Reference" "C9" (id 0) (at 181.61 39.37 0)
       (effects (font (size 1.27 1.27)) (justify right))
     )
-    (property "Value" "10µ" (id 1) (at 186.69 44.45 0)
+    (property "Value" "10µ" (id 1) (at 181.61 44.45 0)
       (effects (font (size 1.27 1.27)) (justify right))
     )
-    (property "Footprint" "Capacitor_SMD:C_1210_3225Metric" (id 2) (at 184.4548 38.1 0)
+    (property "Footprint" "Capacitor_SMD:C_1210_3225Metric" (id 2) (at 179.3748 38.1 0)
       (effects (font (size 1.27 1.27)) hide)
     )
-    (property "Datasheet" "~" (id 3) (at 185.42 41.91 0)
+    (property "Datasheet" "~" (id 3) (at 180.34 41.91 0)
       (effects (font (size 1.27 1.27)) hide)
     )
@@
     (pin "2")
   )
+  (symbol (lib_id "Device:R") (at 196.85 45.72 0) (unit 1)
+    (in_bom yes) (on_board yes)
+    (property "Reference" "R33" (id 0) (at 199.39 48.26 90)
+      (effects (font (size 1.27 1.27)) (justify left))
+    )
+    (property "Value" "1R" (id 1) (at 196.85 46.99 90)
+      (effects (font (size 1.27 1.27)) (justify left))
+    )
+    (property "Footprint" "Resistor_SMD:R_0603_1608Metric" (id 2) (at 195.072 45.72 90)
+      (effects (font (size 1.27 1.27)) hide)
+    )
+    (property "Datasheet" "~" (id 3) (at 196.85 45.72 0)
+      (effects (font (size 1.27 1.27)) hide)
+    )
+    (pin "1")
+    (pin "2")
+  )
   (symbol (lib_id "Device:C") (at 234.95 27.94 180) (unit 1)
     (in_bom yes) (on_board yes)
@@
     (pin "2")
   )
-  (symbol (lib_id "power:GND") (at 185.42 45.72 0) (unit 1)
+  (symbol (lib_id "power:GND") (at 180.34 45.72 0) (unit 1)
     (in_bom yes) (on_board yes)
-    (property "Reference" "#PWR0119" (id 0) (at 185.42 52.07 0)
+    (property "Reference" "#PWR0119" (id 0) (at 180.34 52.07 0)
       (effects (font (size 1.27 1.27)) hide)
     )
-    (property "Value" "GND" (id 1) (at 185.42 49.53 0))
-    (property "Footprint" "" (id 2) (at 185.42 45.72 0)
+    (property "Value" "GND" (id 1) (at 180.34 49.53 0))
+    (property "Footprint" "" (id 2) (at 180.34 45.72 0)
       (effects (font (size 1.27 1.27)) hide)
     )
-    (property "Datasheet" "" (id 3) (at 185.42 45.72 0)
+    (property "Datasheet" "" (id 3) (at 180.34 45.72 0)
       (effects (font (size 1.27 1.27)) hide)
     )
@@
     (pin "1")
   )
+  (symbol (lib_id "Device:R") (at 194.31 45.72 0) (unit 1)
+    (in_bom yes) (on_board yes)
+    (property "Reference" "R32" (id 0) (at 191.77 48.26 90)
+      (effects (font (size 1.27 1.27)) (justify left))
+    )
+    (property "Value" "1R" (id 1) (at 194.31 46.99 90)
+      (effects (font (size 1.27 1.27)) (justify left))
+    )
+    (property "Footprint" "Resistor_SMD:R_0603_1608Metric" (id 2) (at 192.532 45.72 90)
+      (effects (font (size 1.27 1.27)) hide)
+    )
+    (property "Datasheet" "~" (id 3) (at 194.31 45.72 0)
+      (effects (font (size 1.27 1.27)) hide)
+    )
+    (pin "1")
+    (pin "2")
+  )
   (symbol (lib_id "power:+3V3") (at 246.38 82.55 0) (unit 1)
     (in_bom yes) (on_board yes)
@@
     (pin "1")
   )
-  (symbol (lib_id "power:GND") (at 196.85 44.45 0) (unit 1)
+  (symbol (lib_id "power:GND") (at 196.85 49.53 0) (unit 1)
     (in_bom yes) (on_board yes)
-    (property "Reference" "#PWR0124" (id 0) (at 196.85 50.8 0)
+    (property "Reference" "#PWR0124" (id 0) (at 196.85 55.88 0)
       (effects (font (size 1.27 1.27)) hide)
     )
-    (property "Value" "GND" (id 1) (at 196.85 48.26 0))
-    (property "Footprint" "" (id 2) (at 196.85 44.45 0)
+    (property "Value" "GND" (id 1) (at 196.85 53.34 0))
+    (property "Footprint" "" (id 2) (at 196.85 49.53 0)
       (effects (font (size 1.27 1.27)) hide)
     )
-    (property "Datasheet" "" (id 3) (at 196.85 44.45 0)
+    (property "Datasheet" "" (id 3) (at 196.85 49.53 0)
       (effects (font (size 1.27 1.27)) hide)
     )
@@
     )
     (path "/571f6d5e-59b7-44e1-852d-cf47bc65ea21"
-      (reference "J6") (unit 1) (value "Conn_01x02") (footprint "Connector_PinSocket_2.54mm:PinSocket_1x02_P2.54mm_Vertical")
+      (reference "J6") (unit 1) (value "Conn_01x02") (footprint "Connector_JST:JST_EH_B2B-EH-A_1x02_P2.50mm_Vertical")
     )
     (path "/038f88d0-25cb-4cbc-9f1a-53363bad139d"
-      (reference "J7") (unit 1) (value "Conn_01x02") (footprint "Connector_PinSocket_2.54mm:PinSocket_1x02_P2.54mm_Vertical")
+      (reference "J7") (unit 1) (value "Conn_01x02") (footprint "Connector_JST:JST_EH_B2B-EH-A_1x02_P2.50mm_Vertical")
     )
     (path "/116b1d26-d7be-4274-a9fd-1e5101ff22f1"
@@
       (reference "R31") (unit 1) (value "1.1k") (footprint "Resistor_SMD:R_0603_1608Metric")
     )
+    (path "/d14c4765-591d-4cb7-8c13-bf02d74563c6"
+      (reference "R32") (unit 1) (value "1R") (footprint "Resistor_SMD:R_0603_1608Metric")
+    )
+    (path "/cd1a0824-5270-4dae-a15c-2109703f72e0"
+      (reference "R33") (unit 1) (value "1R") (footprint "Resistor_SMD:R_0603_1608Metric")
+    )
     (path "/c6c82006-26c7-4641-9e87-e0fdb5b42a77"

Commit message: wip
Connections:
- net pumpDrivers/P_EN is gone; now on net flowPuls1: U2.32 (GPIO21)
- net LED_DIM: now also U2.36 (GPIO24); no longer U2.17 (GPIO14)
- net flowPuls0: now also U2.35 (GPIO23); no longer U2.16 (GPIO13)
- net flowPuls1: no longer U2.14 (GPIO11)
- net pumpDrivers/PWM0_Iref: now also U2.27 (GPIO16); no longer U2.37 (GPIO25)
- net pumpDrivers/PWM1_Iref: now also U2.28 (GPIO17); no longer U2.36 (GPIO24)
- net pumpDrivers/PWM_P0: now also U2.15 (GPIO12); no longer U2.35 (GPIO23)
- net pumpDrivers/PWM_P1: now also U2.17 (GPIO14); no longer U2.34 (GPIO22)
- net pumpDrivers/S_CLK: now also U2.13 (GPIO10); no longer U2.28 (GPIO17)
- net pumpDrivers/S_CS: now also U2.12 (GPIO9); no longer U2.27 (GPIO16)
- net pumpDrivers/S_D: now also U2.14 (GPIO11); no longer U2.29 (GPIO18)
- net pumpDrivers/S_EN: now also U2.11 (GPIO8); no longer U2.30 (GPIO19)
- net pumpDrivers/P_EN1: now reaches U2.18 (GPIO15)
- net at U2.4 (GPIO2): no longer R10.1
- net at R11.2, R12.1: now also U2.29 (GPIO18); no longer U2.5 (GPIO3)
- net at U2.8 (GPIO6): now also R10.1
- new net pumpDrivers/P_EN0: U2.16 (GPIO13)
Other:
- sheet pumpDrivers ports: added P_EN0, P_EN1; removed P_EN
- note added: "PWM0A PWM0B"
- note added: "PWM2A PWM2B"
- note added: "PWM6A PWM6B"
- note added: "PWM7A PWM7B"
- note removed: "PWM5B"
- note removed: "PWM6B"
- note removed: "PWM7A"
- moved on the sheet: R11, R12

Commit message: wip
Parts:
- R23: value 27k -> 38k
- R26: value 91k -> 157k
Changed lines of the file:
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@@
       (effects (font (size 1.27 1.27)) (justify left))
     )
-    (property "Value" "27k" (id 1) (at 234.95 48.2599 0)
+    (property "Value" "38k" (id 1) (at 234.95 48.2599 0)
       (effects (font (size 1.27 1.27)) (justify left))
     )
@@
       (effects (font (size 1.27 1.27)) (justify left))
     )
-    (property "Value" "91k" (id 1) (at 260.35 36.8299 0)
+    (property "Value" "157k" (id 1) (at 260.35 36.8299 0)
       (effects (font (size 1.27 1.27)) (justify left))
     )
@@
     )
     (path "/3e01fbd3-2dcb-4064-80fd-a9ab6c695306"
-      (reference "R23") (unit 1) (value "27k") (footprint "Resistor_SMD:R_0603_1608Metric")
+      (reference "R23") (unit 1) (value "38k") (footprint "Resistor_SMD:R_0603_1608Metric")
     )
     (path "/64e4c45e-2790-461b-8350-3a4b913f4f00"
@@
     )
     (path "/ef3fe419-54ef-4cc2-a084-79bf7e3147f8"
-      (reference "R26") (unit 1) (value "91k") (footprint "Resistor_SMD:R_0603_1608Metric")
+      (reference "R26") (unit 1) (value "157k") (footprint "Resistor_SMD:R_0603_1608Metric")
     )
     (path "/f21d7fe0-0ec4-4a88-889d-e8a6d3b033f4"
