File: pumpCon/pumpCon.kicad_pcb (KiCad board)
At the start: 2 copper layers, 130 parts, among them J1 USB_B_Micro, J10 Conn_01x02, J11 Conn_01x02, J12 Conn_01x05, J13 Conn_01x05, J14 Conn_01x05, J15 Conn_01x05, J16 Conn_01x05, J17 Conn_01x05, J18 Conn_01x05, J19 Conn_01x05, J2 Conn_01x03, J3 Conn_01x02, J4 Conn_01x03, J5 Conn_01x03, J6 Conn_01x02, J7 Conn_01x02, J8 Conn_01x03, J9 Conn_01x03, U1 W25Q16JVUXIQ, U10 74HC595, U11 ULN2003F12, U12 ULN2003F12, U13 ULN2003F12, U14 ULN2003F12, U15 74HC595, U16 74HC595, U17 ULN2003F12, U18 ULN2003F12, U19 ULN2003F12, U2 RP2040, U20 ULN2003F12, U3 AP2127K-ADJ, U4 TPS92200DxRXL, U5 MCP6001R, U6 AP63357Q, U7 DRV8231ADSGR, U8 DRV8231ADSGR, U9 74HC595, Y1 12Mhz

Commit message: -
Parts:
- added C51: 100nF, Capacitor_SMD:C_0603_1608Metric, F.Cu at (243.2, 35.0)
- added C52: 1µF, Capacitor_SMD:C_0603_1608Metric, F.Cu at (177.5, 27.5)
- added H1: MountingHole, MountingHole:MountingHole_3.2mm_M3_DIN965, F.Cu at (131.8, 74.8)
- added H2: MountingHole, MountingHole:MountingHole_3.2mm_M3_DIN965, F.Cu at (62.0, 74.5)
- added H3: MountingHole, MountingHole:MountingHole_3.2mm_M3_DIN965, F.Cu at (41.4, 81.2)
- added H4: MountingHole, MountingHole:MountingHole_3.2mm_M3_DIN965, F.Cu at (41.4, 74.1)
- C20, C24, C26, R23, R26, R27: moved to B.Cu
- moved C43 142.3 mm to (71.2, 98.5), turned to 90 degrees
- moved C44 139.0 mm to (79.8, 98.5), turned to 90 degrees
- moved C47 138.8 mm to (88.8, 98.5), turned to 90 degrees
- moved C46 138.6 mm to (69.8, 90.0), turned to 90 degrees
- moved C48 111.3 mm to (97.8, 98.5), turned to 90 degrees
- moved C45 108.5 mm to (96.8, 90.0), turned to 90 degrees
- moved C49 108.3 mm to (87.8, 90.0), turned to 90 degrees
- moved C50 105.7 mm to (78.8, 90.0), turned to 90 degrees
- moved R8 93.1 mm to (140.2, 93.8)
- moved C4 90.8 mm to (140.0, 96.8)
- moved R9 90.3 mm to (140.0, 95.2)
- moved C6 79.1 mm to (139.8, 87.0)
- moved R16 76.7 mm to (225.0, 132.2)
- moved U1 76.5 mm to (159.8, 111.8)
- moved R13 76.0 mm to (139.8, 83.2)
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
Commit message: wip
Parts:
- added R32: 1R, Resistor_SMD:R_0603_1608Metric, B.Cu at (113.5, 100.2)
- added R33: 1R, Resistor_SMD:R_0603_1608Metric, B.Cu at (113.5, 101.5)
- C10, C13, C14, C21, C29, C31, C32, C33, C34, C37, C43, C44, C47, C48, C51, C52, C7, C9, L2, L4, R16, R17, R18, R19, R20, R21, R22, R28, R29, U10, U15, U16, U3, U5, U6, U7, U8, U9: moved to B.Cu
- J6, J7: footprint Connector_PinSocket_2.54mm:PinSocket_1x02_P2.54mm_Vertical -> Connector_JST:JST_EH_B2B-EH-A_1x02_P2.50mm_Vertical
- moved R21 192.1 mm to (66.8, 107.1)
- moved C10 191.3 mm to (65.3, 104.9), turned to 90 degrees
- moved U5 191.2 mm to (67.5, 104.4), turned to 90 degrees
- moved C51 187.9 mm to (67.5, 101.6)
- moved R20 184.9 mm to (69.5, 107.1)
- moved R19 183.9 mm to (69.8, 105.1), turned to -90 degrees
- moved R4 154.4 mm to (69.7, 105.0), turned to 90 degrees
- moved R5 135.2 mm to (68.4, 105.0), turned to 90 degrees
- moved R2 133.5 mm to (66.2, 104.8)
- moved R1 129.8 mm to (66.2, 106.0)
- moved J6 128.4 mm to (64.5, 101.8), turned to 180 degrees
- moved J1 124.9 mm to (69.2, 108.8)
- moved J7 118.5 mm to (124.2, 83.2), turned to 90 degrees
- moved R22 117.7 mm to (121.5, 81.0), turned to 180 degrees
- moved C31 117.5 mm to (116.0, 103.2), turned to -90 degrees
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Connections:
- C13 pad 1: GND -> Net-(C13-Pad1)
- U10 pad 1: Net-(U10-Pad1) -> Net-(U14-Pad2)
- U10 pad 2: Net-(U10-Pad2) -> Net-(U14-Pad3)
- U10 pad 3: Net-(U10-Pad3) -> Net-(U14-Pad4)
- U10 pad 4: Net-(U10-Pad4) -> Net-(U13-Pad1)
- U10 pad 5: Net-(U10-Pad5) -> Net-(U13-Pad2)
- U10 pad 7: Net-(U10-Pad7) -> Net-(U13-Pad4)
- U11 pad 1: Net-(U11-Pad1) -> Net-(U9-Pad4)
- U12 pad 1: Net-(U12-Pad1) -> Net-(U9-Pad15)
- U12 pad 2: Net-(U12-Pad2) -> Net-(U9-Pad1)
- U12 pad 3: Net-(U12-Pad3) -> Net-(U9-Pad2)
- U12 pad 4: Net-(U12-Pad4) -> Net-(U9-Pad3)
- U13 pad 1: Net-(U10-Pad3) -> Net-(U13-Pad1)
- U13 pad 2: Net-(U10-Pad2) -> Net-(U13-Pad2)
- U13 pad 3: Net-(U10-Pad1) -> Net-(U10-Pad6)
- U13 pad 4: Net-(U10-Pad15) -> Net-(U13-Pad4)
- U14 pad 1: Net-(U10-Pad7) -> Net-(U10-Pad15)
- U14 pad 2: Net-(U10-Pad6) -> Net-(U14-Pad2)
- U14 pad 3: Net-(U10-Pad5) -> Net-(U14-Pad3)
- U14 pad 4: Net-(U10-Pad4) -> Net-(U14-Pad4)
- U15 pad 1: Net-(U15-Pad1) -> Net-(U18-Pad2)
- U15 pad 15: Net-(U15-Pad15) -> Net-(U18-Pad1)
- U15 pad 2: Net-(U15-Pad2) -> Net-(U18-Pad3)
- U15 pad 3: Net-(U15-Pad3) -> Net-(U18-Pad4)
- U15 pad 4: Net-(U15-Pad4) -> Net-(U17-Pad1)
- U15 pad 5: Net-(U15-Pad5) -> Net-(U17-Pad2)
- U15 pad 6: Net-(U15-Pad6) -> Net-(U17-Pad3)
- U15 pad 7: Net-(U15-Pad7) -> Net-(U17-Pad4)
- U16 pad 1: Net-(U16-Pad1) -> Net-(U20-Pad2)
- U16 pad 15: Net-(U16-Pad15) -> Net-(U20-Pad1)
- U16 pad 2: Net-(U16-Pad2) -> Net-(U20-Pad3)
- U16 pad 3: Net-(U16-Pad3) -> Net-(U20-Pad4)
- U17 pad 1: Net-(U15-Pad3) -> Net-(U17-Pad1)
- U17 pad 2: Net-(U15-Pad2) -> Net-(U17-Pad2)
- U17 pad 3: Net-(U15-Pad1) -> Net-(U17-Pad3)
- U17 pad 4: Net-(U15-Pad15) -> Net-(U17-Pad4)
- U18 pad 1: Net-(U15-Pad7) -> Net-(U18-Pad1)
- U18 pad 2: Net-(U15-Pad6) -> Net-(U18-Pad2)
- U18 pad 3: Net-(U15-Pad5) -> Net-(U18-Pad3)
- U18 pad 4: Net-(U15-Pad4) -> Net-(U18-Pad4)
- U19 pad 1: Net-(U16-Pad3) -> Net-(U16-Pad4)
- U19 pad 2: Net-(U16-Pad2) -> Net-(U16-Pad5)
- U19 pad 3: Net-(U16-Pad1) -> Net-(U16-Pad6)
- U19 pad 4: Net-(U16-Pad15) -> Net-(U16-Pad7)
- U20 pad 1: Net-(U16-Pad7) -> Net-(U20-Pad1)
- U20 pad 2: Net-(U16-Pad6) -> Net-(U20-Pad2)
- U20 pad 3: Net-(U16-Pad5) -> Net-(U20-Pad3)
- U20 pad 4: Net-(U16-Pad4) -> Net-(U20-Pad4)
- U9 pad 1: Net-(U11-Pad3) -> Net-(U9-Pad1)
- U9 pad 15: Net-(U11-Pad4) -> Net-(U9-Pad15)
- U9 pad 2: Net-(U11-Pad2) -> Net-(U9-Pad2)
- U9 pad 3: Net-(U11-Pad1) -> Net-(U9-Pad3)
- U9 pad 4: Net-(U12-Pad4) -> Net-(U9-Pad4)
- U9 pad 5: Net-(U12-Pad3) -> Net-(U11-Pad2)
- U9 pad 6: Net-(U12-Pad2) -> Net-(U11-Pad3)
- U9 pad 7: Net-(U12-Pad1) -> Net-(U11-Pad4)

Commit message: placing done
Parts:
- C1, C11, C12, C15, C16, C17, C18, C19, C2, C22, C23, C25, C27, C28, C3, C30, C4, C5, C6, C8, L1, L3, R13, R14, R15, R24, R25, R3, R6, R8, R9, U1, U4, Y1: moved to B.Cu
- C39, C40, R16: moved to F.Cu
- moved R12 176.1 mm to (66.4, 102.4)
- moved C22 158.7 mm to (77.5, 107.7), turned to 90 degrees
- moved C35 156.4 mm to (75.5, 106.0), turned to 90 degrees
- moved C17 155.1 mm to (80.0, 101.3), turned to 180 degrees
- moved C19 154.1 mm to (83.0, 108.5), turned to 90 degrees
- moved C16 151.9 mm to (81.9, 108.5), turned to 90 degrees
- moved C23 151.6 mm to (80.8, 108.5), turned to 90 degrees
- moved R10 151.5 mm to (89.2, 105.3)
- moved C36 148.5 mm to (75.4, 108.5), turned to -90 degrees
- moved R7 147.7 mm to (86.5, 110.6)
- moved R31 147.5 mm to (76.5, 108.5), turned to -90 degrees
- moved C18 140.9 mm to (86.6, 109.2), turned to 90 degrees
- moved R30 140.6 mm to (76.5, 105.9), turned to 90 degrees
- moved D1 138.8 mm to (64.3, 103.8), turned to -90 degrees
- moved C3 137.1 mm to (86.6, 106.5), turned to -90 degrees
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Other:
- board outline added: 50 x 50 mm
- copper layers 2 -> 4

Commit message: wip
Parts:
- moved R28 4.39 mm to (97.5, 80.8)
- moved C34 4.35 mm to (92.9, 71.3), turned to 180 degrees
- moved C32 3.93 mm to (96.4, 80.8), turned to -90 degrees
- moved C33 2.94 mm to (95.6, 71.2), turned to -90 degrees
- moved U7 2.45 mm to (95.0, 78.2), turned to 180 degrees
- moved C37 2.12 mm to (93.5, 81.0), turned to 180 degrees
- moved R29 1.92 mm to (96.7, 71.3)
- moved U8 1.33 mm to (94.4, 68.6), turned to 180 degrees
- moved J2 1.30 mm to (82.1, 99.0)
- moved C52 1.05 mm to (90.9, 97.0)
- moved C7 1.05 mm to (89.2, 99.2)
- moved R17 1.05 mm to (87.9, 99.2)
- moved R18 1.05 mm to (91.4, 101.5)
- moved U3 1.05 mm to (91.7, 99.2)
- moved C47 1.01 mm to (87.5, 76.9)
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Connections:
- U10 pad 10: +3.3V -> +3V3
- U10 pad 14: /pumpDrivers/S_D3 -> /pumpDrivers/S_D2
- U10 pad 16: +3.3V -> +3V3
- U10 pad 9: unconnected-(U10-Pad9) -> /pumpDrivers/S_D3
- U15 pad 10: +3.3V -> +3V3
- U15 pad 14: /pumpDrivers/S_D -> /pumpDrivers/S_D1
- U15 pad 16: +3.3V -> +3V3
- U15 pad 9: /pumpDrivers/S_D1 -> /pumpDrivers/S_D2
- U16 pad 10: +3.3V -> +3V3
- U16 pad 14: /pumpDrivers/S_D1 -> /pumpDrivers/S_D
- U16 pad 16: +3.3V -> +3V3
- U16 pad 9: /pumpDrivers/S_D2 -> /pumpDrivers/S_D1
- U9 pad 10: +3.3V -> +3V3
- U9 pad 14: /pumpDrivers/S_D2 -> /pumpDrivers/S_D3
- U9 pad 16: +3.3V -> +3V3
- U9 pad 9: /pumpDrivers/S_D3 -> unconnected-(U9-Pad9)
Routing:
- net +3V3: track 0.00 -> 55.7 mm, vias 0 -> 7
- net /pumpDrivers/P_EN: track 0.00 -> 38.1 mm, vias 0 -> 2
- net /pumpDrivers/S_EN: track 0.00 -> 36.0 mm, vias 0 -> 4
- net /pumpDrivers/S_CS: track 0.00 -> 34.4 mm, vias 0 -> 4
- net /pumpDrivers/S_CLK: track 0.00 -> 34.3 mm, vias 0 -> 4
- net GND: track 0.00 -> 31.3 mm, vias 0 -> 37
- net /pumpDrivers/Isens1: track 0.00 -> 28.5 mm, vias 0 -> 2
- net /pumpDrivers/PWM_P1: track 0.00 -> 27.2 mm, vias 0 -> 2
- net +5V: track 0.00 -> 22.4 mm, vias 0 -> 19
- net /pumpDrivers/PWM1_Iref: track 0.00 -> 18.8 mm, vias 0 -> 1
- net /pumpDrivers/Isens0: track 0.00 -> 15.8 mm, vias 0 -> 1
- net /pumpDrivers/PWM_P0: track 0.00 -> 14.7 mm, vias 0 -> 1
- net Net-(J16-Pad2): track 0.00 -> 12.6 mm
- net Net-(J12-Pad2): track 0.00 -> 12.5 mm
- net Net-(J18-Pad2): track 0.00 -> 12.3 mm
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- added copper zone on F.Cu, net +5V
- added copper zone on In2.Cu, net +5V
- added copper zone on B.Cu, net /pumpDrivers/VM
- added copper zone on F.Cu, net /pumpDrivers/VM
- added copper zone on In2.Cu, net /pumpDrivers/VM
- added copper zone on B.Cu, net GND
- added copper zone on F.Cu, net GND
- added copper zone on F.Cu, net Net-(C39-Pad2)
- added copper zone on F.Cu, net Net-(C40-Pad2)
- added copper zone on B.Cu, net Net-(J10-Pad2)
- added copper zone on B.Cu, net Net-(J11-Pad2)
- added copper zone on B.Cu, net Net-(L6-Pad1)
- added copper zone on F.Cu, net Net-(L6-Pad1)
- added copper zone on B.Cu, net Net-(L7-Pad1)
- added copper zone on F.Cu, net Net-(L7-Pad1)

Commit message: wip
Parts:
- C10, C51, R19, R20, R21, R24, R25, U5: moved to F.Cu
- R11, R12: moved to B.Cu
- moved R25 11.2 mm to (87.2, 105.8), turned to -90 degrees
- moved C10 9.63 mm to (71.1, 98.1), turned to 0 degrees
- moved C51 9.14 mm to (64.0, 99.3), turned to -90 degrees
- moved R12 7.63 mm to (69.8, 109.2), turned to -90 degrees
- moved D1 6.71 mm to (70.8, 102.0), turned to 180 degrees
- moved U5 6.49 mm to (66.5, 99.2), turned to 180 degrees
- moved R20 6.43 mm to (71.1, 99.2), turned to 0 degrees
- moved R19 6.40 mm to (71.1, 100.3), turned to 0 degrees
- moved R21 5.89 mm to (69.1, 98.8), turned to -90 degrees
- moved R11 4.62 mm to (69.0, 107.3), turned to 0 degrees
- moved R24 4.52 mm to (87.2, 108.4)
- moved J2 4.43 mm to (86.5, 99.8)
- moved R16 3.80 mm to (74.5, 104.0)
- moved R22 3.36 mm to (64.6, 99.8)
- moved C18 2.89 mm to (84.8, 106.9), turned to 0 degrees
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Connections:
- R10 pad 1: Net-(R10-Pad1) -> Net-(U2-Pad8)
- R11 pad 2: Net-(R11-Pad2) -> Net-(U2-Pad29)
- R12 pad 1: Net-(R11-Pad2) -> Net-(U2-Pad29)
- U2 pad 11: unconnected-(U2-Pad11) -> /pumpDrivers/S_EN
- U2 pad 12: unconnected-(U2-Pad12) -> /pumpDrivers/S_CS
- U2 pad 13: unconnected-(U2-Pad13) -> /pumpDrivers/S_CLK
- U2 pad 14: /flowPuls1 -> /pumpDrivers/S_D
- U2 pad 15: unconnected-(U2-Pad15) -> /pumpDrivers/PWM_P0
- U2 pad 16: /flowPuls0 -> /pumpDrivers/P_EN0
- U2 pad 17: /LED_DIM -> /pumpDrivers/PWM_P1
- U2 pad 18: unconnected-(U2-Pad18) -> /pumpDrivers/P_EN1
- U2 pad 27: /pumpDrivers/S_CS -> /pumpDrivers/PWM0_Iref
- U2 pad 28: /pumpDrivers/S_CLK -> /pumpDrivers/PWM1_Iref
- U2 pad 29: /pumpDrivers/S_D -> Net-(U2-Pad29)
- U2 pad 30: /pumpDrivers/S_EN -> unconnected-(U2-Pad30)
- U2 pad 32: /pumpDrivers/P_EN -> /flowPuls1
- U2 pad 34: /pumpDrivers/PWM_P1 -> unconnected-(U2-Pad34)
- U2 pad 35: /pumpDrivers/PWM_P0 -> /flowPuls0
- U2 pad 36: /pumpDrivers/PWM1_Iref -> /LED_DIM
- U2 pad 37: /pumpDrivers/PWM0_Iref -> unconnected-(U2-Pad37)
- U2 pad 4: Net-(R10-Pad1) -> unconnected-(U2-Pad4)
- U2 pad 5: Net-(R11-Pad2) -> unconnected-(U2-Pad5)
- U2 pad 8: unconnected-(U2-Pad8) -> Net-(U2-Pad8)
- U7 pad 3: /pumpDrivers/P_EN -> /pumpDrivers/P_EN0
- U8 pad 3: /pumpDrivers/P_EN -> /pumpDrivers/P_EN1
Routing:
- net GND: track 31.3 -> 101.2 mm, vias 37 -> 74
- net +24V: track 0.00 -> 51.4 mm, vias 0 -> 11
- net /pumpDrivers/P_EN1: track 0.00 -> 43.9 mm, vias 0 -> 1
- net /flowPuls1: track 0.00 -> 42.7 mm, vias 0 -> 1
- net /pumpDrivers/P_EN: track 38.1 -> 0.00 mm, vias 2 -> 0
- net /pumpDrivers/Isens0: track 15.8 -> 50.6 mm
- net /flowPuls0: track 0.00 -> 33.6 mm, vias 0 -> 1
- net /pumpDrivers/P_EN0: track 0.00 -> 33.3 mm, vias 0 -> 1
- net /pumpDrivers/Isens1: track 28.5 -> 61.1 mm, vias 2 -> 1
- net +3V3: track 55.7 -> 87.0 mm, vias 7 -> 18
- net /pumpDrivers/PWM0_Iref: track 8.15 -> 31.5 mm
- net /pumpDrivers/PWM1_Iref: track 18.8 -> 41.6 mm
- net /pumpDrivers/PWM_P0: track 14.7 -> 33.8 mm
- net /pumpDrivers/S_CS: track 34.4 -> 52.4 mm, vias 4 -> 5
- net /pumpDrivers/S_EN: track 36.0 -> 53.9 mm, vias 4 -> 5
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- added copper zone on B.Cu, net +24V
- added copper zone on F.Cu, net +24V
- added copper zone on In2.Cu, net +24V
- added copper zone on B.Cu, net +3V3
- added copper zone on In2.Cu, net +3V3
- added copper zone on B.Cu, net +5V
- added copper zone on In1.Cu, net GND
- added copper zone on B.Cu, net Net-(C13-Pad2)
- added copper zone on B.Cu, net Net-(C21-Pad1)
- added copper zone on B.Cu, net Net-(C8-Pad2)

Commit message: prepare for Manufacturing
Other:
- outline, holes or cut-outs redrawn
- rule pad_to_mask_clearance: 0 -> 0.05
- board text added: "PumpCon V1.0"
Changed lines of the file:
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@@
       (dielectric_constraints no)
     )
-    (pad_to_mask_clearance 0)
+    (pad_to_mask_clearance 0.05)
+    (solder_mask_min_width 0.1)
+    (aux_axis_origin 59 111.5)
+    (grid_origin 59 111.5)
     (pcbplotparams
       (layerselection 0x00010fc_ffffffff)
@@
     )
   )
-  (gr_line (start 109 111.5) (end 59 111.5) (layer "Edge.Cuts") (width 0.1))
-  (gr_line (start 59 61.5) (end 109 61.5) (layer "Edge.Cuts") (width 0.1))
-  (gr_line (start 59 111.5) (end 59 61.5) (layer "Edge.Cuts") (width 0.1))
-  (gr_line (start 109 111.5) (end 109 61.5) (layer "Edge.Cuts") (width 0.1))
+  (gr_arc (start 59 64.5) (mid 59.87868 62.37868) (end 62 61.5) (layer "Edge.Cuts") (width 0.1))
+  (gr_arc (start 106 61.5) (mid 108.12132 62.37868) (end 109 64.5) (layer "Edge.Cuts") (width 0.1))
+  (gr_line (start 106 111.5) (end 62 111.5) (layer "Edge.Cuts") (width 0.1))
+  (gr_line (start 62 61.5) (end 106 61.5) (layer "Edge.Cuts") (width 0.1))
+  (gr_line (start 59 108.5) (end 59 64.5) (layer "Edge.Cuts") (width 0.1))
+  (gr_line (start 109 108.5) (end 109 64.5) (layer "Edge.Cuts") (width 0.1))
+  (gr_arc (start 62 111.5) (mid 59.87868 110.62132) (end 59 108.5) (layer "Edge.Cuts") (width 0.1))
+  (gr_arc (start 109 108.5) (mid 108.12132 110.62132) (end 106 111.5) (layer "Edge.Cuts") (width 0.1))
+  (gr_text "PumpCon\nV1.0" (at 93 92.5 90) (layer "B.SilkS")
+    (effects (font (size 1 1) (thickness 0.15)) (justify mirror))
+  )
+  (gr_text "PumpCon\nV1.0" (at 93 92.5 90) (layer "F.SilkS")
+    (effects (font (size 1 1) (thickness 0.15)))
+  )
   (dimension (type aligned) (layer "Dwgs.User")
     (pts (xy 59 61.5) (xy 109 61.5))
