File: mainControl/mainControl.kicad_sch (KiCad schematic)
At the start: 78 parts

Commit message: wip
Parts:
- added C? (x4): 100µ, Capacitor_THT:CP_Radial_D6.3mm_P2.50mm, symbol Device:C_Polarized
Connections:
- net +24V: now also C?.1, C?.1, C?.1, C?.1
- net GND: now also C?.2, C?.2, C?.2, C?.2
Other:
- moved on the sheet: R?

Commit message: wip
Parts:
- removed J?: Conn_01x03, Connector_Molex:Molex_KK-254_AE-6410-03A_1x03_P2.54mm_Vertical, symbol Connector_Generic:Conn_01x03
- added H1, H2, H3, H4: MountingHole, MountingHole:MountingHole_3.2mm_M3_DIN965, symbol Mechanical:MountingHole
- added J9: Conn_01x04, Connector_PinSocket_2.54mm:PinSocket_1x04_P2.54mm_Vertical, symbol Connector_Generic:Conn_01x04
- added U?: TVS2700DRV, Package_SON:WSON-6-1EP_2x2mm_P0.65mm_EP1x1.6mm, symbol Power_Protection:TVS2700DRV
- J4: renamed from J?; footprint (none) -> Connector_Phoenix_MSTB:PhoenixContact_MSTBVA_2,5_2-G-5,08_1x02_P5.08mm_Vertical
- gave numbers to parts that had none: 80
Connections:
- net +24V: now also U?.4 (IN), U?.5 (IN), U?.6 (IN)
- net +3V3: now also J9.2 (Pin_2)
- net GND: now also J9.1 (Pin_1), U?.1 (GND), U?.2 (GND), U?.3 (GND), U?.7 (GND)
- net termUART_RX: now also J9.3 (Pin_3)
- net termUART_TX: now also J9.4 (Pin_4)
Other:
- moved on the sheet: C5

Commit message: wip
Parts:
- gave numbers to parts that had none: 1
Connections:
- net 24V_Isens: now also U2.38 (GPIO26_ADC0)
- net 24V_Vsens: now also U2.39 (GPIO27_ADC1)
Changed lines of the file:
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@@
     (effects (font (size 1.27 1.27)) (justify left bottom))
   )
+  (label "24V_Vsens" (at 105.41 133.35 0)
+    (effects (font (size 1.27 1.27)) (justify left bottom))
+  )
   (label "QSPI_CLK" (at 54.61 95.25 180)
     (effects (font (size 1.27 1.27)) (justify right bottom))
@@
     (effects (font (size 1.27 1.27)) (justify left bottom))
   )
+  (label "24V_Isens" (at 105.41 130.81 0)
+    (effects (font (size 1.27 1.27)) (justify left bottom))
+  )
   (label "UART0" (at 139.7 52.07 180)
     (effects (font (size 1.27 1.27)) (justify right bottom))
@@
   (symbol (lib_id "Power_Protection:TVS2700DRV") (at 165.1 142.24 0) (unit 1)
     (in_bom yes) (on_board yes) (fields_autoplaced)
-    (property "Reference" "U?" (id 0) (at 168.91 140.9699 0)
+    (property "Reference" "U9" (id 0) (at 168.91 140.9699 0)
       (effects (font (size 1.27 1.27)) (justify left))
     )
@@
   (symbol (lib_id "power:+24V") (at 165.1 134.62 0) (unit 1)
     (in_bom yes) (on_board yes) (fields_autoplaced)
-    (property "Reference" "#PWR?" (id 0) (at 165.1 138.43 0)
+    (property "Reference" "#PWR0115" (id 0) (at 165.1 138.43 0)
       (effects (font (size 1.27 1.27)) hide)
     )
@@
   (symbol (lib_id "power:GND") (at 165.1 149.86 0) (unit 1)
     (in_bom yes) (on_board yes) (fields_autoplaced)
-    (property "Reference" "#PWR?" (id 0) (at 165.1 156.21 0)
+    (property "Reference" "#PWR0114" (id 0) (at 165.1 156.21 0)
       (effects (font (size 1.27 1.27)) hide)
     )
@@
       (reference "#PWR0113") (unit 1) (value "GND") (footprint "")
     )
-    (path "/f66f760f-2235-4072-968d-73a2680ff3c3"
-      (reference "#PWR?") (unit 1) (value "+24V") (footprint "")
-    )
     (path "/faae0301-837f-4de9-8a80-7300286205c1"
-      (reference "#PWR?") (unit 1) (value "GND") (footprint "")
+      (reference "#PWR0114") (unit 1) (value "GND") (footprint "")
+    )
+    (path "/f66f760f-2235-4072-968d-73a2680ff3c3"
+      (reference "#PWR0115") (unit 1) (value "+24V") (footprint "")
     )
     (path "/00951d70-84c9-440a-8a3d-19c365aab257"
@@
     )
     (path "/6b4f1e21-947d-4609-aa33-1952ea0696fa"
-      (reference "U?") (unit 1) (value "TVS2700DRV") (footprint "Package_SON:WSON-6-1EP_2x2mm_P0.65mm_EP1x1.6mm")
+      (reference "U9") (unit 1) (value "TVS2700DRV") (footprint "Package_SON:WSON-6-1EP_2x2mm_P0.65mm_EP1x1.6mm")
     )
     (path "/f4c66923-385a-4c20-9d97-ec9c56ffcb8f"

Commit message: wip
Parts:
- removed BT1: Battery_Cell, Battery:BatteryHolder_Keystone_1060_1x2032, symbol Device:Battery_Cell
- removed C11, C5: 100n, Capacitor_SMD:C_0603_1608Metric, symbol Device:C
- removed C12, C14, C3: 100nF, Capacitor_SMD:C_0603_1608Metric, symbol Device:C
- removed C26, C28: 10p, Capacitor_SMD:C_0603_1608Metric, symbol Device:C
- removed C30: 100p, Capacitor_SMD:C_0603_1608Metric, symbol Device:C
- removed C8: DNP, Capacitor_SMD:C_0603_1608Metric, symbol Device:C
- removed D3: BAT54W, Diode_SMD:D_SOD-323, symbol Device:D_Filled
- removed J4: Conn_01x02, Connector_Phoenix_MSTB:PhoenixContact_MSTBVA_2,5_2-G-5,08_1x02_P5.08mm_Vertical, symbol Connector_Generic:Conn_01x02
- removed R11, R12: 0R01, Resistor_SMD:R_0805_2012Metric, symbol Device:R
- removed R13, R9: 0R, Resistor_SMD:R_0603_1608Metric, symbol Device:R
- removed R20: 1k5, Resistor_SMD:R_0603_1608Metric, symbol Device:R
- removed R21, R22, R6: 10k, Resistor_SMD:R_0603_1608Metric, symbol Device:R
- removed R26, R7: 1k, Resistor_SMD:R_0603_1608Metric, symbol Device:R
- removed U3: INA186A3IDDF, Package_TO_SOT_SMD:SOT-23-8, symbol Bergi:INA186A3IDDF
- removed U4: ILPS22QS, Bergi:HLGA-10L, symbol Bergi:ILPS22QS
- removed U6: MCP79410T-I/MNY, Package_DFN_QFN:DFN-8-1EP_3x2mm_P0.5mm_EP1.36x1.46mm, symbol Timer_RTC:MCP7940N-xMNY
- removed Y2: Crystal, Crystal:Crystal_SMD_2012-2Pin_2.0x1.2mm, symbol Device:Crystal
Connections:
- net termUART_RX: no longer U2.3 (GPIO1)
- net termUART_TX: no longer U2.2 (GPIO0)
- net at R14.2, R15.1: now also U2.37 (GPIO25); no longer U2.16 (GPIO13)
- net at R10.1: now also U2.36 (GPIO24); no longer U2.15 (GPIO12)
- net pheri/SCK: now reaches U2.17 (GPIO14)
- net pheri/SDI: now reaches U2.18 (GPIO15)
- net pheri/SDA: now reaches U2.29 (GPIO18)
- net pheri/SCL: now reaches U2.30 (GPIO19)
- net ESP/TXD: now reaches U2.40 (GPIO28_ADC2)
- net ESP/RXD: now reaches U2.41 (GPIO29_ADC3)
- net 24V_Isens: no longer names the net of U2.38 (GPIO26_ADC0)
- net 24V_Vsens: no longer names the net of U2.39 (GPIO27_ADC1)
- net SCL: no longer names the net of U2.28 (GPIO17)
- net SDA: no longer names the net of U2.27 (GPIO16)
- new net pheri/CS: U2.16 (GPIO13)
- new net pheri/SDO: U2.15 (GPIO12)
Other:
- added sheet pheri (pheri.kicad_sch)
- note removed: "ADR: 0x5C"
- note removed: "I2C Address EEPROM: 0x57 SRAM, RTC: 0x6F"
- note removed: "f = 1,06 kHz k = 0.5 V/A"
- moved on the sheet: D2, H1, H2, H3, H4, R10, R14, R15, U9

Commit message: wip
Connections:
- net termUART_RX is gone; now on net ESP/RXD: J9.3 (Pin_3)
- net termUART_TX is gone; now on net ESP/TXD: J9.4 (Pin_4)
- net UART0: now also U2.11 (GPIO8), U2.12 (GPIO9); no longer U2.4 (GPIO2), U2.5 (GPIO3)
- net UART1: now also U2.8 (GPIO6), U2.9 (GPIO7); no longer U2.6 (GPIO4), U2.7 (GPIO5)
- net UART2: now also U2.6 (GPIO4), U2.7 (GPIO5); no longer U2.8 (GPIO6), U2.9 (GPIO7)
- net UART3: now also U2.4 (GPIO2), U2.5 (GPIO3); no longer U2.11 (GPIO8), U2.12 (GPIO9)
Other:
- moved on the sheet: J9
Changed lines of the file:
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@@
   (junction (at 85.09 53.34) (diameter 0) (color 0 0 0 0)
   )
+  (junction (at 106.68 135.89) (diameter 0) (color 0 0 0 0)
+  )
   (junction (at 87.63 53.34) (diameter 0) (color 0 0 0 0)
   )
@@
   (junction (at 232.41 41.91) (diameter 0) (color 0 0 0 0)
   )
+  (junction (at 109.22 138.43) (diameter 0) (color 0 0 0 0)
+  )
   (junction (at 257.81 38.1) (diameter 0) (color 0 0 0 0)
   )
@@
     (stroke (width 0) (type default) (color 0 0 0 0))
   )
+  (wire (pts (xy 109.22 151.13) (xy 109.22 138.43))
+    (stroke (width 0) (type default) (color 0 0 0 0))
+  )
   (wire (pts (xy 250.19 38.1) (xy 257.81 38.1))
     (stroke (width 0) (type default) (color 0 0 0 0))
@@
     (stroke (width 0) (type default) (color 0 0 0 0))
   )
-  (wire (pts (xy 105.41 135.89) (xy 109.22 135.89))
+  (wire (pts (xy 105.41 135.89) (xy 106.68 135.89))
     (stroke (width 0) (type default) (color 0 0 0 0))
   )
@@
     (stroke (width 0) (type default) (color 0 0 0 0))
   )
+  (wire (pts (xy 109.22 138.43) (xy 115.57 138.43))
+    (stroke (width 0) (type default) (color 0 0 0 0))
+  )
   (wire (pts (xy 276.86 30.48) (xy 269.24 30.48))
     (stroke (width 0) (type default) (color 0 0 0 0))
   )
+  (wire (pts (xy 106.68 135.89) (xy 115.57 135.89))
+    (stroke (width 0) (type default) (color 0 0 0 0))
+  )
   (wire (pts (xy 105.41 82.55) (xy 105.41 85.09))
     (stroke (width 0) (type default) (color 0 0 0 0))
@@
     (stroke (width 0) (type default) (color 0 0 0 0))
   )
+  (wire (pts (xy 115.57 151.13) (xy 109.22 151.13))
+    (stroke (width 0) (type default) (color 0 0 0 0))
+  )
   (wire (pts (xy 38.1 72.39) (xy 38.1 73.66))
     (stroke (width 0) (type default) (color 0 0 0 0))
@@
     (stroke (width 0) (type default) (color 0 0 0 0))
   )
+  (wire (pts (xy 115.57 153.67) (xy 106.68 153.67))
+    (stroke (width 0) (type default) (color 0 0 0 0))
+  )
   (wire (pts (xy 147.32 21.59) (xy 158.75 21.59))
     (stroke (width 0) (type default) (color 0 0 0 0))
@@
   )
   (wire (pts (xy 241.3 48.26) (xy 241.3 41.91))
+    (stroke (width 0) (type default) (color 0 0 0 0))
+  )
+  (wire (pts (xy 106.68 153.67) (xy 106.68 135.89))
     (stroke (width 0) (type default) (color 0 0 0 0))
   )
@@
     (effects (font (size 1.27 1.27)) (justify right bottom))
   )
-  (label "termUART_RX" (at 193.04 86.36 180)
-    (effects (font (size 1.27 1.27)) (justify right bottom))
-  )
-  (label "UART2" (at 105.41 77.47 0)
+  (label "UART2" (at 105.41 74.93 0)
     (effects (font (size 1.27 1.27)) (justify left bottom))
   )
@@
     (effects (font (size 1.27 1.27)) (justify right bottom))
   )
-  (label "UART3" (at 105.41 82.55 0)
+  (label "UART3" (at 105.41 69.85 0)
     (effects (font (size 1.27 1.27)) (justify left bottom))
   )
@@
     (effects (font (size 1.27 1.27)) (justify right bottom))
   )
-  (label "termUART_TX" (at 193.04 88.9 180)
-    (effects (font (size 1.27 1.27)) (justify right bottom))
-  )
   (label "QSPI_D0" (at 54.61 85.09 180)
     (effects (font (size 1.27 1.27)) (justify right bottom))
@@
     (effects (font (size 1.27 1.27)) (justify left bottom))
   )
-  (label "UART0" (at 105.41 67.31 0)
+  (label "UART0" (at 105.41 85.09 0)
     (effects (font (size 1.27 1.27)) (justify left bottom))
   )
@@
     (effects (font (size 1.27 1.27)) (justify left bottom))
   )
-  (label "UART1" (at 105.41 72.39 0)
+  (label "UART1" (at 105.41 80.01 0)
     (effects (font (size 1.27 1.27)) (justify left bottom))
   )
@@
     (pin "1")
   )
-  (symbol (lib_id "Connector_Generic:Conn_01x04") (at 198.12 83.82 0) (unit 1)
-    (in_bom yes) (on_board yes) (fields_autoplaced)
-    (property "Reference" "J9" (id 0) (at 200.66 83.8199 0)
-      (effects (font (size 1.27 1.27)) (justify left))
-    )
-    (property "Value" "Conn_01x04" (id 1) (at 200.66 86.3599 0)
-      (effects (font (size 1.27 1.27)) (justify left))
-    )
-    (property "Footprint" "Connector_PinSocket_2.54mm:PinSocket_1x04_P2.54mm_Vertical" (id 2) (at 198.12 83.82 0)
-      (effects (font (size 1.27 1.27)) hide)
-    )
-    (property "Datasheet" "~" (id 3) (at 198.12 83.82 0)
+  (symbol (lib_id "Connector_Generic:Conn_01x04") (at 120.65 148.59 0) (unit 1)
+    (in_bom yes) (on_board yes) (fields_autoplaced)
+    (property "Reference" "J9" (id 0) (at 123.19 148.5899 0)
+      (effects (font (size 1.27 1.27)) (justify left))
+    )
+    (property "Value" "Conn_01x04" (id 1) (at 123.19 151.1299 0)
+      (effects (font (size 1.27 1.27)) (justify left))
+    )
+    (property "Footprint" "Connector_PinSocket_2.54mm:PinSocket_1x04_P2.54mm_Vertical" (id 2) (at 120.65 148.59 0)
+      (effects (font (size 1.27 1.27)) hide)
+    )
+    (property "Datasheet" "~" (id 3) (at 120.65 148.59 0)
       (effects (font (size 1.27 1.27)) hide)
     )
@@
     (pin "2")
   )
-  (symbol (lib_id "power:GND") (at 193.04 81.28 270) (unit 1)
-    (in_bom yes) (on_board yes)
-    (property "Reference" "#PWR057" (id 0) (at 186.69 81.28 0)
-      (effects (font (size 1.27 1.27)) hide)
-    )
-    (property "Value" "GND" (id 1) (at 187.96 81.28 90))
-    (property "Footprint" "" (id 2) (at 193.04 81.28 0)
-      (effects (font (size 1.27 1.27)) hide)
-    )
-    (property "Datasheet" "" (id 3) (at 193.04 81.28 0)
+  (symbol (lib_id "power:GND") (at 115.57 146.05 270) (unit 1)
+    (in_bom yes) (on_board yes)
+    (property "Reference" "#PWR057" (id 0) (at 109.22 146.05 0)
+      (effects (font (size 1.27 1.27)) hide)
+    )
+    (property "Value" "GND" (id 1) (at 110.49 146.05 90))
+    (property "Footprint" "" (id 2) (at 115.57 146.05 0)
+      (effects (font (size 1.27 1.27)) hide)
+    )
+    (property "Datasheet" "" (id 3) (at 115.57 146.05 0)
       (effects (font (size 1.27 1.27)) hide)
     )
@@
     (pin "1")
   )
-  (symbol (lib_id "power:+3V3") (at 193.04 83.82 90) (unit 1)
-    (in_bom yes) (on_board yes)
-    (property "Reference" "#PWR058" (id 0) (at 196.85 83.82 0)
-      (effects (font (size 1.27 1.27)) hide)
-    )
-    (property "Value" "+3V3" (id 1) (at 184.15 83.82 90)
-      (effects (font (size 1.27 1.27)) (justify right))
-    )
-    (property "Footprint" "" (id 2) (at 193.04 83.82 0)
-      (effects (font (size 1.27 1.27)) hide)
-    )
-    (property "Datasheet" "" (id 3) (at 193.04 83.82 0)
+  (symbol (lib_id "power:+3V3") (at 115.57 148.59 90) (unit 1)
+    (in_bom yes) (on_board yes)
+    (property "Reference" "#PWR058" (id 0) (at 119.38 148.59 0)
+      (effects (font (size 1.27 1.27)) hide)
+    )
+    (property "Value" "+3V3" (id 1) (at 106.68 148.59 90)
+      (effects (font (size 1.27 1.27)) (justify right))
+    )
+    (property "Footprint" "" (id 2) (at 115.57 148.59 0)
+      (effects (font (size 1.27 1.27)) hide)
+    )
+    (property "Datasheet" "" (id 3) (at 115.57 148.59 0)
       (effects (font (size 1.27 1.27)) hide)
     )
@@
     )
   )
-  (sheet (at 109.22 134.62) (size 12.7 5.08)
+  (sheet (at 115.57 134.62) (size 12.7 5.08)
     (stroke (width 0.1524) (type solid) (color 0 0 0 0))
     (fill (color 0 0 0 0.0000))
-    (property "Sheet name" "ESP" (id 0) (at 124.46 139.7 90)
+    (property "Sheet name" "ESP" (id 0) (at 130.81 139.7 90)
       (effects (font (size 1.27 1.27)) (justify left bottom))
     )
-    (property "Sheet file" "ESP.kicad_sch" (id 1) (at 109.22 140.2846 0)
+    (property "Sheet file" "ESP.kicad_sch" (id 1) (at 115.57 140.2846 0)
       (effects (font (size 1.27 1.27)) (justify left top))
     )
-    (pin "RXD" input (at 109.22 138.43 180)
-      (effects (font (size 1.27 1.27)) (justify left))
-    )
-    (pin "TXD" input (at 109.22 135.89 180)
+    (pin "RXD" input (at 115.57 138.43 180)
+      (effects (font (size 1.27 1.27)) (justify left))
+    )
+    (pin "TXD" input (at 115.57 135.89 180)
       (effects (font (size 1.27 1.27)) (justify left))
     )
@@
     )
     (path "/9b3c49ee-41bf-409c-be02-15aff49f8f07/4af497d0-89e5-4817-a24b-4ce5953028c4"
-      (reference "BT1") (unit 1) (value "Battery_Cell") (footprint "Battery:BatteryHolder_Keystone_1060_1x2032")
+      (reference "BT1") (unit 1) (value "Battery_Cell") (footprint "Battery:BatteryHolder_Keystone_3034_1x20mm")
     )
     (path "/ad31394b-5981-432e-9245-fa7d4fc31f29"
