File: mainControl/mainControl.kicad_pcb (KiCad board)
At the start: 4 copper layers, 50 x 50 mm, 117 parts, among them J1 USB_B_Micro, J10 USB_B_Micro, J11 Conn_01x02, J12 Conn_01x02, J2 Conn_01x03, J3 Conn_01x02, J4 Conn_01x02, J5 Conn_01x03, J6 Conn_01x03, J7 Conn_01x03, J8 Conn_01x03, J9 Conn_01x04, Q1 MMBT3904LP, Q2 MMBT3904LP, U1 W25Q16JVUXIQ, U2 RP2040, U3 INA186A3IDDF, U4 ILPS22QS, U5 AP63357Q, U6 MCP79410T-I/MNY, U7 ESP32-WROOM-32, U8 CP2102N-Axx-xQFN24, Y1 12Mhz, Y2 Crystal

Commit message: wip
Parts:
- added U9: TVS2700DRV, Package_SON:WSON-6-1EP_2x2mm_P0.65mm_EP1x1.6mm, F.Cu at (110.8, 178.0)
- C1, C11, C13, C15, C16, C17, C18, C19, C2, C20, C21, C22, C23, C24, C25, C27, C29, C31, C32, C33, C4, L1, L2, R16, R17, R18, R19, R20, R23, R24, R25, R3, R8, U1, U5, Y1: moved to B.Cu
- moved R14 140.3 mm to (66.3, 163.5)
- moved C3 137.9 mm to (64.2, 161.4)
- moved D1 136.0 mm to (58.1, 159.4)
- moved R3 133.0 mm to (88.6, 164.3)
- moved R1 131.2 mm to (59.0, 165.0)
- moved C21 130.4 mm to (85.7, 164.3), turned to 180 degrees
- moved R6 130.2 mm to (63.7, 164.7)
- moved R2 129.7 mm to (59.1, 163.1)
- moved R19 129.1 mm to (106.0, 174.4), turned to 90 degrees
- moved D2 127.4 mm to (72.5, 172.8), turned to 90 degrees
- moved C27 126.3 mm to (84.0, 163.0), turned to -90 degrees
- moved R4 126.1 mm to (60.0, 168.6)
- moved Y1 122.1 mm to (87.4, 161.6)
- moved C24 120.9 mm to (90.7, 161.6), turned to 90 degrees
- moved R8 118.9 mm to (79.9, 158.8), turned to 180 degrees
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Connections:
- U2 pad 38: unconnected-(U2-Pad38) -> /24V_Isens
- U2 pad 39: unconnected-(U2-Pad39) -> /24V_Vsens

Commit message: wip
Parts:
- added C41: 100nF, Capacitor_SMD:C_0603_1608Metric, F.Cu at (99.2, 167.9)
- added C42: 100nF, Capacitor_SMD:C_0603_1608Metric, F.Cu at (97.2, 167.4)
- added C43: 100nF, Capacitor_SMD:C_0603_1608Metric, F.Cu at (97.2, 164.6)
- added C44: 22µ, Capacitor_SMD:C_1206_3216Metric, B.Cu at (97.7, 160.3)
- added C45: 22µ, Capacitor_SMD:C_1206_3216Metric, B.Cu at (100.4, 157.9)
- added L3: 4.7u, Inductor_SMD:L_1008_2520Metric, B.Cu at (101.6, 160.1)
- added R43: 0R, Inductor_SMD:L_0603_1608Metric, F.Cu at (99.2, 169.0)
- added R44: 1R, Inductor_SMD:L_0603_1608Metric, B.Cu at (96.9, 157.5)
- added R45: 1R, Inductor_SMD:L_0603_1608Metric, B.Cu at (96.9, 158.6)
- added U10: MCP3465R, Bergi:QFN-12_EP_2x2_Pitch0.4mm, F.Cu at (99.5, 165.7)
- C14, U4: moved to B.Cu
- moved R6 41.7 mm to (105.3, 168.3)
- moved R7 38.8 mm to (102.6, 168.3), turned to 0 degrees
- moved C3 38.8 mm to (102.6, 167.2), turned to 180 degrees
- moved R5 18.4 mm to (76.8, 163.2)
- moved J3 18.2 mm to (91.2, 165.7), turned to 90 degrees
- moved R2 17.7 mm to (76.5, 159.8), turned to -90 degrees
- moved R4 17.4 mm to (76.8, 164.3)
- moved D1 17.2 mm to (75.2, 157.3)
- moved R1 17.2 mm to (75.4, 159.8), turned to -90 degrees
- moved R15 15.7 mm to (77.8, 159.8), turned to 90 degrees
- moved R14 10.6 mm to (76.8, 161.8)
- moved J2 9.90 mm to (93.6, 160.4), turned to 180 degrees
- moved R8 8.98 mm to (86.2, 165.2), turned to 0 degrees
- moved C29 7.96 mm to (82.1, 164.2), turned to -90 degrees
- moved C18 7.84 mm to (91.2, 157.7), turned to 90 degrees
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Connections:
- C11 pad 1: /24V_Isens -> /pheri/24V_Isens
- C3 pad 1: /24V_Vsens -> /pheri/24V_Vsens
- R20 pad 1: /24V_Isens -> /pheri/24V_Isens
- R21 pad 1: /SDA -> /pheri/SDA
- R22 pad 1: /SCL -> /pheri/SCL
- R27 pad 1: /termUART_TX -> /ESP/TXD
- R28 pad 1: /termUART_RX -> /ESP/RXD
- R6 pad 1: /24V_Vsens -> /pheri/24V_Vsens
- R7 pad 2: /24V_Vsens -> /pheri/24V_Vsens
- U2 pad 15: Net-(R10-Pad1) -> /pheri/SDO
- U2 pad 16: Net-(R14-Pad2) -> /pheri/CS
- U2 pad 17: unconnected-(U2-Pad17) -> /pheri/SCK
- U2 pad 18: unconnected-(U2-Pad18) -> /pheri/SDI
- U2 pad 2: /termUART_TX -> unconnected-(U2-Pad2)
- U2 pad 27: /SDA -> unconnected-(U2-Pad27)
- U2 pad 28: /SCL -> unconnected-(U2-Pad28)
- U2 pad 29: unconnected-(U2-Pad29) -> /pheri/SDA
- U2 pad 3: /termUART_RX -> unconnected-(U2-Pad3)
- U2 pad 30: unconnected-(U2-Pad30) -> /pheri/SCL
- U2 pad 36: unconnected-(U2-Pad36) -> Net-(R10-Pad1)
- U2 pad 37: unconnected-(U2-Pad37) -> Net-(R14-Pad2)
- U2 pad 38: /24V_Isens -> unconnected-(U2-Pad38)
- U2 pad 39: /24V_Vsens -> unconnected-(U2-Pad39)
- U2 pad 40: unconnected-(U2-Pad40) -> /ESP/TXD
- U2 pad 41: unconnected-(U2-Pad41) -> /ESP/RXD
- U3 pad 1: +3.3V -> +3.3VA
- U4 pad 2: /SCL -> /pheri/SCL
- U4 pad 4: /SDA -> /pheri/SDA
- U6 pad 5: /SDA -> /pheri/SDA
- U6 pad 6: /SCL -> /pheri/SCL

Commit message: wip
Parts:
- BT1: footprint Battery:BatteryHolder_Keystone_1060_1x2032 -> Battery:BatteryHolder_Keystone_3034_1x20mm
- R16, R17, R18, R19: moved to F.Cu
- moved R26 15.0 mm to (116.1, 140.5), turned to -90 degrees
- moved C33 14.1 mm to (103.2, 150.5), turned to 180 degrees
- moved C13 12.5 mm to (107.5, 152.1), turned to 0 degrees
- moved C31 11.4 mm to (103.2, 152.5), turned to 180 degrees
- moved D3 10.1 mm to (113.0, 143.8), turned to 0 degrees
- moved C14 9.96 mm to (98.2, 140.2)
- moved U4 9.96 mm to (98.2, 142.1)
- moved L1 9.75 mm to (108.4, 154.3), turned to 0 degrees
- moved C30 8.98 mm to (109.9, 143.8)
- moved Y2 8.98 mm to (110.9, 140.9)
- moved C12 8.98 mm to (106.7, 140.2)
- moved C26 8.98 mm to (113.3, 141.2)
- moved U6 8.98 mm to (107.5, 142.1)
- moved C28 8.98 mm to (113.3, 139.9)
- moved C19 8.88 mm to (110.2, 156.9), turned to 90 degrees
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Connections:
- J9 pad 3: /termUART_RX -> /ESP/RXD
- J9 pad 4: /termUART_TX -> /ESP/TXD
- U2 pad 11: /UART3 -> /UART0
- U2 pad 12: /UART3 -> /UART0
- U2 pad 4: /UART0 -> /UART3
- U2 pad 5: /UART0 -> /UART3
- U2 pad 6: /UART1 -> /UART2
- U2 pad 7: /UART1 -> /UART2
- U2 pad 8: /UART2 -> /UART1
- U2 pad 9: /UART2 -> /UART1
Routing:
- net GND: track 0.00 -> 112.1 mm, vias 0 -> 48
- net +24V: track 0.00 -> 99.7 mm, vias 0 -> 12
- net +3V3: track 0.00 -> 58.0 mm, vias 0 -> 27
- net Net-(BT1-Pad1): track 0.00 -> 43.1 mm, vias 0 -> 10
- net /ESP/TXD: track 0.00 -> 41.6 mm
- net /ESP/RXD: track 0.00 -> 39.6 mm
- net /pheri/SCL: track 0.00 -> 29.6 mm, vias 0 -> 1
- net /pheri/SDA: track 0.00 -> 29.3 mm, vias 0 -> 1
- net /UART0: track 0.00 -> 21.3 mm
- net /ESP/ESP_EN: track 0.00 -> 20.8 mm, vias 0 -> 1
- net +3.3VA: track 0.00 -> 20.2 mm, vias 0 -> 3
- net Net-(R10-Pad1): track 0.00 -> 18.5 mm, vias 0 -> 2
- net +1V1: track 0.00 -> 17.3 mm, vias 0 -> 3
- net /pheri/CS: track 0.00 -> 17.2 mm
- net /pheri/SCK: track 0.00 -> 15.8 mm, vias 0 -> 2
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- added copper zone on B.Cu, net +24V
- added copper zone on F.Cu, net +24V
- added copper zone on B.Cu, net +3.3VA
- added copper zone on B.Cu, net +3V3
- added copper zone on In2.Cu, net +3V3
- added copper zone on B.Cu, net GND
- added copper zone on F.Cu, net GND
- added copper zone on In1.Cu, net GND
- added copper zone on In2.Cu, net GND
- added copper zone on B.Cu, net Net-(BT1-Pad1)
- added copper zone on B.Cu, net Net-(C13-Pad2)
- added copper zone on B.Cu, net Net-(C20-Pad1)
- added copper zone on B.Cu, net Net-(C45-Pad1)
- added copper zone on B.Cu, net Net-(J4-Pad2)
Other:
- board size 50 x 50 mm -> 50 x 45 mm

Commit message: prepare for Manufacturing
Other:
- outline, holes or cut-outs redrawn
- rule pad_to_mask_clearance: 0 -> 0.05
- board text added: "MainCon V1.0"
Changed lines of the file:
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@@
       (dielectric_constraints no)
     )
-    (pad_to_mask_clearance 0)
+    (pad_to_mask_clearance 0.05)
+    (solder_mask_min_width 0.1)
+    (aux_axis_origin 70 177)
+    (grid_origin 70 177)
     (pcbplotparams
       (layerselection 0x00010fc_ffffffff)
@@
       (effects (font (size 1 1) (thickness 0.15)))
     )
-    (fp_line (start 0.8 1.15) (end 1.15 1.15) (layer "F.SilkS") (width 0.12))
-    (fp_line (start 1.15 1.15) (end 1.15 0.8) (layer "F.SilkS") (width 0.12))
     (fp_line (start -1.15 1.15) (end -1.15 0.8) (layer "F.SilkS") (width 0.12))
-    (fp_line (start 0.8 -1.15) (end 1.15 -1.15) (layer "F.SilkS") (width 0.12))
     (fp_line (start 1.15 -1.15) (end 1.15 -0.8) (layer "F.SilkS") (width 0.12))
-    (fp_line (start -0.8 -1.15) (end -1.35 -1.15) (layer "F.SilkS") (width 0.12))
     (fp_line (start -0.8 1.15) (end -1.15 1.15) (layer "F.SilkS") (width 0.12))
-    (fp_line (start -1.6 1.6) (end -1.6 -1.6) (layer "F.CrtYd") (width 0.05))
+    (fp_line (start 1.15 1.15) (end 1.15 0.8) (layer "F.SilkS") (width 0.12))
+    (fp_line (start -0.8 -1.15) (end -1.35 -1.15) (layer "F.SilkS") (width 0.12))
+    (fp_line (start 0.8 1.15) (end 1.15 1.15) (layer "F.SilkS") (width 0.12))
+    (fp_line (start 0.8 -1.15) (end 1.15 -1.15) (layer "F.SilkS") (width 0.12))
     (fp_line (start -1.6 -1.6) (end 1.6 -1.6) (layer "F.CrtYd") (width 0.05))
-    (fp_line (start 1.6 -1.6) (end 1.6 1.6) (layer "F.CrtYd") (width 0.05))
     (fp_line (start 1.6 1.6) (end -1.6 1.6) (layer "F.CrtYd") (width 0.05))
-    (fp_line (start -1 1) (end 1 1) (layer "F.Fab") (width 0.15))
+    (fp_line (start 1.6 -1.6) (end 1.6 1.6) (layer "F.CrtYd") (width 0.05))
+    (fp_line (start -1.6 1.6) (end -1.6 -1.6) (layer "F.CrtYd") (width 0.05))
     (fp_line (start 1 -1) (end -0.7 -1) (layer "F.Fab") (width 0.15))
     (fp_line (start -1 -0.7) (end -1 1) (layer "F.Fab") (width 0.15))
     (fp_line (start 1 1) (end 1 -1) (layer "F.Fab") (width 0.15))
+    (fp_line (start -1 1) (end 1 1) (layer "F.Fab") (width 0.15))
     (fp_line (start -0.7 -1) (end -1 -0.7) (layer "F.Fab") (width 0.15))
     (pad "1" smd oval (at -1.075 -0.4 180) (size 0.2 0.7) (layers "F.Cu" "F.Paste" "F.Mask")
@@
       (net 123 "+3.3VA") (pinfunction "AVDD") (pintype "unspecified"))
     (pad "13" smd rect (at 0 0 90) (size 1 1) (layers "F.Cu" "F.Paste" "F.Mask")
-      (net 2 "GND") (pinfunction "EP") (pintype "unspecified") (solder_paste_margin -0.75))
+      (net 2 "GND") (pinfunction "EP") (pintype "unspecified") (solder_paste_margin -0.1))
   )
   (footprint "Inductor_SMD:L_0603_1608Metric" (layer "F.Cu")
@@
     )
   )
-  (gr_line (start 120 132) (end 70 132) (layer "Edge.Cuts") (width 0.1))
-  (gr_line (start 70 177) (end 120 177) (layer "Edge.Cuts") (width 0.1))
-  (gr_line (start 120 132) (end 120 177) (layer "Edge.Cuts") (width 0.1))
-  (gr_line (start 70 132) (end 70 177) (layer "Edge.Cuts") (width 0.1))
+  (gr_line (start 117 132) (end 73 132) (layer "Edge.Cuts") (width 0.1))
+  (gr_arc (start 70 135) (mid 70.87868 132.87868) (end 73 132) (layer "Edge.Cuts") (width 0.1))
+  (gr_arc (start 120 174) (mid 119.12132 176.12132) (end 117 177) (layer "Edge.Cuts") (width 0.1))
+  (gr_line (start 73 177) (end 117 177) (layer "Edge.Cuts") (width 0.1))
+  (gr_arc (start 73 177) (mid 70.87868 176.12132) (end 70 174) (layer "Edge.Cuts") (width 0.1))
+  (gr_arc (start 117 132) (mid 119.12132 132.87868) (end 120 135) (layer "Edge.Cuts") (width 0.1))
+  (gr_line (start 120 135) (end 120 174) (layer "Edge.Cuts") (width 0.1))
+  (gr_line (start 70 135) (end 70 174) (layer "Edge.Cuts") (width 0.1))
+  (gr_text "MainCon V1.0" (at 111 161.25) (layer "B.SilkS")
+    (effects (font (size 1 1) (thickness 0.15)) (justify mirror))
+  )
+  (gr_text "MainCon	V1.0" (at 111.25 161.25) (layer "F.SilkS")
+    (effects (font (size 1 1) (thickness 0.15)))
+  )
+  (dimension (type aligned) (layer "Dwgs.User")
+    (pts (xy 117 132) (xy 117 177))
+    (height -9.4)
+    (gr_text "45,0000 mm" (at 125.25 154.5 90) (layer "Dwgs.User")
+      (effects (font (size 1 1) (thickness 0.15)))
+    )
+    (format (units 3) (units_format 1) (precision 4))
+    (style (thickness 0.15) (arrow_length 1.27) (text_position_mode 0) (extension_height 0.58642) (extension_offset 0.5) keep_text_aligned)
+  )
+  (dimension (type aligned) (layer "Dwgs.User")
+    (pts (xy 120 174) (xy 70 174))
+    (height -7.5)
+    (gr_text "50,0000 mm" (at 95 180.35) (layer "Dwgs.User")
+      (effects (font (size 1 1) (thickness 0.15)))
+    )
+    (format (units 3) (units_format 1) (precision 4))
+    (style (thickness 0.15) (arrow_length 1.27) (text_position_mode 0) (extension_height 0.58642) (extension_offset 0.5) keep_text_aligned)
+  )
   (segment (start 109.6 159.785) (end 109.6 159.8) (width 0.2) (layer "F.Cu") (net 1))
   (via (at 109.6 159.8) (size 0.5) (drill 0.2) (layers "F.Cu" "B.Cu") (net 1))
