File: hydCircCon/hydCircCon.kicad_sch (KiCad schematic)
At the start: 69 parts

Commit message: wip
Parts:
- removed C?: 100µ, Capacitor_THT:CP_Radial_D6.3mm_P2.50mm, symbol Device:C_Polarized
- removed J? (x3): Conn_01x03, Connector_Molex:Molex_KK-254_AE-6410-03A_1x03_P2.54mm_Vertical, symbol Connector_Generic:Conn_01x03
- removed R? (x3): 1k, Resistor_SMD:R_0603_1608Metric, symbol Device:R
- added H1, H2, H3, H4: MountingHole, MountingHole:MountingHole_3.2mm_M3_DIN965, symbol Mechanical:MountingHole
- added J16, J17, J9: Conn_01x02, Connector_JST:JST_EH_B2B-EH-A_1x02_P2.50mm_Vertical, symbol Connector_Generic:Conn_01x02
- added R18, R35: 1k, Resistor_SMD:R_0603_1608Metric, symbol Device:R
- J10: renamed from J?; footprint Connector_Molex:Molex_KK-254_AE-6410-03A_1x03_P2.54mm_Vertical -> Connector_JST:JST_EH_B3B-EH-A_1x03_P2.50mm_Vertical
- J8: renamed from J?; footprint Connector_PinSocket_2.54mm:PinSocket_1x02_P2.54mm_Vertical -> Connector_JST:JST_EH_B2B-EH-A_1x02_P2.50mm_Vertical
- L1: renamed from L?; footprint (none) -> Inductor_SMD:L_0603_1608Metric
- gave numbers to parts that had none: 59
Connections:
- net DIN2: now also R35.1
- net GND: now also J16.2 (Pin_2), J17.2 (Pin_2), J9.2 (Pin_2)
- net at C7.1, R17.1, U3.3 (+): now also J9.1 (Pin_1)
- new net: J16.1 (Pin_1), R35.2
- new net: J17.1 (Pin_1), R18.2
- new net DIN3: R18.1

Commit message: wip
Parts:
- added C39: 390p, Capacitor_SMD:C_0603_1608Metric, symbol Device:C
- added C40: 1µF, Capacitor_SMD:C_0603_1608Metric, symbol Device:C
- added R36: 56k, Resistor_SMD:R_0603_1608Metric, symbol Device:R
- added R37: 18k, Resistor_SMD:R_0603_1608Metric, symbol Device:R
- added U8: AP2127K-ADJ, Package_TO_SOT_SMD:SOT-23-5, symbol Regulator_Linear:AP2127K-ADJ
- L3: value 4.7u -> 6.8u; footprint Inductor_SMD:L_1008_2520Metric -> Inductor_SMD:L_Taiyo-Yuden_NR-30xx; HTN (none) -> NR3015T6R8M
- R19: value 27k -> 38k
- R21: value 91k -> 157k
Connections:
- net +3V3: now also C39.1, C40.1, R36.2, U8.5 (VOUT); no longer C19.2, C23.2, C25.2, L3.2, R21.1
- net +5V: now also C19.2, C23.2, C25.2, L3.2, R21.1, U8.1 (VIN), U8.3 (EN)
- net DIN1: now also U2.13 (GPIO10); no longer U2.11 (GPIO8)
- net DIN3: now also U2.11 (GPIO8)
- net GND: now also C40.2, R37.1, U8.2 (GND)
- net UART0: now also R10.2; no longer R11.2
- net UART1: now also R11.2; no longer R10.2
- net LED_PWM1 renamed pheri/LED_PWM1
- net LED_PWM2 renamed pheri/LED_PWM2
- new net: C39.2, R36.1, R37.2, U8.4 (ADJ)
Other:
- sheet pheri ports: added LED_PWM1, LED_PWM2; removed none
