File: hydCircCon/hydCircCon.kicad_pcb (KiCad board)
At the start: 2 copper layers, 50 x 50 mm, 109 parts, among them J1 USB_B_Micro, J10 Conn_01x03, J11 Conn_01x04, J12 Conn_01x02, J13 Conn_01x02, J14 Conn_01x03, J15 Conn_01x03, J16 Conn_01x02, J17 Conn_01x02, J2 Conn_01x03, J3 Conn_01x03, J4 Conn_01x03, J5 Conn_01x02, J6 Conn_01x03, J7 Conn_01x03, J8 Conn_01x02, J9 Conn_01x02, U1 W25Q16JVUXIQ, U2 RP2040, U3 MCP6001R, U4 AP63357Q, U5 TMP451, U6 DRV8231ADSGR, U7 DRV8231ADSGR, Y1 12Mhz

Commit message: wip
Parts:
- added C38: 10µ, Capacitor_SMD:C_1210_3225Metric, B.Cu at (177.9, 122.0)
- added C39: 390p, Capacitor_SMD:C_0603_1608Metric, B.Cu at (158.6, 100.8)
- added C40: 1µF, Capacitor_SMD:C_0603_1608Metric, B.Cu at (160.7, 103.5)
- added R36: 56k, Resistor_SMD:R_0603_1608Metric, B.Cu at (158.6, 102.0)
- added R37: 18k, Resistor_SMD:R_0603_1608Metric, B.Cu at (156.2, 104.7)
- added U8: AP2127K-ADJ, Package_TO_SOT_SMD:SOT-23-5, B.Cu at (158.3, 104.5)
- C1, C10, C11, C12, C13, C14, C15, C16, C17, C19, C2, C20, C21, C22, C23, C24, C25, C26, C27, C3, C36, C4, C6, C7, C8, C9, D1, L1, L2, R1, R10, R11, R12, R13, R14, R15, R16, R17, R18, R2, R20, R22, R23, R24, R27, R28, R3, R33, R34, R35, R8, U1, U3, U4, U5, Y1: moved to B.Cu
- L3: value 4.7u -> 6.8u; footprint Inductor_SMD:L_1008_2520Metric -> Inductor_SMD:L_Taiyo-Yuden_NR-30xx; moved to B.Cu
- R19: value 27k -> 38k; moved to B.Cu
- R21: value 91k -> 157k; moved to B.Cu
- moved J11 161.9 mm to (181.9, 88.2)
- moved J12 143.0 mm to (179.0, 95.3)
- moved R27 138.1 mm to (176.8, 94.0), turned to -90 degrees
- moved J10 138.1 mm to (171.6, 88.2)
- moved R28 135.9 mm to (176.8, 99.2), turned to 90 degrees
- moved C27 135.4 mm to (176.8, 96.6)
- moved C26 131.9 mm to (174.8, 94.9), turned to 180 degrees
- moved U5 131.9 mm to (174.8, 96.7), turned to 180 degrees
- moved R26 129.1 mm to (174.8, 96.8), turned to 180 degrees
- moved R25 128.5 mm to (174.8, 95.5), turned to 180 degrees
- moved U3 125.1 mm to (189.2, 91.2), turned to 180 degrees
- moved R16 124.1 mm to (186.6, 92.0), turned to -90 degrees
- moved C7 123.2 mm to (189.7, 93.3), turned to 180 degrees
- moved R17 122.6 mm to (191.7, 92.1), turned to 90 degrees
- moved J9 120.1 mm to (196.4, 95.3), turned to -90 degrees
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Connections:
- C19 pad 2: +3V3 -> +5V
- C23 pad 2: +3V3 -> +5V
- C25 pad 2: +3V3 -> +5V
- L3 pad 2: +3V3 -> +5V
- R10 pad 2: /UART1 -> /UART0
- R11 pad 2: /UART0 -> /UART1
- R21 pad 1: +3V3 -> +5V
- U2 pad 11: /DIN1 -> /DIN3
- U2 pad 13: unconnected-(U2-Pad13) -> /DIN1
- U2 pad 17: /LED_PWM1 -> /pheri/LED_PWM1
- U2 pad 18: /LED_PWM2 -> /pheri/LED_PWM2
Routing:
- net GND: track 0.00 -> 50.1 mm, vias 0 -> 54
- net /pheri/Isens0: track 0.00 -> 39.7 mm, vias 0 -> 1
- net +5V: track 0.00 -> 38.6 mm, vias 0 -> 8
- net /pheri/PWM0_Iref: track 0.00 -> 37.4 mm, vias 0 -> 1
- net /DIN3: track 0.00 -> 37.1 mm, vias 0 -> 1
- net /pheri/PWM_P0: track 0.00 -> 36.6 mm, vias 0 -> 1
- net /pheri/P_EN: track 0.00 -> 34.9 mm, vias 0 -> 1
- net /pheri/F0_Tach: track 0.00 -> 33.9 mm, vias 0 -> 1
- net +3V3: track 0.00 -> 32.0 mm, vias 0 -> 14
- net /DIN2: track 0.00 -> 31.7 mm, vias 0 -> 1
- net /pheri/F1_Tach: track 0.00 -> 28.3 mm, vias 0 -> 1
- net /pheri/SDA: track 0.00 -> 25.7 mm, vias 0 -> 2
- net /pheri/SCL: track 0.00 -> 25.3 mm, vias 0 -> 2
- net /pheri/LED_PWM2: track 0.00 -> 25.2 mm, vias 0 -> 2
- net /DIN1: track 0.00 -> 24.7 mm, vias 0 -> 1
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- added copper zone on B.Cu, net +24V
- added copper zone on F.Cu, net +24V
- added copper zone on B.Cu, net +3V3
- added copper zone on In2.Cu, net +3V3
- added copper zone on B.Cu, net +5V
- added copper zone on B.Cu, net /pheri/VM
- added copper zone on F.Cu, net /pheri/VM
- added copper zone on B.Cu, net GND
- added copper zone on F.Cu, net GND
- added copper zone on In1.Cu, net GND
- added copper zone on B.Cu, net Net-(C14-Pad1)
- added copper zone on F.Cu, net Net-(C32-Pad2)
- added copper zone on F.Cu, net Net-(C33-Pad2)
- added copper zone on B.Cu, net Net-(C8-Pad2)
- added copper zone on B.Cu, net Net-(J13-Pad2)
- added copper zone on B.Cu, net Net-(J14-Pad1)
- added copper zone on B.Cu, net Net-(L4-Pad1)
- added copper zone on F.Cu, net Net-(L4-Pad1)
- added copper zone on B.Cu, net Net-(L5-Pad1)
- added copper zone on F.Cu, net Net-(L5-Pad1)
Other:
- board size 50 x 50 mm -> 50 x 40 mm
- copper layers 2 -> 4

Commit message: prepare for Manufacturing
Other:
- outline, holes or cut-outs redrawn
- rule pad_to_mask_clearance: 0 -> 0.05
- board text added: "HydCircCon V1.0"
Changed lines of the file:
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@@
       (dielectric_constraints no)
     )
-    (pad_to_mask_clearance 0)
+    (pad_to_mask_clearance 0.05)
+    (solder_mask_min_width 0.1)
+    (aux_axis_origin 148.25 126.5)
+    (grid_origin 148.25 126.5)
     (pcbplotparams
       (layerselection 0x00010fc_ffffffff)
@@
     )
   )
-  (gr_line (start 148.25 86.5) (end 148.25 126.5) (layer "Edge.Cuts") (width 0.1))
-  (gr_line (start 198.25 86.5) (end 148.25 86.5) (layer "Edge.Cuts") (width 0.1))
-  (gr_line (start 198.25 86.5) (end 198.25 126.5) (layer "Edge.Cuts") (width 0.1))
-  (gr_line (start 198.25 126.5) (end 148.25 126.5) (layer "Edge.Cuts") (width 0.1))
+  (gr_line (start 148.25 89.5) (end 148.25 123.5) (layer "Edge.Cuts") (width 0.1))
+  (gr_line (start 195.25 86.5) (end 151.25 86.5) (layer "Edge.Cuts") (width 0.1))
+  (gr_line (start 198.25 89.5) (end 198.25 123.5) (layer "Edge.Cuts") (width 0.1))
+  (gr_arc (start 151.25 126.5) (mid 149.12868 125.62132) (end 148.25 123.5) (layer "Edge.Cuts") (width 0.1))
+  (gr_arc (start 198.25 123.5) (mid 197.37132 125.62132) (end 195.25 126.5) (layer "Edge.Cuts") (width 0.1))
+  (gr_arc (start 148.25 89.5) (mid 149.12868 87.37868) (end 151.25 86.5) (layer "Edge.Cuts") (width 0.1))
+  (gr_arc (start 195.25 86.5) (mid 197.37132 87.37868) (end 198.25 89.5) (layer "Edge.Cuts") (width 0.1))
+  (gr_line (start 195.25 126.5) (end 151.25 126.5) (layer "Edge.Cuts") (width 0.1))
+  (gr_text "HydCircCon\nV1.0" (at 171.85 97.3 -90) (layer "B.SilkS")
+    (effects (font (size 1 1) (thickness 0.15)) (justify mirror))
+  )
+  (gr_text "HydCircCon\nV1.0" (at 171.95 96 270) (layer "F.SilkS")
+    (effects (font (size 1 1) (thickness 0.15)))
+  )
+  (dimension (type orthogonal) (layer "Dwgs.User")
+    (pts (xy 148.25 89.5) (xy 198.25 89.6))
+    (height -14.6)
+    (orientation 0)
+    (gr_text "50,0000 mm" (at 173.25 73.75) (layer "Dwgs.User")
+      (effects (font (size 1 1) (thickness 0.15)))
+    )
+    (format (units 3) (units_format 1) (precision 4))
+    (style (thickness 0.15) (arrow_length 1.27) (text_position_mode 0) (extension_height 0.58642) (extension_offset 0.5) keep_text_aligned)
+  )
+  (dimension (type orthogonal) (layer "Dwgs.User")
+    (pts (xy 151.25 123.5) (xy 151.25 89.5))
+    (height -9.3)
+    (orientation 1)
+    (gr_text "34,0000 mm" (at 140.8 106.5 90) (layer "Dwgs.User")
+      (effects (font (size 1 1) (thickness 0.15)))
+    )
+    (format (units 3) (units_format 1) (precision 4))
+    (style (thickness 0.15) (arrow_length 1.27) (text_position_mode 0) (extension_height 0.58642) (extension_offset 0.5) keep_text_aligned)
+  )
+  (dimension (type orthogonal) (layer "Dwgs.User")
+    (pts (xy 151.25 126.5) (xy 152.35 86.5))
+    (height -14.3)
+    (orientation 1)
+    (gr_text "40,0000 mm" (at 135.8 106.5 90) (layer "Dwgs.User")
+      (effects (font (size 1 1) (thickness 0.15)))
+    )
+    (format (units 3) (units_format 1) (precision 4))
+    (style (thickness 0.15) (arrow_length 1.27) (text_position_mode 0) (extension_height 0.58642) (extension_offset 0.5) keep_text_aligned)
+  )
+  (dimension (type orthogonal) (layer "Dwgs.User")
+    (pts (xy 151.25 89.5) (xy 195.25 89.5))
+    (height -9.5)
+    (orientation 0)
+    (gr_text "44,0000 mm" (at 173.25 78.85) (layer "Dwgs.User")
+      (effects (font (size 1 1) (thickness 0.15)))
+    )
+    (format (units 3) (units_format 1) (precision 4))
+    (style (thickness 0.15) (arrow_length 1.27) (text_position_mode 0) (extension_height 0.58642) (extension_offset 0.5) keep_text_aligned)
+  )
   (segment (start 165.05 100.1125) (end 165.05 99.45) (width 0.2) (layer "F.Cu") (net 1))
   (segment (start 165.05 99.45) (end 164.8 99.2) (width 0.2) (layer "F.Cu") (net 1))
@@
   (segment (start 162.502979 93.647021) (end 162.502979 92.502979) (width 0.127) (layer "B.Cu") (net 57))
   (segment (start 163.175 90.425) (end 163.35 90.425) (width 0.127) (layer "B.Cu") (net 57))
-  (segment (start 163.375 88.525) (end 163.375 88.3) (width 0.2) (layer "F.Cu") (net 58))
   (segment (start 162.7 89.5) (end 162.4 89.5) (width 0.2) (layer "F.Cu") (net 58))
   (segment (start 160.55 95.9) (end 160.825104 95.9) (width 0.2) (layer "F.Cu") (net 58))
