File: DualValveCon/DualValveCon.kicad_sch (KiCad schematic)
At the start: 48 parts

Commit message: wip
Parts:
- added C? (x2): 10µ, Capacitor_SMD:C_1210_3225Metric, symbol Device:C
- added C?: 1µF, Capacitor_SMD:C_0603_1608Metric, symbol Device:C
- added C? (x4): 100nF, Capacitor_SMD:C_0603_1608Metric, symbol Device:C
- added C? (x2): DNP, Capacitor_SMD:C_0603_1608Metric, symbol Device:C
- added J? (x2): Conn_01x02, Connector_PinSocket_2.54mm:PinSocket_1x02_P2.54mm_Vertical, symbol Connector_Generic:Conn_01x02
- added L?: 600R, symbol Device:L_Ferrite
- added R? (x2): 1.1k, Resistor_SMD:R_0603_1608Metric, symbol Device:R
- added R? (x2): 10k, Resistor_SMD:R_0603_1608Metric, symbol Device:R
Connections:
- net +24V: now also U?.5 (VM), U?.5 (VM), C?.2, C?.2
- net +3V3: now also U?.1 (VDD), U?.1 (VDD), C?.1, C?.1, L?.2; no longer U?.43 (ADC_AVDD)
- net GND: now also U?.2 (VSS), U?.2 (VSS), U?.5 (EP), U?.5 (EP), U?.7 (GND), U?.7 (GND), U?.9 (EP), U?.9 (EP), C?.1, C?.1, C?.2, C?.2, C?.2, C?.2, C?.2, C?.2, C?.2, R?.2, R?.2
- net UART0: now also U?.6 (GPIO4), U?.7 (GPIO5); no longer U?.40 (GPIO28_ADC2), U?.41 (GPIO29_ADC3)
- net UART1: now also U?.2 (GPIO0), U?.3 (GPIO1); no longer U?.36 (GPIO24), U?.37 (GPIO25)
- net V2_Isens: now reaches U?.1 (IPROPI)
- net V2_Isens: now also C?.1, R?.1
- net V2_IN2: now reaches U?.2 (IN2)
- net V2_IN1: now reaches U?.3 (IN1)
- net at U?.4 (VREF): now also C?.1, R?.1 (x2)
- net at U?.6 (OUT1): now also J?.1 (Pin_1) (x2)
- net at U?.8 (OUT2): now also J?.2 (Pin_2) (x2)
- net V1_Isens: now reaches U?.1 (IPROPI)
- net V1_Isens: now also C?.1, R?.1
- net V1_IN2: now reaches U?.2 (IN2)
- net V1_IN1: now reaches U?.3 (IN1)
- net V1_PosS: now reaches U?.3 (OUT_S)
- net V1_PosN: now reaches U?.4 (OUT_N)
- net V2_PosS: now reaches U?.3 (OUT_S)
- net V2_PosN: now reaches U?.4 (OUT_N)
- new net: C?.1, L?.1, U?.43 (ADC_AVDD)
- new net V1_IRef: R?.2
- new net V2_IRef: R?.2
Other:
- moved on the sheet: C?, L?, R?, U?

Commit message: wip
Parts:
- removed C?: 10µ, Capacitor_SMD:C_1210_3225Metric, symbol Device:C
- removed C? (x2): 100nF, Capacitor_SMD:C_0603_1608Metric, symbol Device:C
- removed C? (x2): DNP, Capacitor_SMD:C_0603_1608Metric, symbol Device:C
- removed D?: BAT54W, Diode_SMD:D_SOD-323, symbol Device:D_Filled
- removed D?: Green, LED_SMD:LED_0603_1608Metric, symbol Device:LED_Filled
- removed J? (x2): Conn_01x02, Connector_PinSocket_2.54mm:PinSocket_1x02_P2.54mm_Vertical, symbol Connector_Generic:Conn_01x02
- removed R?: 470R, Resistor_SMD:R_0603_1608Metric, symbol Device:R
- removed R? (x2): 1.1k, Resistor_SMD:R_0603_1608Metric, symbol Device:R
- removed R? (x3): 10k, Resistor_SMD:R_0603_1608Metric, symbol Device:R
- removed R?: 5.6k, Resistor_SMD:R_0603_1608Metric, symbol Device:R
- removed U? (x2): DRV8231ADSGR, Package_SON:WSON-8-1EP_2x2mm_P0.5mm_EP0.9x1.6mm, symbol Bergi:DRV8231ADSGR
- added D? (x2): Yellow, LED_SMD:LED_0603_1608Metric, symbol Device:LED_Filled
- added D? (x3): Green, LED_SMD:LED_0603_1608Metric, symbol Device:LED_Filled
- added D?: BAT54W, Diode_SMD:D_SOD-323, symbol Device:D_Filled
- added L?: 1µ, Inductor_SMD:L_0805_2012Metric, symbol Device:L_Ferrite
- added R? (x5): 470R, Resistor_SMD:R_0603_1608Metric, symbol Device:R
- added R? (x2): 20R, Resistor_SMD:R_0603_1608Metric, symbol Device:R
- added R?: 10k, Resistor_SMD:R_0603_1608Metric, symbol Device:R
- added R?: 5.6k, Resistor_SMD:R_0603_1608Metric, symbol Device:R
Connections:
- net +24V: now also D?.1 (K), L?.2; no longer C?.2, U?.1 (VIN), U?.2 (EN)
- net +3V3: now also R?.2, R?.2, R?.2, R?.2
- net GND: now also D?.1 (K), R?.2
- net V1_PosN: now also U?.15 (GPIO12)
- net V1_PosS: now also U?.14 (GPIO11)
- net V2_PosN: now also U?.17 (GPIO14)
- net V2_PosS: now also U?.16 (GPIO13)
- net VBUS: now also R?.1, R?.2, R?.2
- net at U?.11 (GPIO8): now also R?.1
- net at U?.12 (GPIO9): now also R?.1, R?.2
- net motorDriver/PWM1A: now reaches U?.27 (GPIO16)
- net motorDriver/PWM1B: now reaches U?.28 (GPIO17)
- net motorDriver/PWM2A: now reaches U?.29 (GPIO18)
- net motorDriver/PWM2B: now reaches U?.30 (GPIO19)
- net motorDriver/PWM1_Iref: now reaches U?.31 (GPIO20)
- net motorDriver/PWM2_Iref: now reaches U?.32 (GPIO21)
- net motorDriver/Isens1: now reaches U?.38 (GPIO26_ADC0)
- net motorDriver/Isens2: now reaches U?.39 (GPIO27_ADC1)
- net at U?.4 (GPIO2): now also D?.2 (A)
- net at U?.5 (GPIO3): now also D?.2 (A)
- net at U?.8 (GPIO6): now also D?.2 (A)
- net at U?.9 (GPIO7): now also D?.2 (A)
- new net: D?.1 (K), R?.1 (x4)
- new net: D?.2 (A), R?.1, R?.1
- new net: C?.2, L?.1, U?.1 (VIN), U?.2 (EN)
- new net: D?.2 (A), R?.2
Other:
- added sheet motorDriver (motorDriver.kicad_sch)

Commit message: wip
Parts:
- removed D?: Green, LED_SMD:LED_0603_1608Metric, symbol Device:LED_Filled
- removed R?: 470R, Resistor_SMD:R_0603_1608Metric, symbol Device:R
- removed R?: 10k, Resistor_SMD:R_0603_1608Metric, symbol Device:R
- removed R?: 5.6k, Resistor_SMD:R_0603_1608Metric, symbol Device:R
- added D?: Green, LED_SMD:LED_0603_1608Metric, symbol Device:LED_Filled
- added R?: 10k, Resistor_SMD:R_0603_1608Metric, symbol Device:R
- added R?: 5.6k, Resistor_SMD:R_0603_1608Metric, symbol Device:R
- added R?: 470R, Resistor_SMD:R_0603_1608Metric, symbol Device:R
- L?: value 1µ -> 10µ
Connections:
- net GND: now also D?.1 (K), R?.2
- net VBUS: now also R?.1
- net at U?.11 (GPIO8): now also R?.1
- net at U?.12 (GPIO9): now also R?.1, R?.2
- new net: D?.2 (A), R?.2

Commit message: wip
Parts:
- added H1, H2, H3, H4: MountingHole, MountingHole:MountingHole_3.2mm_M3_DIN965, symbol Mechanical:MountingHole
- C12, C17: renamed from C?; footprint Capacitor_SMD:C_0603_1608Metric -> Capacitor_SMD:C_0402_1005Metric
- L1: renamed from L?; footprint (none) -> Inductor_SMD:L_0603_1608Metric
- gave numbers to parts that had none: 59
Connections:
- net UART0: now also U2.40 (GPIO28_ADC2), U2.41 (GPIO29_ADC3); no longer U2.6 (GPIO4), U2.7 (GPIO5)
- net UART1: now also U2.36 (GPIO24), U2.37 (GPIO25); no longer U2.2 (GPIO0), U2.3 (GPIO1)
- net V1_PosN: now also U2.12 (GPIO9); no longer U2.15 (GPIO12)
- net V1_PosS: now also U2.13 (GPIO10); no longer U2.14 (GPIO11)
- net V2_PosN: now also U2.6 (GPIO4); no longer U2.17 (GPIO14)
- net V2_PosS: now also U2.7 (GPIO5); no longer U2.16 (GPIO13)
- net at R14.1: now also J5.3 (Pin_3); no longer J4.3 (Pin_3)
- net at R12.2, R13.1: now also U2.35 (GPIO23); no longer U2.12 (GPIO9)
- net at U2.11 (GPIO8): now also D6.2 (A); no longer R7.1
- net at U2.4 (GPIO2): now also R7.1; no longer D2.2 (A)
- net at D5.2 (A): now also U2.14 (GPIO11); no longer U2.8 (GPIO6)
- net at U2.9 (GPIO7): no longer D6.2 (A)
- net at R15.1: now also J4.3 (Pin_3); no longer J5.3 (Pin_3)
- new net: D2.2 (A), U2.8 (GPIO6)
Other:
- note added: "PWM0A PWM0B"
- note added: "PWM1A PWM1B"
- note added: "PWM2A PWM2B"
- moved on the sheet: D2, D3, D4, D5, D6, R10, R11, R12, R13, R14, R15, R7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
