File: DualValveCon/DualValveCon.kicad_pcb (KiCad board)
At the start: 2 copper layers, 82 x 50 mm, 82 parts, among them J1 USB_B_Micro, J2 Conn_01x03, J3 Conn_01x02, J4 Conn_01x03, J5 Conn_01x03, J6 Conn_01x02, J7 Conn_01x02, U1 W25Q16JVUXIQ, U2 RP2040, U3 AP63357Q, U4 MHA100KN, U5 MHA100KN, U6 DRV8231ADSGR, U7 DRV8231ADSGR, Y1 12Mhz

Commit message: prepare for Manufacturing
Routing:
- net Net-(D2-Pad1): track 9.42 -> 8.72 mm
Other:
- outline, holes or cut-outs redrawn
- rule pad_to_mask_clearance: 0 -> 0.05
- board text added: "DualValveCon V1.0"
Changed lines of the file:
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@@
       (dielectric_constraints no)
     )
-    (pad_to_mask_clearance 0)
+    (pad_to_mask_clearance 0.05)
+    (solder_mask_min_width 0.1)
+    (aux_axis_origin 126 112)
+    (grid_origin 126 112)
     (pcbplotparams
       (layerselection 0x00010fc_ffffffff)
@@
   (gr_line (start 137 102) (end 138 102) (layer "Dwgs.User") (width 0.15))
   (gr_line (start 147 102) (end 148 102) (layer "Dwgs.User") (width 0.15))
-  (gr_line (start 201 84) (end 194 84) (layer "Edge.Cuts") (width 0.1))
-  (gr_line (start 126 84) (end 119 84) (layer "Edge.Cuts") (width 0.1))
+  (gr_line (start 201 84) (end 196 84) (layer "Edge.Cuts") (width 0.1))
+  (gr_line (start 124 84) (end 119 84) (layer "Edge.Cuts") (width 0.1))
   (gr_line (start 126 62) (end 194 62) (layer "Edge.Cuts") (width 0.1))
   (gr_line (start 201 90) (end 201 84) (layer "Edge.Cuts") (width 0.1))
+  (gr_arc (start 124 90) (mid 125.414214 90.585786) (end 126 92) (layer "Edge.Cuts") (width 0.1))
   (gr_line (start 119 84) (end 119 90) (layer "Edge.Cuts") (width 0.1))
-  (gr_line (start 119 90) (end 126 90) (layer "Edge.Cuts") (width 0.1))
-  (gr_line (start 194 90) (end 194 112) (layer "Edge.Cuts") (width 0.1))
-  (gr_line (start 194 84) (end 194 62) (layer "Edge.Cuts") (width 0.1))
-  (gr_line (start 126 84) (end 126 62) (layer "Edge.Cuts") (width 0.1))
+  (gr_line (start 119 90) (end 124 90) (layer "Edge.Cuts") (width 0.1))
+  (gr_arc (start 126 82) (mid 125.414214 83.414214) (end 124 84) (layer "Edge.Cuts") (width 0.1))
+  (gr_line (start 194 92) (end 194 112) (layer "Edge.Cuts") (width 0.1))
+  (gr_line (start 194 82) (end 194 62) (layer "Edge.Cuts") (width 0.1))
+  (gr_line (start 126 82) (end 126 62) (layer "Edge.Cuts") (width 0.1))
   (gr_line (start 194 112) (end 126 112) (layer "Edge.Cuts") (width 0.1))
-  (gr_line (start 126 112) (end 126 90) (layer "Edge.Cuts") (width 0.1))
-  (gr_line (start 194 90) (end 201 90) (layer "Edge.Cuts") (width 0.1))
+  (gr_arc (start 194 92) (mid 194.585786 90.585786) (end 196 90) (layer "Edge.Cuts") (width 0.1))
+  (gr_line (start 126 112) (end 126 92) (layer "Edge.Cuts") (width 0.1))
+  (gr_arc (start 196 84) (mid 194.585786 83.414214) (end 194 82) (layer "Edge.Cuts") (width 0.1))
+  (gr_line (start 196 90) (end 201 90) (layer "Edge.Cuts") (width 0.1))
+  (gr_text "DualValveCon V1.0" (at 161 110) (layer "B.SilkS")
+    (effects (font (size 1 1) (thickness 0.15)) (justify mirror))
+  )
+  (gr_text "DualValveCon V1.0" (at 161 110) (layer "F.SilkS")
+    (effects (font (size 1 1) (thickness 0.15)))
+  )
   (dimension (type aligned) (layer "Dwgs.User")
     (pts (xy 193 97) (xy 193 112))
@@
   (segment (start 143 92.1375) (end 143 94.025) (width 0.2) (layer "F.Cu") (net 4))
   (segment (start 145 85.2625) (end 145 84.833263) (width 0.2) (layer "F.Cu") (net 4))
-  (segment (start 135.5 75.275) (end 135.7 75.075) (width 0.5) (layer "F.Cu") (net 4))
   (segment (start 149.373 69.227) (end 149.85 68.75) (width 1) (layer "F.Cu") (net 4))
   (segment (start 146.2375 89.7) (end 147.1 89.7) (width 0.2) (layer "F.Cu") (net 4))
@@
   (segment (start 127 97.7875) (end 135.6625 97.7875) (width 0.2) (layer "F.Cu") (net 20))
   (segment (start 135.6625 97.7875) (end 135.7 97.825) (width 0.2) (layer "F.Cu") (net 20))
-  (segment (start 135.7 97.825) (end 135 97.825) (width 0.2) (layer "F.Cu") (net 20))
   (segment (start 135.8 67.675) (end 135.8 63.2875) (width 0.2) (layer "F.Cu") (net 21))
   (segment (start 135.8 63.2875) (end 135.3125 62.8) (width 0.2) (layer "F.Cu") (net 21))
