File: FluidPresenceSensor/AntennaL/FPS_AL.kicad_pcb (KiCad board)
At the start: 2 copper layers, 26.5 x 10.5 mm, 9 parts, among them K1 capPad, K2 capPad, K3 capPad, K4 capPad, K5 capPad, K6 capPad, K7 capPad, K8 capPad, K9 capPad

Commit message: prepare for Manufacturing
Other:
- outline, holes or cut-outs redrawn
- rule pad_to_mask_clearance: 0 -> 0.05
- board text added: "FPC_AntennaL V1.0"
Changed lines of the file:
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@@
       (dielectric_constraints no)
     )
-    (pad_to_mask_clearance 0)
+    (pad_to_mask_clearance 0.05)
+    (solder_mask_min_width 0.1)
+    (aux_axis_origin 83.8 70.75)
+    (grid_origin 83.8 70.75)
     (pcbplotparams
       (layerselection 0x00010fc_ffffffff)
@@
       (net 3 "Net-(K3-Pad1)") (pinfunction "Pin_1") (pintype "passive"))
   )
-  (gr_line (start 90.05 60.25) (end 90.05 61.75) (layer "Edge.Cuts") (width 0.1))
-  (gr_line (start 83.8 70.75) (end 83.8 61.75) (layer "Edge.Cuts") (width 0.1))
-  (gr_line (start 104.05 61.75) (end 104.05 60.25) (layer "Edge.Cuts") (width 0.1))
-  (gr_line (start 110.3 70.75) (end 83.8 70.75) (layer "Edge.Cuts") (width 0.1))
-  (gr_line (start 90.05 61.75) (end 83.8 61.75) (layer "Edge.Cuts") (width 0.1))
+  (gr_line (start 90.05 60.25) (end 90.05 61.25) (layer "Edge.Cuts") (width 0.1))
+  (gr_line (start 83.8 70) (end 83.8 61.75) (layer "Edge.Cuts") (width 0.1))
+  (gr_arc (start 104.55 61.75) (mid 104.196447 61.603553) (end 104.05 61.25) (layer "Edge.Cuts") (width 0.1))
+  (gr_line (start 104.05 61.25) (end 104.05 60.25) (layer "Edge.Cuts") (width 0.1))
+  (gr_line (start 109.55 70.75) (end 84.55 70.75) (layer "Edge.Cuts") (width 0.1))
+  (gr_arc (start 84.55 70.75) (mid 84.01967 70.53033) (end 83.8 70) (layer "Edge.Cuts") (width 0.1))
+  (gr_line (start 89.55 61.75) (end 83.8 61.75) (layer "Edge.Cuts") (width 0.1))
   (gr_line (start 104.05 60.25) (end 90.05 60.25) (layer "Edge.Cuts") (width 0.1))
-  (gr_line (start 110.3 70.75) (end 110.3 61.75) (layer "Edge.Cuts") (width 0.1))
-  (gr_line (start 104.05 61.75) (end 110.3 61.75) (layer "Edge.Cuts") (width 0.1))
+  (gr_arc (start 110.3 70) (mid 110.08033 70.53033) (end 109.55 70.75) (layer "Edge.Cuts") (width 0.1))
+  (gr_line (start 110.3 70) (end 110.3 61.75) (layer "Edge.Cuts") (width 0.1))
+  (gr_arc (start 90.05 61.25) (mid 89.903553 61.603553) (end 89.55 61.75) (layer "Edge.Cuts") (width 0.1))
+  (gr_line (start 104.55 61.75) (end 110.3 61.75) (layer "Edge.Cuts") (width 0.1))
+  (gr_text "FPC_AntennaL V1.0" (at 96.8 66.75) (layer "B.SilkS")
+    (effects (font (size 1 1) (thickness 0.15)) (justify mirror))
+  )
+  (gr_text "FPC_AntennaL V1.0" (at 97.05 66.75) (layer "F.SilkS")
+    (effects (font (size 1 1) (thickness 0.15)))
+  )
+  (dimension (type aligned) (layer "Dwgs.User")
+    (pts (xy 83.8 70.75) (xy 110.3 70.75))
+    (height 3.25)
+    (gr_text "26,5000 mm" (at 97.05 72.85) (layer "Dwgs.User")
+      (effects (font (size 1 1) (thickness 0.15)))
+    )
+    (format (units 3) (units_format 1) (precision 4))
+    (style (thickness 0.15) (arrow_length 1.27) (text_position_mode 0) (extension_height 0.58642) (extension_offset 0.5) keep_text_aligned)
+  )
+  (dimension (type orthogonal) (layer "Dwgs.User")
+    (pts (xy 90.05 60.25) (xy 104.05 60.25))
+    (height -2.95)
+    (orientation 0)
+    (gr_text "14,0000 mm" (at 97.05 56.15) (layer "Dwgs.User")
+      (effects (font (size 1 1) (thickness 0.15)))
+    )
+    (format (units 3) (units_format 1) (precision 4))
+    (style (thickness 0.15) (arrow_length 1.27) (text_position_mode 0) (extension_height 0.58642) (extension_offset 0.5) keep_text_aligned)
+  )
+  (dimension (type orthogonal) (layer "Dwgs.User")
+    (pts (xy 90.05 60.25) (xy 83.8 70.75))
+    (height -8.65)
+    (orientation 1)
+    (gr_text "10,5000 mm" (at 80.25 65.5 90) (layer "Dwgs.User")
+      (effects (font (size 1 1) (thickness 0.15)))
+    )
+    (format (units 3) (units_format 1) (precision 4))
+    (style (thickness 0.15) (arrow_length 1.27) (text_position_mode 0) (extension_height 0.58642) (extension_offset 0.5) keep_text_aligned)
+  )
+  (dimension (type orthogonal) (layer "Dwgs.User")
+    (pts (xy 90.05 61.75) (xy 90.05 60.25))
+    (height -6.65)
+    (orientation 1)
+    (gr_text "1,5000 mm" (at 82.25 61 90) (layer "Dwgs.User")
+      (effects (font (size 1 1) (thickness 0.15)))
+    )
+    (format (units 3) (units_format 1) (precision 4))
+    (style (thickness 0.15) (arrow_length 1.27) (text_position_mode 0) (extension_height 0.58642) (extension_offset 0.5) keep_text_aligned)
+  )
   (segment (start 87 66.75) (end 90.8 66.75) (width 0.127) (layer "F.Cu") (net 1))
   (segment (start 86.05 62.55) (end 86.05 65.8) (width 0.127) (layer "F.Cu") (net 1))
