File: FluidPresenceSensor/AntennaR/FPS_AR.kicad_pcb (KiCad board)
At the start: 2 copper layers, 26.5 x 10.5 mm, 9 parts, among them K1 capPad, K2 capPad, K3 capPad, K4 capPad, K5 capPad, K6 capPad, K7 capPad, K8 capPad, K9 capPad

Commit message: prepare for Manufacturing
Other:
- outline, holes or cut-outs redrawn
- rule pad_to_mask_clearance: 0 -> 0.05
- board text added: "FPC_AntennaR V1.0"
Changed lines of the file:
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@@
       (dielectric_constraints no)
     )
-    (pad_to_mask_clearance 0)
+    (pad_to_mask_clearance 0.05)
+    (solder_mask_min_width 0.1)
+    (aux_axis_origin 98.6 81.5)
+    (grid_origin 98.6 81.5)
     (pcbplotparams
       (layerselection 0x00010fc_ffffffff)
@@
       (net 4 "Net-(K8-Pad1)") (pinfunction "Pin_1") (pintype "passive"))
   )
-  (gr_line (start 104.85 81.5) (end 98.6 81.5) (layer "Edge.Cuts") (width 0.1))
-  (gr_line (start 125.1 81.5) (end 125.1 72.5) (layer "Edge.Cuts") (width 0.1))
-  (gr_line (start 98.6 81.5) (end 98.6 72.5) (layer "Edge.Cuts") (width 0.1))
-  (gr_line (start 104.85 81.5) (end 104.85 83) (layer "Edge.Cuts") (width 0.1))
+  (gr_arc (start 124.35 72.5) (mid 124.88033 72.71967) (end 125.1 73.25) (layer "Edge.Cuts") (width 0.1))
+  (gr_arc (start 118.85 82) (mid 118.996447 81.646447) (end 119.35 81.5) (layer "Edge.Cuts") (width 0.1))
+  (gr_line (start 104.35 81.5) (end 98.6 81.5) (layer "Edge.Cuts") (width 0.1))
+  (gr_line (start 125.1 81.5) (end 125.1 73.25) (layer "Edge.Cuts") (width 0.1))
+  (gr_arc (start 98.6 73.25) (mid 98.81967 72.71967) (end 99.35 72.5) (layer "Edge.Cuts") (width 0.1))
+  (gr_line (start 98.6 81.5) (end 98.6 73.25) (layer "Edge.Cuts") (width 0.1))
+  (gr_line (start 104.85 82) (end 104.85 83) (layer "Edge.Cuts") (width 0.1))
   (gr_line (start 104.85 83) (end 118.85 83) (layer "Edge.Cuts") (width 0.1))
-  (gr_line (start 118.85 83) (end 118.85 81.5) (layer "Edge.Cuts") (width 0.1))
-  (gr_line (start 118.85 81.5) (end 125.1 81.5) (layer "Edge.Cuts") (width 0.1))
-  (gr_line (start 98.6 72.5) (end 125.1 72.5) (layer "Edge.Cuts") (width 0.1))
+  (gr_arc (start 104.35 81.5) (mid 104.703553 81.646447) (end 104.85 82) (layer "Edge.Cuts") (width 0.1))
+  (gr_line (start 118.85 83) (end 118.85 82) (layer "Edge.Cuts") (width 0.1))
+  (gr_line (start 119.35 81.5) (end 125.1 81.5) (layer "Edge.Cuts") (width 0.1))
+  (gr_line (start 99.35 72.5) (end 124.35 72.5) (layer "Edge.Cuts") (width 0.1))
+  (gr_text "FPC_AntennaR V1.0" (at 112.1 76.5) (layer "B.SilkS")
+    (effects (font (size 1 1) (thickness 0.15)) (justify mirror))
+  )
+  (gr_text "FPC_AntennaR V1.0" (at 111.85 76.5) (layer "F.SilkS")
+    (effects (font (size 1 1) (thickness 0.15)))
+  )
+  (dimension (type orthogonal) (layer "Dwgs.User")
+    (pts (xy 104.85 83) (xy 118.85 83))
+    (height 5)
+    (orientation 0)
+    (gr_text "14,0000 mm" (at 111.85 86.85) (layer "Dwgs.User")
+      (effects (font (size 1 1) (thickness 0.15)))
+    )
+    (format (units 3) (units_format 1) (precision 4))
+    (style (thickness 0.15) (arrow_length 1.27) (text_position_mode 0) (extension_height 0.58642) (extension_offset 0.5) keep_text_aligned)
+  )
+  (dimension (type orthogonal) (layer "Dwgs.User")
+    (pts (xy 104.85 83) (xy 99.35 72.5))
+    (height -12.25)
+    (orientation 1)
+    (gr_text "10,5000 mm" (at 91.45 77.75 90) (layer "Dwgs.User")
+      (effects (font (size 1 1) (thickness 0.15)))
+    )
+    (format (units 3) (units_format 1) (precision 4))
+    (style (thickness 0.15) (arrow_length 1.27) (text_position_mode 0) (extension_height 0.58642) (extension_offset 0.5) keep_text_aligned)
+  )
+  (dimension (type orthogonal) (layer "Dwgs.User")
+    (pts (xy 98.6 81.5) (xy 125.1 81.5))
+    (height 10.5)
+    (orientation 0)
+    (gr_text "26,5000 mm" (at 111.85 90.85) (layer "Dwgs.User")
+      (effects (font (size 1 1) (thickness 0.15)))
+    )
+    (format (units 3) (units_format 1) (precision 4))
+    (style (thickness 0.15) (arrow_length 1.27) (text_position_mode 0) (extension_height 0.58642) (extension_offset 0.5) keep_text_aligned)
+  )
+  (dimension (type orthogonal) (layer "Dwgs.User")
+    (pts (xy 104.85 83) (xy 104.35 81.5))
+    (height -8.75)
+    (orientation 1)
+    (gr_text "1,5000 mm" (at 94.95 82.25 90) (layer "Dwgs.User")
+      (effects (font (size 1 1) (thickness 0.15)))
+    )
+    (format (units 3) (units_format 1) (precision 4))
+    (style (thickness 0.15) (arrow_length 1.27) (text_position_mode 0) (extension_height 0.58642) (extension_offset 0.5) keep_text_aligned)
+  )
   (segment (start 100.85 76.95) (end 101.3 76.5) (width 0.127) (layer "F.Cu") (net 1))
   (segment (start 101.3 76.5) (end 105.6 76.5) (width 0.127) (layer "F.Cu") (net 1))
