File: FluidPresenceSensor/BasePcb/FluidPresenceSensor.kicad_pcb (KiCad board)
At the start: 4 copper layers, 40 x 63 mm, 131 parts, among them J1 USB_B_Micro, J2 Conn_01x03, J3 Conn_01x03, J4 Conn_01x03, J5 Conn_01x02, K1 capPad, K10 capPad, K11 capPad, K12 capPad, K13 capPad, K14 capPad, K15 capPad, K16 capPad, K17 capPad, K18 capPad, K19 capPad, K2 capPad, K20 capPad, K21 capPad, K22 capPad, K3 capPad, K4 capPad, K41 capPad, K42 capPad, K43 capPad, K44 capPad, K45 capPad, K46 capPad, K47 capPad, K48 capPad, K49 capPad, K5 capPad, K50 capPad, K51 capPad, K52 capPad, K53 capPad, K54 capPad, K55 capPad, K56 capPad, K57 capPad, K58 capPad, K59 capPad, K6 capPad, K60 capPad, K61 capPad, K62 capPad, K63 capPad, K64 capPad, K65 capPad, K66 capPad, K67 capPad, K68 capPad, K69 capPad, K7 capPad, K70 capPad, K71 capPad, K72 capPad, K73 capPad, K74 capPad, K75 capPad, K76 capPad, K77 capPad, K78 capPad, K8 capPad, K9 capPad, U1 W25Q16JVUXIQ, U2 RP2040, U3 AP63357Q, Y1 12Mhz

Commit message: prepare for Manufacturing
Other:
- outline, holes or cut-outs redrawn
- board text added: "FluidPresenceSensor V1.0"
