File: PressureSensor/PressureSensor.kicad_pcb (KiCad board)
At the start: 2 copper layers, 10 x 10 mm, 6 parts, among them J1 Conn_01x01, J2 Conn_01x01, J3 Conn_01x01, J4 Conn_01x01, U1 ILPS22QS

Commit message: prepare for Manufacturing
Other:
- board text added: "V1.0"
Changed lines of the file:
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@@
   (gr_circle (center 163 74) (end 163 71) (layer "Dwgs.User") (width 0.15) (fill none))
   (gr_circle (center 163 74) (end 168 74) (layer "Edge.Cuts") (width 0.1) (fill none))
+  (gr_text "V1.0" (at 163.2 70.8) (layer "F.SilkS")
+    (effects (font (size 1.5 1.5) (thickness 0.3)))
+  )
+  (dimension (type aligned) (layer "Dwgs.User")
+    (pts (xy 163 69) (xy 163 79))
+    (height -8)
+    (gr_text "10,0000 mm" (at 169.85 74 90) (layer "Dwgs.User")
+      (effects (font (size 1 1) (thickness 0.15)))
+    )
+    (format (units 3) (units_format 1) (precision 4))
+    (style (thickness 0.15) (arrow_length 1.27) (text_position_mode 0) (extension_height 0.58642) (extension_offset 0.5) keep_text_aligned)
+  )
   (segment (start 162.5 76.1) (end 162.4 76.1) (width 0.2) (layer "F.Cu") (net 1))
   (segment (start 162.4 76.1) (end 162 75.7) (width 0.2) (layer "F.Cu") (net 1))
@@
   (segment (start 162.184199 73.769037) (end 162.184199 73.315801) (width 0.2) (layer "F.Cu") (net 3))
   (segment (start 161 73.8) (end 162.153236 73.8) (width 0.2) (layer "F.Cu") (net 3))
-  (segment (start 162.184199 73.384199) (end 162 73.2) (width 0.2) (layer "F.Cu") (net 3))
-  (segment (start 162.184199 73.315801) (end 162.315801 73.184199) (width 0.2) (layer "F.Cu") (net 3))
+  (segment (start 160.9 73.7) (end 160.9 74.5) (width 0.2) (layer "F.Cu") (net 3))
   (segment (start 162.315801 73.184199) (end 162.518974 73.184199) (width 0.2) (layer "F.Cu") (net 3))
   (segment (start 160.9 73.7) (end 161 73.8) (width 0.2) (layer "F.Cu") (net 3))
@@
   (segment (start 164.2 74.615162) (end 163.854001 74.269163) (width 0.2) (layer "F.Cu") (net 3))
   (segment (start 162.518974 73.184199) (end 162.015801 73.184199) (width 0.2) (layer "F.Cu") (net 3))
-  (segment (start 162.015801 73.184199) (end 162 73.2) (width 0.2) (layer "F.Cu") (net 3))
   (segment (start 164.2 75.1) (end 164.2 74.615162) (width 0.2) (layer "F.Cu") (net 3))
   (via (at 160.9 73.7) (size 0.5) (drill 0.2) (layers "F.Cu" "B.Cu") (net 3))
@@
   (via (at 160.9 74.5) (size 0.5) (drill 0.2) (layers "F.Cu" "B.Cu") (net 3))
   (segment (start 164.2 75.1) (end 163.025 75.1) (width 0.2) (layer "B.Cu") (net 3))
+  (segment (start 162.125 74.2) (end 162.125 73.178984) (width 0.2) (layer "B.Cu") (net 3))
+  (segment (start 162.151992 73.151992) (end 161.848008 73.151992) (width 0.5) (layer "B.Cu") (net 3))
   (segment (start 161.848008 73.151992) (end 160.9 74.1) (width 0.5) (layer "B.Cu") (net 3))
-  (segment (start 162.125 73.178984) (end 162.151992 73.151992) (width 0.2) (layer "B.Cu") (net 3))
-  (segment (start 162.125 74.2) (end 162.125 73.178984) (width 0.2) (layer "B.Cu") (net 3))
-  (segment (start 162.125 73.325) (end 162 73.2) (width 0.5) (layer "B.Cu") (net 3))
   (segment (start 163.025 75.1) (end 162.125 74.2) (width 0.2) (layer "B.Cu") (net 3))
-  (segment (start 162.151992 73.151992) (end 161.848008 73.151992) (width 0.5) (layer "B.Cu") (net 3))
   (segment (start 163.4 71.9) (end 163.0191 72.2809) (width 0.2) (layer "F.Cu") (net 4))
   (segment (start 163.130963 73.769037) (end 163.0191 73.8809) (width 0.2) (layer "F.Cu") (net 4))
