File: reservoirCon/reservoirCon.kicad_pcb (KiCad board)
At the start: 4 copper layers, 30 x 30 mm, 70 parts, among them J1 USB_B_Micro, J10 Conn_01x02, J2 Conn_01x03, J3 Conn_01x02, J4 Conn_01x04, J5 Conn_01x03, J6 Conn_01x03, J7 Conn_01x02, J8 Conn_01x02, J9 Conn_01x02, U1 W25Q16JVUXIQ, U2 RP2040, U3 MCP6001R, U4 AP63357Q, Y1 12Mhz

Commit message: prepare for Manufacturing
Routing:
- net +24V: track 8.19 -> 21.2 mm
Other:
- outline, holes or cut-outs redrawn
- rule pad_to_mask_clearance: 0 -> 0.05
- board text added: "ReservoirCon V1.0"
Changed lines of the file:
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@@
       (dielectric_constraints no)
     )
-    (pad_to_mask_clearance 0)
+    (pad_to_mask_clearance 0.05)
+    (solder_mask_min_width 0.1)
+    (aux_axis_origin 137.4 124)
+    (grid_origin 137.4 124)
     (pcbplotparams
       (layerselection 0x00010fc_ffffffff)
@@
     )
   )
-  (gr_line (start 137.4 94) (end 167.4 94) (layer "Edge.Cuts") (width 0.1))
-  (gr_line (start 137.4 124) (end 137.4 94) (layer "Edge.Cuts") (width 0.1))
-  (gr_line (start 137.4 124) (end 167.4 124) (layer "Edge.Cuts") (width 0.1))
-  (gr_line (start 167.4 124) (end 167.4 94) (layer "Edge.Cuts") (width 0.1))
+  (gr_arc (start 164.4 94) (mid 166.52132 94.87868) (end 167.4 97) (layer "Edge.Cuts") (width 0.1))
+  (gr_arc (start 167.4 121) (mid 166.52132 123.12132) (end 164.4 124) (layer "Edge.Cuts") (width 0.1))
+  (gr_arc (start 137.4 97) (mid 138.27868 94.87868) (end 140.4 94) (layer "Edge.Cuts") (width 0.1))
+  (gr_line (start 140.4 94) (end 164.4 94) (layer "Edge.Cuts") (width 0.1))
+  (gr_arc (start 140.4 124) (mid 138.27868 123.12132) (end 137.4 121) (layer "Edge.Cuts") (width 0.1))
+  (gr_line (start 137.4 121) (end 137.4 97) (layer "Edge.Cuts") (width 0.1))
+  (gr_line (start 140.4 124) (end 164.4 124) (layer "Edge.Cuts") (width 0.1))
+  (gr_line (start 167.4 121) (end 167.4 97) (layer "Edge.Cuts") (width 0.1))
+  (gr_text "ReservoirCon\nV1.0" (at 143.4 108 -90) (layer "B.SilkS")
+    (effects (font (size 1 1) (thickness 0.15)) (justify mirror))
+  )
+  (gr_text "ReservoirCon\nV1.0" (at 155.4 101 270) (layer "F.SilkS")
+    (effects (font (size 1 1) (thickness 0.15)))
+  )
+  (dimension (type aligned) (layer "Dwgs.User")
+    (pts (xy 140.4 94) (xy 140.4 124))
+    (height 6.999999)
+    (gr_text "30,0000 mm" (at 132.250001 109 90) (layer "Dwgs.User")
+      (effects (font (size 1 1) (thickness 0.15)))
+    )
+    (format (units 3) (units_format 1) (precision 4))
+    (style (thickness 0.15) (arrow_length 1.27) (text_position_mode 0) (extension_height 0.58642) (extension_offset 0.5) keep_text_aligned)
+  )
+  (dimension (type aligned) (layer "Dwgs.User")
+    (pts (xy 137.4 97) (xy 167.4 97))
+    (height -7)
+    (gr_text "30,0000 mm" (at 152.4 88.85) (layer "Dwgs.User")
+      (effects (font (size 1 1) (thickness 0.15)))
+    )
+    (format (units 3) (units_format 1) (precision 4))
+    (style (thickness 0.15) (arrow_length 1.27) (text_position_mode 0) (extension_height 0.58642) (extension_offset 0.5) keep_text_aligned)
+  )
   (segment (start 149.5 109.4) (end 149.5 110.2375) (width 0.2) (layer "F.Cu") (net 1))
   (segment (start 149.6 109.3) (end 149.5 109.4) (width 0.2) (layer "F.Cu") (net 1))
@@
   (via (at 147.5 112) (size 0.5) (drill 0.2) (layers "F.Cu" "B.Cu") (free) (net 6))
   (via (at 149.3 112) (size 0.5) (drill 0.2) (layers "F.Cu" "B.Cu") (free) (net 6))
+  (segment (start 143.5 111) (end 142.6 111.9) (width 2) (layer "B.Cu") (net 6))
+  (segment (start 140.42 103.9) (end 142.5 103.9) (width 2) (layer "B.Cu") (net 6))
+  (segment (start 142.5 103.9) (end 143.5 104.9) (width 2) (layer "B.Cu") (net 6))
   (segment (start 141 103.9) (end 140.42 103.9) (width 0.3) (layer "B.Cu") (net 6))
+  (segment (start 143.5 104.9) (end 143.5 111) (width 2) (layer "B.Cu") (net 6))
   (segment (start 145.5 99.4) (end 141 103.9) (width 0.3) (layer "B.Cu") (net 6))
   (segment (start 146.75 99.4) (end 145.5 99.4) (width 0.3) (layer "B.Cu") (net 6))
+  (segment (start 142.6 111.9) (end 140.42 111.9) (width 2) (layer "B.Cu") (net 6))
   (segment (start 164.82125 101.5825) (end 164.82125 101.2625) (width 0.25) (layer "F.Cu") (net 7))
   (segment (start 164.875 101.075) (end 164.1 100.3) (width 0.25) (layer "F.Cu") (net 7))
@@
         (xy 149.3 117.2)
         (xy 147.1 117.2)
-        (xy 146 116.1)
-        (xy 146 115.7)
+        (xy 146.2 116.3)
+        (xy 146.2 115.7)
         (xy 149.4 115.7)
       )
