File: reservoirCon/reservoirCon.kicad_sch (KiCad schematic)
At the start: 60 parts

Commit message: wip
Parts:
- added J?: Conn_01x02, Connector_PinSocket_2.54mm:PinSocket_1x02_P2.54mm_Vertical, symbol Connector_Generic:Conn_01x02
- added R? (x2): 10k, Resistor_SMD:R_0603_1608Metric, symbol Device:R
- added R?: 1k, Resistor_SMD:R_0603_1608Metric, symbol Device:R
Connections:
- net +3V3: now also R?.2, R?.2
- net DIN2: now also R?.1; no longer R?.1
- net GND: now also J?.2 (Pin_2)
- net DIN3: now reaches U?.13 (GPIO10)
- net DIN3: now also R?.1
- net at J?.1 (Pin_1), U?.14 (GPIO11): now also R?.1
- net at J?.2 (Pin_2), U?.15 (GPIO12): now also R?.1
- new net: J?.1 (Pin_1), R?.2
Changed lines of the file:
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@@
 (kicad_sch (version 20211123) (generator eeschema)
   (paper "A4")
+  (junction (at 119.38 91.44) (diameter 0) (color 0 0 0 0)
+  )
   (junction (at 208.28 27.94) (diameter 0) (color 0 0 0 0)
   )
@@
   (junction (at 181.61 140.97) (diameter 0) (color 0 0 0 0)
   )
+  (junction (at 123.19 88.9) (diameter 0) (color 0 0 0 0)
+  )
   (junction (at 39.37 58.42) (diameter 0) (color 0 0 0 0)
   )
+  (junction (at 123.19 78.74) (diameter 0) (color 0 0 0 0)
+  )
   (junction (at 267.97 29.21) (diameter 0) (color 0 0 0 0)
   )
@@
     (stroke (width 0) (type default) (color 0 0 0 0))
   )
+  (wire (pts (xy 123.19 88.9) (xy 125.73 88.9))
+    (stroke (width 0) (type default) (color 0 0 0 0))
+  )
   (wire (pts (xy 50.8 138.43) (xy 50.8 137.16))
     (stroke (width 0) (type default) (color 0 0 0 0))
@@
     (stroke (width 0) (type default) (color 0 0 0 0))
   )
+  (wire (pts (xy 119.38 78.74) (xy 123.19 78.74))
+    (stroke (width 0) (type default) (color 0 0 0 0))
+  )
   (wire (pts (xy 39.37 167.64) (xy 39.37 173.99))
     (stroke (width 0) (type default) (color 0 0 0 0))
@@
     (stroke (width 0) (type default) (color 0 0 0 0))
   )
+  (wire (pts (xy 119.38 86.36) (xy 119.38 91.44))
+    (stroke (width 0) (type default) (color 0 0 0 0))
+  )
   (wire (pts (xy 201.93 41.91) (xy 201.93 39.37))
     (stroke (width 0) (type default) (color 0 0 0 0))
@@
     (stroke (width 0) (type default) (color 0 0 0 0))
   )
+  (wire (pts (xy 119.38 91.44) (xy 125.73 91.44))
+    (stroke (width 0) (type default) (color 0 0 0 0))
+  )
   (wire (pts (xy 31.75 63.5) (xy 31.75 58.42))
     (stroke (width 0) (type default) (color 0 0 0 0))
@@
     (stroke (width 0) (type default) (color 0 0 0 0))
   )
-  (wire (pts (xy 104.14 91.44) (xy 125.73 91.44))
+  (wire (pts (xy 104.14 91.44) (xy 119.38 91.44))
     (stroke (width 0) (type default) (color 0 0 0 0))
   )
@@
     (stroke (width 0) (type default) (color 0 0 0 0))
   )
-  (wire (pts (xy 104.14 88.9) (xy 125.73 88.9))
+  (wire (pts (xy 104.14 88.9) (xy 123.19 88.9))
     (stroke (width 0) (type default) (color 0 0 0 0))
   )
   (wire (pts (xy 104.14 71.12) (xy 104.14 73.66))
+    (stroke (width 0) (type default) (color 0 0 0 0))
+  )
+  (wire (pts (xy 123.19 86.36) (xy 123.19 88.9))
     (stroke (width 0) (type default) (color 0 0 0 0))
   )
@@
     (effects (font (size 1.27 1.27)) (justify right bottom))
   )
-  (label "DIN2" (at 199.39 137.16 180)
+  (label "DIN3" (at 199.39 137.16 180)
     (effects (font (size 1.27 1.27)) (justify right bottom))
   )
@@
     (effects (font (size 1.27 1.27)) (justify left bottom))
   )
+  (label "DIN3" (at 104.14 86.36 0)
+    (effects (font (size 1.27 1.27)) (justify left bottom))
+  )
   (label "UART1" (at 104.14 63.5 0)
     (effects (font (size 1.27 1.27)) (justify left bottom))
@@
   (label "LeakSens" (at 104.14 137.16 0)
     (effects (font (size 1.27 1.27)) (justify left bottom))
+  )
+  (label "DIN2" (at 177.8 92.71 180)
+    (effects (font (size 1.27 1.27)) (justify right bottom))
   )
   (label "UART1" (at 132.08 173.99 180)
@@
     (pin "1")
   )
+  (symbol (lib_id "power:GND") (at 185.42 95.25 0) (unit 1)
+    (in_bom yes) (on_board yes)
+    (property "Reference" "#PWR?" (id 0) (at 185.42 101.6 0)
+      (effects (font (size 1.27 1.27)) hide)
+    )
+    (property "Value" "GND" (id 1) (at 185.42 99.06 0))
+    (property "Footprint" "" (id 2) (at 185.42 95.25 0)
+      (effects (font (size 1.27 1.27)) hide)
+    )
+    (property "Datasheet" "" (id 3) (at 185.42 95.25 0)
+      (effects (font (size 1.27 1.27)) hide)
+    )
+    (pin "1")
+  )
   (symbol (lib_id "Device:L_Ferrite") (at 86.36 41.91 180) (unit 1)
     (in_bom yes) (on_board yes) (fields_autoplaced)
@@
     (pin "1")
   )
+  (symbol (lib_id "Device:R") (at 119.38 82.55 180) (unit 1)
+    (in_bom yes) (on_board yes)
+    (property "Reference" "R?" (id 0) (at 116.84 82.55 90))
+    (property "Value" "10k" (id 1) (at 119.38 82.55 90))
+    (property "Footprint" "Resistor_SMD:R_0603_1608Metric" (id 2) (at 121.158 82.55 90)
+      (effects (font (size 1.27 1.27)) hide)
+    )
+    (property "Datasheet" "~" (id 3) (at 119.38 82.55 0)
+      (effects (font (size 1.27 1.27)) hide)
+    )
+    (pin "1")
+    (pin "2")
+  )
+  (symbol (lib_id "power:+3V3") (at 123.19 78.74 0) (mirror y) (unit 1)
+    (in_bom yes) (on_board yes)
+    (property "Reference" "#PWR?" (id 0) (at 123.19 82.55 0)
+      (effects (font (size 1.27 1.27)) hide)
+    )
+    (property "Value" "+3V3" (id 1) (at 123.19 74.93 0))
+    (property "Footprint" "" (id 2) (at 123.19 78.74 0)
+      (effects (font (size 1.27 1.27)) hide)
+    )
+    (property "Datasheet" "" (id 3) (at 123.19 78.74 0)
+      (effects (font (size 1.27 1.27)) hide)
+    )
+    (pin "1")
+  )
   (symbol (lib_id "power:GND") (at 267.97 44.45 0) (unit 1)
     (in_bom yes) (on_board yes) (fields_autoplaced)
@@
     )
     (property "Datasheet" "~" (id 3) (at 201.93 35.56 0)
+      (effects (font (size 1.27 1.27)) hide)
+    )
+    (pin "1")
+    (pin "2")
+  )
+  (symbol (lib_id "Device:R") (at 181.61 92.71 90) (unit 1)
+    (in_bom yes) (on_board yes)
+    (property "Reference" "R?" (id 0) (at 181.61 90.17 90))
+    (property "Value" "1k" (id 1) (at 181.61 92.71 90))
+    (property "Footprint" "Resistor_SMD:R_0603_1608Metric" (id 2) (at 181.61 94.488 90)
+      (effects (font (size 1.27 1.27)) hide)
+    )
+    (property "Datasheet" "~" (id 3) (at 181.61 92.71 0)
       (effects (font (size 1.27 1.27)) hide)
     )
@@
     (pin "2")
   )
+  (symbol (lib_id "Connector_Generic:Conn_01x02") (at 190.5 92.71 0) (unit 1)
+    (in_bom yes) (on_board yes) (fields_autoplaced)
+    (property "Reference" "J?" (id 0) (at 193.04 92.7099 0)
+      (effects (font (size 1.27 1.27)) (justify left))
+    )
+    (property "Value" "Conn_01x02" (id 1) (at 193.04 95.2499 0)
+      (effects (font (size 1.27 1.27)) (justify left))
+    )
+    (property "Footprint" "Connector_PinSocket_2.54mm:PinSocket_1x02_P2.54mm_Vertical" (id 2) (at 190.5 92.71 0)
+      (effects (font (size 1.27 1.27)) hide)
+    )
+    (property "Datasheet" "~" (id 3) (at 190.5 92.71 0)
+      (effects (font (size 1.27 1.27)) hide)
+    )
+    (pin "1")
+    (pin "2")
+  )
   (symbol (lib_id "Device:R") (at 172.72 140.97 90) (unit 1)
     (in_bom yes) (on_board yes)
@@
     (pin "1")
   )
+  (symbol (lib_id "Device:R") (at 123.19 82.55 180) (unit 1)
+    (in_bom yes) (on_board yes)
+    (property "Reference" "R?" (id 0) (at 125.73 82.55 90))
+    (property "Value" "10k" (id 1) (at 123.19 82.55 90))
+    (property "Footprint" "Resistor_SMD:R_0603_1608Metric" (id 2) (at 124.968 82.55 90)
+      (effects (font (size 1.27 1.27)) hide)
+    )
+    (property "Datasheet" "~" (id 3) (at 123.19 82.55 0)
+      (effects (font (size 1.27 1.27)) hide)
+    )
+    (pin "1")
+    (pin "2")
+  )
   (symbol (lib_id "power:GND") (at 151.13 179.07 270) (unit 1)
     (in_bom yes) (on_board yes)
@@
       (reference "#PWR?") (unit 1) (value "GND") (footprint "")
     )
+    (path "/06ae5956-707b-4a9a-a12c-cce220a42550"
+      (reference "#PWR?") (unit 1) (value "GND") (footprint "")
+    )
     (path "/097a60d7-3467-434a-bf97-911595800c7a"
       (reference "#PWR?") (unit 1) (value "GND") (footprint "")
@@
       (reference "#PWR?") (unit 1) (value "GND") (footprint "")
     )
+    (path "/43c36972-9dc2-4123-87f2-06360f1c335f"
+      (reference "#PWR?") (unit 1) (value "+3V3") (footprint "")
+    )
     (path "/43c4d2e5-dca7-4f2f-b606-cfe41b9aa6fc"
       (reference "#PWR?") (unit 1) (value "GND") (footprint "")
@@
       (reference "J?") (unit 1) (value "Conn_01x03") (footprint "Connector_Molex:Molex_KK-254_AE-6410-03A_1x03_P2.54mm_Vertical")
     )
+    (path "/938f8a57-6622-48e2-9d6d-065d4934ec13"
+      (reference "J?") (unit 1) (value "Conn_01x02") (footprint "Connector_PinSocket_2.54mm:PinSocket_1x02_P2.54mm_Vertical")
+    )
     (path "/b9946f79-cf85-4420-a0ba-077ac7862238"
       (reference "J?") (unit 1) (value "Conn_01x03") (footprint "Connector_Molex:Molex_KK-254_AE-6410-03A_1x03_P2.54mm_Vertical")
@@
       (reference "R?") (unit 1) (value "10k") (footprint "Resistor_SMD:R_0603_1608Metric")
     )
+    (path "/4295c6e2-301a-4f08-b53d-9bb876079985"
+      (reference "R?") (unit 1) (value "10k") (footprint "Resistor_SMD:R_0603_1608Metric")
+    )
     (path "/567af4ae-252f-444f-94ee-f6b6ec2e58a0"
       (reference "R?") (unit 1) (value "470R") (footprint "Resistor_SMD:R_0603_1608Metric")
     )
+    (path "/5f9f5e8e-b342-4ce2-9f8c-1e0e47781028"
+      (reference "R?") (unit 1) (value "1k") (footprint "Resistor_SMD:R_0603_1608Metric")
+    )
     (path "/6462e071-137c-4a10-8535-8e24bc919c18"
       (reference "R?") (unit 1) (value "1M") (footprint "Resistor_SMD:R_0603_1608Metric")
@@
       (reference "R?") (unit 1) (value "1k") (footprint "Resistor_SMD:R_0603_1608Metric")
     )
+    (path "/e7bdf424-0f27-4fe4-9baf-7ea9fd28b9b5"
+      (reference "R?") (unit 1) (value "10k") (footprint "Resistor_SMD:R_0603_1608Metric")
+    )
     (path "/fc25f40d-768a-4b30-b5ea-e04fcd5bea41"

Commit message: wip
Parts:
- gave numbers to parts that had none: 64

Commit message: wip
Parts:
- removed J9: Conn_01x03, Connector_Molex:Molex_KK-254_AE-6410-03A_1x03_P2.54mm_Vertical, symbol Connector_Generic:Conn_01x03
- added C24: 100nF, Capacitor_SMD:C_0603_1608Metric, symbol Device:C
- added H1, H2, H3, H4: MountingHole, MountingHole:MountingHole_3.2mm_M3_DIN965, symbol Mechanical:MountingHole
- added J10, J9: Conn_01x02, Connector_JST:JST_EH_B2B-EH-A_1x02_P2.50mm_Vertical, symbol Connector_Generic:Conn_01x02
- J4: footprint (none) -> Connector_JST:JST_EH_B4B-EH-A_1x04_P2.50mm_Vertical
- J7, J8: footprint Connector_PinSocket_2.54mm:PinSocket_1x02_P2.54mm_Vertical -> Connector_JST:JST_EH_B2B-EH-A_1x02_P2.50mm_Vertical
- L1: footprint (none) -> Inductor_SMD:L_0603_1608Metric
Connections:
- net +3V3: now also C24.1
- net DIN1: now also U2.36 (GPIO24); no longer U2.11 (GPIO8)
- net DIN2: now also U2.35 (GPIO23); no longer U2.12 (GPIO9)
- net DIN3: now also U2.34 (GPIO22); no longer U2.13 (GPIO10)
- net GND: now also C24.2, J10.2 (Pin_2), J9.2 (Pin_2)
- net at U2.4 (GPIO2): no longer R7.1
- net at R19.2: now also J9.1 (Pin_1)
- net at C6.1, R18.1, U3.3 (+): now also J10.1 (Pin_1)
- new net LED: R7.1, U2.13 (GPIO10)
Other:
- moved on the sheet: D2, R19, R7
