File: Hardware/FluidPresenceSensor/BasePcb/capSens.kicad_sch (KiCad schematic)
At the start: 80 parts, among them K1 capPad, K10 capPad, K11 capPad, K12 capPad, K13 capPad, K14 capPad, K15 capPad, K16 capPad, K17 capPad, K18 capPad, K19 capPad, K2 capPad, K20 capPad, K21 capPad, K22 capPad, K3 capPad, K4 capPad, K41 capPad, K42 capPad, K43 capPad, K44 capPad, K45 capPad, K46 capPad, K47 capPad, K48 capPad, K49 capPad, K5 capPad, K50 capPad, K51 capPad, K52 capPad, K53 capPad, K54 capPad, K55 capPad, K56 capPad, K57 capPad, K58 capPad, K59 capPad, K6 capPad, K60 capPad, K61 capPad, K62 capPad, K63 capPad, K64 capPad, K65 capPad, K66 capPad, K67 capPad, K68 capPad, K69 capPad, K7 capPad, K70 capPad, K71 capPad, K72 capPad, K73 capPad, K74 capPad, K75 capPad, K76 capPad, K77 capPad, K78 capPad, K8 capPad, K9 capPad

Commit message: wip
Parts:
- C4, C5: value 100n -> 10n
- R5, R6: value 1k -> 81R
Changed lines of the file:
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@@
       (effects (font (size 1.27 1.27)) (justify right))
     )
-    (property "Value" "1k" (id 1) (at 158.75 58.42 90)
+    (property "Value" "81R" (id 1) (at 158.75 58.42 90)
       (effects (font (size 1.27 1.27)) (justify right))
     )
@@
       (effects (font (size 1.27 1.27)) (justify right))
     )
-    (property "Value" "1k" (id 1) (at 158.75 60.96 90)
+    (property "Value" "81R" (id 1) (at 158.75 60.96 90)
       (effects (font (size 1.27 1.27)) (justify right))
     )
@@
       (effects (font (size 1.27 1.27)) (justify right))
     )
-    (property "Value" "100n" (id 1) (at 177.8 54.61 0)
+    (property "Value" "10n" (id 1) (at 177.8 54.61 0)
       (effects (font (size 1.27 1.27)) (justify right))
     )
@@
       (effects (font (size 1.27 1.27)) (justify right))
     )
-    (property "Value" "100n" (id 1) (at 168.91 54.61 0)
-      (effects (font (size 1.27 1.27)) (justify right))
-    )
+    (property "Value" "10n" (id 1) (at 168.91 54.61 0)
+      (effects (font (size 1.27 1.27)) (justify right))
+    )
