File: Hardware/DualValveCon/DualValveCon.kicad_sch (KiCad schematic)
At the start: 66 parts, among them J1 USB_B_Micro, J2 Conn_01x03, J3 Conn_01x02, J4 Conn_01x03, J5 Conn_01x03, U1 W25Q16JVUXIQ, U2 RP2040, U3 AP63357Q, U4 MHA100KN, U5 MHA100KN, Y1 12Mhz

Commit message: wip
Parts:
- D2, D5: value Green -> red
- L1: value 600R -> 22uH
- R1, R2: value 20R -> 10R
- R14, R15: value 1k -> 100R
Changed lines of the file:
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@@
       (effects (font (size 1.27 1.27)) (justify right))
     )
-    (property "Value" "600R" (id 1) (at 90.17 43.1799 0)
+    (property "Value" "22uH" (id 1) (at 90.17 43.1799 0)
       (effects (font (size 1.27 1.27)) (justify right))
     )
@@
       (effects (font (size 1.27 1.27)) (justify right))
     )
-    (property "Value" "1k" (id 1) (at 158.75 151.13 90)
+    (property "Value" "100R" (id 1) (at 160.02 151.13 90)
       (effects (font (size 1.27 1.27)) (justify right))
     )
@@
       (effects (font (size 1.27 1.27)) (justify right))
     )
-    (property "Value" "20R" (id 1) (at 39.37 63.5 90)
+    (property "Value" "10R" (id 1) (at 39.37 63.5 90)
       (effects (font (size 1.27 1.27)) (justify right))
     )
@@
       (effects (font (size 1.27 1.27)) (justify right))
     )
-    (property "Value" "20R" (id 1) (at 39.37 58.42 90)
+    (property "Value" "10R" (id 1) (at 39.37 58.42 90)
       (effects (font (size 1.27 1.27)) (justify right))
     )
@@
     (in_bom yes) (on_board yes)
     (property "Reference" "D5" (id 0) (at 162.56 59.69 0))
-    (property "Value" "Green" (id 1) (at 161.29 54.61 0))
+    (property "Value" "red" (id 1) (at 161.29 54.61 0))
     (property "Footprint" "LED_SMD:LED_0603_1608Metric" (id 2) (at 165.1 57.15 0)
       (effects (font (size 1.27 1.27)) hide)
@@
     (in_bom yes) (on_board yes)
     (property "Reference" "D2" (id 0) (at 146.05 59.69 0))
-    (property "Value" "Green" (id 1) (at 144.78 54.61 0))
+    (property "Value" "red" (id 1) (at 144.78 54.61 0))
     (property "Footprint" "LED_SMD:LED_0603_1608Metric" (id 2) (at 148.59 57.15 0)
       (effects (font (size 1.27 1.27)) hide)
@@
       (effects (font (size 1.27 1.27)) (justify right))
     )
-    (property "Value" "1k" (id 1) (at 158.75 140.97 90)
+    (property "Value" "100R" (id 1) (at 160.02 140.97 90)
       (effects (font (size 1.27 1.27)) (justify right))
     )
@@
     )
     (path "/92ebece5-f029-40b4-9292-c2dc77e6dabc"
-      (reference "D2") (unit 1) (value "Green") (footprint "LED_SMD:LED_0603_1608Metric")
+      (reference "D2") (unit 1) (value "red") (footprint "LED_SMD:LED_0603_1608Metric")
     )
     (path "/f8f10886-3b6c-4e22-a63f-f0a82f09200d"
@@
     )
     (path "/71927b46-ada4-4e15-b493-b800e53cc089"
-      (reference "D5") (unit 1) (value "Green") (footprint "LED_SMD:LED_0603_1608Metric")
+      (reference "D5") (unit 1) (value "red") (footprint "LED_SMD:LED_0603_1608Metric")
     )
     (path "/6a009069-99bb-4809-b57a-c8285f00205b"
@@
     )
     (path "/01443907-a10f-48eb-84b8-03c86efac89b"
-      (reference "L1") (unit 1) (value "600R") (footprint "Inductor_SMD:L_0603_1608Metric")
+      (reference "L1") (unit 1) (value "22uH") (footprint "Inductor_SMD:L_0603_1608Metric")
     )
     (path "/232d1454-bc9c-4835-a6b7-e8e9071904ee"
@@
     )
     (path "/2d0f0fc5-8692-4d86-92a2-27280a3b39ee"
-      (reference "R1") (unit 1) (value "20R") (footprint "Resistor_SMD:R_0603_1608Metric")
+      (reference "R1") (unit 1) (value "10R") (footprint "Resistor_SMD:R_0603_1608Metric")
     )
     (path "/20f6488f-7f82-48f9-a32e-a63c9f8ffe3c"
-      (reference "R2") (unit 1) (value "20R") (footprint "Resistor_SMD:R_0603_1608Metric")
+      (reference "R2") (unit 1) (value "10R") (footprint "Resistor_SMD:R_0603_1608Metric")
     )
     (path "/1d87027e-5601-4c9a-9961-59bcc8def247"
@@
     )
     (path "/11e7c2fc-97ea-4b1c-9dac-b6a19fe2b44f"
-      (reference "R14") (unit 1) (value "1k") (footprint "Resistor_SMD:R_0603_1608Metric")
+      (reference "R14") (unit 1) (value "100R") (footprint "Resistor_SMD:R_0603_1608Metric")
     )
     (path "/fd4aa458-da66-4856-ab10-ff957768e780"
-      (reference "R15") (unit 1) (value "1k") (footprint "Resistor_SMD:R_0603_1608Metric")
+      (reference "R15") (unit 1) (value "100R") (footprint "Resistor_SMD:R_0603_1608Metric")
     )
     (path "/e6afa010-749a-4975-bf50-cf6ca677fcf7"

Commit message: wip
Other:
- note added: "Notiz für V2.0: -) Spannunsgmessung 24V sinvvol"
Changed lines of the file:
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@@
+    (effects (font (size 1.27 1.27)) (justify left bottom))
+  )
+  (text "Notiz für V2.0:\n-) Spannunsgmessung 24V sinvvol" (at 97.79 162.56 0)
     (effects (font (size 1.27 1.27)) (justify left bottom))
   )
