File: Hardware/LED-Balken/LED-Treiber/Treiber.kicad_pcb (KiCad board)
At the start: 2 copper layers, 279.5 x 36.6 mm, 46 parts, among them J1 Conn_01x01_Female, J2 Conn_01x01_Female, J3 Conn_01x01_Female, J4 Conn_01x01_Female, J5 Conn_01x01_Female, J6 Conn_01x01_Female, U1 TPS92200DxRXL

Commit message: added FlatTVS
Parts:
- added U2: TVS2700DRV, Package_SON:WSON-6-1EP_2x2mm_P0.65mm_EP1x1.6mm, F.Cu at (359.9, 103.2)
- R1: value 0R18 -> 0R36
- moved J3 2.23 mm to (357.8, 105.5)
- moved R1 0.40 mm to (351.4, 104.5)
Connections:
- net Net-(C1-Pad2) renamed +24V
Routing:
- net Net-(D25-K): track 353.3 -> 351.1 mm
Other:
- board text added: "LED_Driver V1.1"
- board text removed: "LED_Driver V1.0"
